File: Carte-Principale/Actionneurs.kicad_sch (KiCad schematic)
At the start: 38 parts, among them J17 I2C_Sensors, J20 AX12, M1 Motor_Servo, M10 Motor_Servo, M11 Motor_Servo, M12 Motor_Servo, M13 Motor_Servo, M2 Motor_Servo, M3 Motor_Servo, M4 Motor_Servo, M5 Motor_Servo, M6 Motor_Servo, M7 Motor_Servo, M8 Motor_Servo, M9 Motor_Servo, U1 PCA9685PW

Commit message: Final pcb modification
Parts:
- renumbered D3 to D1, D1 to D3, J17 to J14, J20 to J15, M8 to M12, M4 to M2, M2 to M4, M7 to M6, M6 to M7, M12 to M8, R15 to R13, R13 to R14, R14 to R15, R20 to R16, R18 to R17, R22 to R18, R21 to R20, R17 to R21, R16 to R22, R26 to R25, R25 to R26, R6 to R7
Changed lines of the file:
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@@
 		(on_board yes)
 		(dnp no)
-		(property "Reference" "R15"
+		(property "Reference" "R13"
 			(at 123.19 58.42 90)
 			(effects
@@
 			(project "Carte-Principale"
 				(path "/88b0dd29-ac24-4c5d-804c-fc642ecf6263/ec3b2e47-1720-4ba3-b32d-adf5bc711683"
-					(reference "R15")
+					(reference "R13")
 					(unit 1)
 				)
@@
 		(on_board yes)
 		(dnp no)
-		(property "Reference" "R17"
+		(property "Reference" "R21"
 			(at 123.19 63.5 90)
 			(effects
@@
 			(project "Carte-Principale"
 				(path "/88b0dd29-ac24-4c5d-804c-fc642ecf6263/ec3b2e47-1720-4ba3-b32d-adf5bc711683"
-					(reference "R17")
+					(reference "R21")
 					(unit 1)
 				)
@@
 		(on_board yes)
 		(dnp no)
-		(property "Reference" "R26"
+		(property "Reference" "R25"
 			(at 123.19 81.28 90)
 			(effects
@@
 			(project "Carte-Principale"
 				(path "/88b0dd29-ac24-4c5d-804c-fc642ecf6263/ec3b2e47-1720-4ba3-b32d-adf5bc711683"
-					(reference "R26")
+					(reference "R25")
 					(unit 1)
 				)
@@
 		(on_board yes)
 		(dnp no)
-		(property "Reference" "R16"
+		(property "Reference" "R22"
 			(at 123.19 76.2 90)
 			(effects
@@
 			(project "Carte-Principale"
 				(path "/88b0dd29-ac24-4c5d-804c-fc642ecf6263/ec3b2e47-1720-4ba3-b32d-adf5bc711683"
-					(reference "R16")
+					(reference "R22")
 					(unit 1)
 				)
@@
 		(on_board yes)
 		(dnp no)
-		(property "Reference" "R6"
+		(property "Reference" "R7"
 			(at 123.19 93.98 90)
 			(effects
@@
 			(project "Carte-Principale"
 				(path "/88b0dd29-ac24-4c5d-804c-fc642ecf6263/ec3b2e47-1720-4ba3-b32d-adf5bc711683"
-					(reference "R6")
+					(reference "R7")
 					(unit 1)
 				)
@@
 		(dnp no)
 		(fields_autoplaced yes)
-		(property "Reference" "M12"
+		(property "Reference" "M8"
 			(at 173.99 97.3565 0)
 			(effects
@@
 			(project "Carte-Principale"
 				(path "/88b0dd29-ac24-4c5d-804c-fc642ecf6263/ec3b2e47-1720-4ba3-b32d-adf5bc711683"
-					(reference "M12")
+					(reference "M8")
 					(unit 1)
 				)
@@
 		(on_board yes)
 		(dnp no)
-		(property "Reference" "D3"
+		(property "Reference" "D1"
 			(at 158.75 173.99 0)
 			(effects
@@
 			(project "Carte-Principale"
 				(path "/88b0dd29-ac24-4c5d-804c-fc642ecf6263/ec3b2e47-1720-4ba3-b32d-adf5bc711683"
-					(reference "D3")
+					(reference "D1")
 					(unit 1)
 				)
@@
 		(dnp no)
 		(fields_autoplaced yes)
-		(property "Reference" "M6"
+		(property "Reference" "M7"
 			(at 173.99 124.0265 0)
 			(effects
@@
 			(project "Carte-Principale"
 				(path "/88b0dd29-ac24-4c5d-804c-fc642ecf6263/ec3b2e47-1720-4ba3-b32d-adf5bc711683"
-					(reference "M6")
+					(reference "M7")
 					(unit 1)
 				)
@@
 		(dnp no)
 		(fields_autoplaced yes)
-		(property "Reference" "M2"
+		(property "Reference" "M4"
 			(at 173.99 70.6865 0)
 			(effects
@@
 			(project "Carte-Principale"
 				(path "/88b0dd29-ac24-4c5d-804c-fc642ecf6263/ec3b2e47-1720-4ba3-b32d-adf5bc711683"
-					(reference "M2")
+					(reference "M4")
 					(unit 1)
 				)
@@
 		(dnp no)
 		(fields_autoplaced yes)
-		(property "Reference" "M8"
+		(property "Reference" "M12"
 			(at 173.99 150.6965 0)
 			(effects
@@
 			(project "Carte-Principale"
 				(path "/88b0dd29-ac24-4c5d-804c-fc642ecf6263/ec3b2e47-1720-4ba3-b32d-adf5bc711683"
-					(reference "M8")
+					(reference "M12")
 					(unit 1)
 				)
@@
 		(dnp no)
 		(fields_autoplaced yes)
-		(property "Reference" "M4"
+		(property "Reference" "M2"
 			(at 173.99 61.7965 0)
 			(effects
@@
 			(project "Carte-Principale"
 				(path "/88b0dd29-ac24-4c5d-804c-fc642ecf6263/ec3b2e47-1720-4ba3-b32d-adf5bc711683"
-					(reference "M4")
+					(reference "M2")
 					(unit 1)
 				)
@@
 		(on_board yes)
 		(dnp no)
-		(property "Reference" "R22"
+		(property "Reference" "R18"
 			(at 123.19 66.04 90)
 			(effects
@@
 			(project "Carte-Principale"
 				(path "/88b0dd29-ac24-4c5d-804c-fc642ecf6263/ec3b2e47-1720-4ba3-b32d-adf5bc711683"
-					(reference "R22")
+					(reference "R18")
 					(unit 1)
 				)
@@
 		(on_board yes)
 		(dnp no)
-		(property "Reference" "R25"
+		(property "Reference" "R26"
 			(at 123.19 78.74 90)
 			(effects
@@
 			(project "Carte-Principale"
 				(path "/88b0dd29-ac24-4c5d-804c-fc642ecf6263/ec3b2e47-1720-4ba3-b32d-adf5bc711683"
-					(reference "R25")
+					(reference "R26")
 					(unit 1)
 				)
@@
 		(on_board yes)
 		(dnp no)
-		(property "Reference" "R14"
+		(property "Reference" "R15"
 			(at 123.19 55.88 90)
 			(effects
@@
 			(project "Carte-Principale"
 				(path "/88b0dd29-ac24-4c5d-804c-fc642ecf6263/ec3b2e47-1720-4ba3-b32d-adf5bc711683"
-					(reference "R14")
+					(reference "R15")
 					(unit 1)
 				)
@@
 		(dnp no)
 		(fields_autoplaced yes)
-		(property "Reference" "J17"
+		(property "Reference" "J14"
 			(at 54.61 41.9099 0)
 			(effects
@@
 			(project "Carte-Principale"
 				(path "/88b0dd29-ac24-4c5d-804c-fc642ecf6263/ec3b2e47-1720-4ba3-b32d-adf5bc711683"
-					(reference "J17")
+					(reference "J14")
 					(unit 1)
 				)
@@
 		(on_board yes)
 		(dnp no)
-		(property "Reference" "R13"
+		(property "Reference" "R14"
 			(at 123.19 60.96 90)
 			(effects
@@
 			(project "Carte-Principale"
 				(path "/88b0dd29-ac24-4c5d-804c-fc642ecf6263/ec3b2e47-1720-4ba3-b32d-adf5bc711683"
-					(reference "R13")
+					(reference "R14")
 					(unit 1)
 				)
@@
 		(dnp no)
 		(fields_autoplaced yes)
-		(property "Reference" "M7"
+		(property "Reference" "M6"
 			(at 173.99 106.2465 0)
 			(effects
@@
 			(project "Carte-Principale"
 				(path "/88b0dd29-ac24-4c5d-804c-fc642ecf6263/ec3b2e47-1720-4ba3-b32d-adf5bc711683"
-					(reference "M7")
+					(reference "M6")
 					(unit 1)
 				)
@@
 		(dnp no)
 		(fields_autoplaced yes)
-		(property "Reference" "J20"
+		(property "Reference" "J15"
 			(at 54.61 29.2099 0)
 			(effects
@@
 			(project "Carte-Principale"
 				(path "/88b0dd29-ac24-4c5d-804c-fc642ecf6263/ec3b2e47-1720-4ba3-b32d-adf5bc711683"
-					(reference "J20")
+					(reference "J15")
 					(unit 1)
 				)
@@
 		(on_board yes)
 		(dnp no)
-		(property "Reference" "D1"
+		(property "Reference" "D3"
 			(at 158.75 179.07 0)
 			(effects
@@
 			(project "Carte-Principale"
 				(path "/88b0dd29-ac24-4c5d-804c-fc642ecf6263/ec3b2e47-1720-4ba3-b32d-adf5bc711683"
-					(reference "D1")
+					(reference "D3")
 					(unit 1)
 				)
@@
 		(on_board yes)
 		(dnp no)
-		(property "Reference" "R20"
+		(property "Reference" "R16"
 			(at 123.19 73.66 90)
 			(effects
@@
 			(project "Carte-Principale"
 				(path "/88b0dd29-ac24-4c5d-804c-fc642ecf6263/ec3b2e47-1720-4ba3-b32d-adf5bc711683"
-					(reference "R20")
+					(reference "R16")
 					(unit 1)
 				)
@@
 		(on_board yes)
 		(dnp no)
-		(property "Reference" "R18"
+		(property "Reference" "R17"
 			(at 123.19 71.12 90)
 			(effects
@@
 			(project "Carte-Principale"
 				(path "/88b0dd29-ac24-4c5d-804c-fc642ecf6263/ec3b2e47-1720-4ba3-b32d-adf5bc711683"
-					(reference "R18")
+					(reference "R17")
 					(unit 1)
 				)
@@
 		(on_board yes)
 		(dnp no)
-		(property "Reference" "R21"
+		(property "Reference" "R20"
 			(at 73.66 69.85 90)
 			(effects
@@
 			(project "Carte-Principale"
 				(path "/88b0dd29-ac24-4c5d-804c-fc642ecf6263/ec3b2e47-1720-4ba3-b32d-adf5bc711683"
-					(reference "R21")
+					(reference "R20")
 					(unit 1)
 				)
