File: Carte-Principale/Actionneurs.kicad_sch (KiCad schematic)
At the start: 38 parts, among them J14 I2C_Sensors, J15 AX12, M1 Motor_Servo, M10 Motor_Servo, M11 Motor_Servo, M12 Motor_Servo, M13 Motor_Servo, M2 Motor_Servo, M3 Motor_Servo, M4 Motor_Servo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

Commit message: Cartes élec à refaire et TODO
Parts:
- removed C1: x, Capacitor_THT:CP_Radial_D8.0mm_P3.50mm, symbol Device:C_Polarized
- removed C2: 10u, Capacitor_SMD:C_1210_3225Metric_Pad1.33x2.70mm_HandSolder, symbol Device:C
- removed D1, D2, D3: LED, LED_SMD:LED_2010_5025Metric_Pad1.52x2.65mm_HandSolder, symbol Device:LED
- removed M1, M10, M11, M12, M13, M2, M3, M4, M5, M6, M7, M8, M9: Motor_Servo, Connector_PinHeader_2.54mm:PinHeader_1x03_P2.54mm_Vertical, symbol Motor:Motor_Servo
- removed R13, R14, R15, R21: 220, LED_SMD:LED_1210_3225Metric_Pad1.42x2.65mm_HandSolder, symbol Device:R
- removed R16, R17, R18, R19, R22, R23, R24, R25, R26: 220, Resistor_SMD:R_1210_3225Metric_Pad1.30x2.65mm_HandSolder, symbol Device:R
- removed R2, R5, R7: x, Resistor_SMD:R_1210_3225Metric_Pad1.30x2.65mm_HandSolder, symbol Device:R
- removed R20: 10k, LED_SMD:LED_1210_3225Metric_Pad1.42x2.65mm_HandSolder, symbol Device:R_Small
- removed U1: PCA9685PW, Package_SO:TSSOP-28_4.4x9.7mm_P0.65mm, symbol Driver_LED:PCA9685PW
- added J18: PCA9685, Connector_JST:JST_XH_B4B-XH-A_1x04_P2.50mm_Vertical, symbol Connector:Conn_01x04_Pin
- J14: footprint Connector_Molex:Molex_KK-254_AE-6410-04A_1x04_P2.54mm_Vertical -> Connector_JST:JST_XH_B4B-XH-A_1x04_P2.50mm_Vertical
- J15: footprint Connector_Molex:Molex_KK-254_AE-6410-03A_1x03_P2.54mm_Vertical -> Connector_JST:JST_XH_B3B-XH-A_1x03_P2.50mm_Vertical
Connections:
- net +5V: now also J18.1 (Pin_1)
- net GND: now also J18.4 (Pin_4)
- net SCL_Servo: now also J18.3 (Pin_3)
- net SDA_Servo: now also J18.2 (Pin_2)
Other:
- note removed: "Adresse: 1000 001x"

Commit message: FInal
Parts:
- removed J14: I2C_Sensors, Connector_JST:JST_XH_B4B-XH-A_1x04_P2.50mm_Vertical, symbol Connector:Conn_01x04_Pin
- added J10: Sensors, Connector_JST:JST_XH_B10B-XH-A_1x10_P2.50mm_Vertical, symbol Connector:Conn_01x10_Pin
Connections:
- net SCL_Sensors: now also J10.1 (Pin_1)
- net SDA_Sensors: now also J10.2 (Pin_2)
- new net SHUT_1: J10.3 (Pin_3)
- new net SHUT_2: J10.4 (Pin_4)
- new net SHUT_3: J10.5 (Pin_5)
- new net SHUT_4: J10.6 (Pin_6)
- new net SHUT_5: J10.7 (Pin_7)
- new net SHUT_6: J10.8 (Pin_8)
- new net SHUT_7: J10.9 (Pin_9)
- new net SHUT_8: J10.10 (Pin_10)
Other:
- note added: "PCB pour les Servos https://www.adafruit.com/product/815"
- note removed: "On peut acheter le PCB pour les Servos https://www.adafruit.com/product/815"
- note removed: "TODO: faire carte sensors (bien penser aux R de termination)"
Changed lines of the file:
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@@
 	(wire
 		(pts
-			(xy 41.91 46.99) (xy 48.26 46.99)
+			(xy 44.45 33.02) (xy 48.26 33.02)
 		)
 		(stroke
@@
 		)
 	)
-	(wire
-		(pts
-			(xy 44.45 33.02) (xy 48.26 33.02)
-		)
-		(stroke
-			(width 0)
-			(type default)
-		)
-	)
-	(text "TODO: faire carte sensors\n(bien penser aux R de termination)"
-		(exclude_from_sim no)
-		(at 49.53 50.8 0)
-		(effects
-			(font
-				(size 1.27 1.27)
-			)
-		)
-	)
-	(text "On peut acheter le PCB pour les Servos\nhttps://www.adafruit.com/product/815"
-		(exclude_from_sim no)
-		(at 43.18 21.59 0)
+	(text "PCB pour les Servos\nhttps://www.adafruit.com/product/815"
+		(exclude_from_sim no)
+		(at 48.26 71.12 0)
 		(effects
 			(font
@@
 	(hierarchical_label "SDA_Sensors"
 		(shape bidirectional)
-		(at 48.26 41.91 180)
-		(fields_autoplaced yes)
-		(effects
-			(font
-				(size 1.27 1.27)
-			)
-			(justify right)
+		(at 100.33 40.64 0)
+		(fields_autoplaced yes)
+		(effects
+			(font
+				(size 1.27 1.27)
+			)
+			(justify left)
+		)
+	)
+	(hierarchical_label "SCL_Sensors"
+		(shape bidirectional)
+		(at 100.33 38.1 0)
+		(fields_autoplaced yes)
+		(effects
+			(font
+				(size 1.27 1.27)
+			)
+			(justify left)
+		)
+	)
+	(hierarchical_label "SHUT_4"
+		(shape input)
+		(at 100.33 50.8 0)
+		(fields_autoplaced yes)
+		(effects
+			(font
+				(size 1.27 1.27)
+			)
+			(justify left)
+		)
+	)
+	(hierarchical_label "SHUT_1"
+		(shape input)
+		(at 100.33 43.18 0)
+		(fields_autoplaced yes)
+		(effects
+			(font
+				(size 1.27 1.27)
+			)
+			(justify left)
 		)
 	)
@@
 		)
 	)
-	(hierarchical_label "SCL_Sensors"
-		(shape bidirectional)
-		(at 48.26 44.45 180)
-		(fields_autoplaced yes)
-		(effects
-			(font
-				(size 1.27 1.27)
-			)
-			(justify right)
+	(hierarchical_label "SHUT_5"
+		(shape input)
+		(at 100.33 53.34 0)
+		(fields_autoplaced yes)
+		(effects
+			(font
+				(size 1.27 1.27)
+			)
+			(justify left)
+		)
+	)
+	(hierarchical_label "SHUT_7"
+		(shape input)
+		(at 100.33 58.42 0)
+		(fields_autoplaced yes)
+		(effects
+			(font
+				(size 1.27 1.27)
+			)
+			(justify left)
 		)
 	)
@@
 		)
 	)
-	(hierarchical_label "IT_Ready_Sensors"
-		(shape output)
-		(at 48.26 39.37 180)
-		(fields_autoplaced yes)
-		(effects
-			(font
-				(size 1.27 1.27)
-			)
-			(justify right)
+	(hierarchical_label "SHUT_2"
+		(shape input)
+		(at 100.33 45.72 0)
+		(fields_autoplaced yes)
+		(effects
+			(font
+				(size 1.27 1.27)
+			)
+			(justify left)
+		)
+	)
+	(hierarchical_label "SHUT_8"
+		(shape input)
+		(at 100.33 60.96 0)
+		(fields_autoplaced yes)
+		(effects
+			(font
+				(size 1.27 1.27)
+			)
+			(justify left)
+		)
+	)
+	(hierarchical_label "SHUT_6"
+		(shape input)
+		(at 100.33 55.88 0)
+		(fields_autoplaced yes)
+		(effects
+			(font
+				(size 1.27 1.27)
+			)
+			(justify left)
+		)
+	)
+	(hierarchical_label "SHUT_3"
+		(shape input)
+		(at 100.33 48.26 0)
+		(fields_autoplaced yes)
+		(effects
+			(font
+				(size 1.27 1.27)
+			)
+			(justify left)
 		)
 	)
@@
 	)
 	(symbol
+		(lib_id "Connector:Conn_01x10_Pin")
+		(at 95.25 48.26 0)
+		(unit 1)
+		(exclude_from_sim no)
+		(in_bom yes)
+		(on_board yes)
+		(dnp no)
+		(fields_autoplaced yes)
+		(property "Reference" "J10"
+			(at 95.885 33.02 0)
+			(effects
+				(font
+					(size 1.27 1.27)
+				)
+			)
+		)
+		(property "Value" "Sensors"
+			(at 95.885 35.56 0)
+			(effects
+				(font
+					(size 1.27 1.27)
+				)
+			)
+		)
+		(property "Footprint" "Connector_JST:JST_XH_B10B-XH-A_1x10_P2.50mm_Vertical"
+			(at 95.25 48.26 0)
+			(effects
+				(font
+					(size 1.27 1.27)
+				)
+				(hide yes)
+			)
+		)
+		(property "Datasheet" "~"
+			(at 95.25 48.26 0)
+			(effects
+				(font
+					(size 1.27 1.27)
+				)
+				(hide yes)
+			)
+		)
+		(property "Description" "Generic connector, single row, 01x10, script generated"
+			(at 95.25 48.26 0)
+			(effects
+				(font
+					(size 1.27 1.27)
+				)
+				(hide yes)
+			)
+		)
+		(pin "3"
+		)
+		(pin "7"
+		)
+		(pin "8"
+		)
+		(pin "9"
+		)
+		(pin "5"
+		)
+		(pin "6"
+		)
+		(pin "2"
+		)
+		(pin "1"
+		)
+		(pin "10"
+		)
+		(pin "4"
+		)
+		(instances
+			(project "Carte-Principale"
+				(path "/88b0dd29-ac24-4c5d-804c-fc642ecf6263/ec3b2e47-1720-4ba3-b32d-adf5bc711683"
+					(reference "J10")
+					(unit 1)
+				)
+			)
+		)
+	)
+	(symbol
 		(lib_id "power:+5V")
 		(at 43.18 66.04 90)
@@
 	)
 	(symbol
-		(lib_id "Connector:Conn_01x04_Pin")
-		(at 53.34 44.45 180)
-		(unit 1)
-		(exclude_from_sim no)
-		(in_bom yes)
-		(on_board yes)
-		(dnp no)
-		(fields_autoplaced yes)
-		(property "Reference" "J14"
-			(at 54.61 41.9099 0)
-			(effects
-				(font
-					(size 1.27 1.27)
-				)
-				(justify right)
-			)
-		)
-		(property "Value" "I2C_Sensors"
-			(at 54.61 44.4499 0)
-			(effects
-				(font
-					(size 1.27 1.27)
-				)
-				(justify right)
-			)
-		)
-		(property "Footprint" "Connector_JST:JST_XH_B4B-XH-A_1x04_P2.50mm_Vertical"
-			(at 53.34 44.45 0)
-			(effects
-				(font
-					(size 1.27 1.27)
-				)
-				(hide yes)
-			)
-		)
-		(property "Datasheet" "~"
-			(at 53.34 44.45 0)
-			(effects
-				(font
-					(size 1.27 1.27)
-				)
-				(hide yes)
-			)
-		)
-		(property "Description" "Generic connector, single row, 01x04, script generated"
-			(at 53.34 44.45 0)
-			(effects
-				(font
-					(size 1.27 1.27)
-				)
-				(hide yes)
-			)
-		)
-		(pin "4"
-		)
-		(pin "3"
-		)
-		(pin "2"
-		)
-		(pin "1"
-		)
-		(instances
-			(project "Carte-Principale"
-				(path "/88b0dd29-ac24-4c5d-804c-fc642ecf6263/ec3b2e47-1720-4ba3-b32d-adf5bc711683"
-					(reference "J14")
-					(unit 1)
-				)
-			)
-		)
-	)
-	(symbol
 		(lib_id "power:GND")
 		(at 44.45 33.02 270)
@@
 					(unit 1)
 				)
-			)
-		)
-	)
-	(symbol
-		(lib_id "power:GND")
-		(at 41.91 46.99 270)
-		(unit 1)
-		(exclude_from_sim no)
-		(in_bom yes)
-		(on_board yes)
-		(dnp no)
-		(fields_autoplaced yes)
-		(property "Reference" "#PWR047"
-			(at 35.56 46.99 0)
-			(effects
-				(font
-					(size 1.27 1.27)
-				)
-				(hide yes)
-			)
-		)
-		(property "Value" "GND"
-			(at 38.1 46.9899 90)
-			(effects
-				(font
-					(size 1.27 1.27)
-				)
-				(justify right)
-			)
-		)
-		(property "Footprint" ""
-			(at 41.91 46.99 0)
-			(effects
-				(font
-					(size 1.27 1.27)
-				)
-				(hide yes)
-			)
-		)
-		(property "Datasheet" ""
-			(at 41.91 46.99 0)
-			(effects
-				(font
-					(size 1.27 1.27)
-				)
-				(hide yes)
-			)
-		)
-		(property "Description" "Power symbol creates a global label with name \"GND\" , ground"
-			(at 41.91 46.99 0)
-			(effects
-				(font
-					(size 1.27 1.27)
-				)
-				(hide yes)
-			)
-		)
-		(pin "1"
-		)
-		(instances
-			(project "Carte-Principale"
-				(path "/88b0dd29-ac24-4c5d-804c-fc642ecf6263/ec3b2e47-1720-4ba3-b32d-adf5bc711683"
-					(reference "#PWR047")
-					(unit 1)
-				)

Commit message: abcdefgh
Other:
- company: CRINSA -> CRINSA - Boris HILKENS
Changed lines of the file:
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@@
 	(title_block
 		(title "Carte Principale")
-		(date "2024-08-12")
-		(company "CRINSA")
+		(date "2024-12-27")
+		(rev "V1")
+		(company "CRINSA - Boris HILKENS")
 		(comment 1 "Carte de contrôle pour le robot")
 	)
