File: Carte-Principale/encodeurs.kicad_sch (KiCad schematic)
At the start: 0 parts

Commit message: Moteurs + Encodeurs
Parts:
- added J3: Encodeur_G, symbol Connector:Conn_01x08_Pin
- added J4: Encodeur_D, symbol Connector:Conn_01x08_Pin
- added R1, R2, R3, R4: 100, symbol Device:R_Small
- added U6: AM26LV32xD, Package_SO:SOIC-16_3.9x9.9mm_P1.27mm, symbol Interface:AM26LV32xD
Connections:
- new net +3.3V: U6.16 (VDD), U6.4 (G)
- new net +5V: J3.1 (Pin_1), J4.1 (Pin_1)
- new net A+_DROITE: J4.6 (Pin_6), R4.2, U6.2 (1A)
- new net A+_GAUCHE: J3.6 (Pin_6), R2.2, U6.10 (3A)
- new net A-_DROITE: J4.7 (Pin_7), R4.1, U6.1 (1B)
- new net A-_GAUCHE: J3.7 (Pin_7), R2.1, U6.9 (3B)
- new net A_DROITE: U6.3 (1Y)
- new net A_GAUCHE: U6.11 (3Y)
- new net B+_DROITE: J4.5 (Pin_5), R3.2, U6.6 (2A)
- new net B+_GAUCHE: J3.5 (Pin_5), R1.2, U6.14 (4A)
- new net B-_DROITE: J4.4 (Pin_4), R3.1, U6.7 (2B)
- new net B-_GAUCHE: J3.4 (Pin_4), R1.1, U6.15 (4B)
- new net B_DROITE: U6.5 (2Y)
- new net B_GAUCHE: U6.13 (4Y)
- new net GND: J3.8 (Pin_8), J4.8 (Pin_8), U6.12 (~{G}), U6.8 (GND)
- new net Z+_DROITE: J4.2 (Pin_2)
- new net Z+_GAUCHE: J3.2 (Pin_2)
- new net Z-_DROITE: J4.3 (Pin_3)
- new net Z-_GAUCHE: J3.3 (Pin_3)
Other:
- note added: "Bien mettre dans le bon sens dans le PCB"

Commit message: wiring
Parts:
- added TP1: Test_Gauche, TestPoint:TestPoint_2Pads_Pitch2.54mm_Drill0.8mm, symbol Connector:TestPoint_2Pole
- added TP2: Test_Droit, TestPoint:TestPoint_2Pads_Pitch2.54mm_Drill0.8mm, symbol Connector:TestPoint_2Pole
- J4: renamed from J3; footprint (none) -> Connector_PinHeader_2.54mm:PinHeader_1x08_P2.54mm_Vertical
- J5: renamed from J4; footprint (none) -> Connector_PinHeader_2.54mm:PinHeader_1x08_P2.54mm_Vertical
- R10: renamed from R4; footprint (none) -> Resistor_THT:R_Axial_DIN0207_L6.3mm_D2.5mm_P10.16mm_Horizontal
- R7: renamed from R1; footprint (none) -> Resistor_THT:R_Axial_DIN0207_L6.3mm_D2.5mm_P10.16mm_Horizontal
- R8: renamed from R2; footprint (none) -> Resistor_THT:R_Axial_DIN0207_L6.3mm_D2.5mm_P10.16mm_Horizontal
- R9: renamed from R3; footprint (none) -> Resistor_THT:R_Axial_DIN0207_L6.3mm_D2.5mm_P10.16mm_Horizontal
- renumbered U6 to U2
Connections:
- net A_DROITE: now also TP2.1
- net A_GAUCHE: now also TP1.1
- net B_DROITE: now also TP2.2
- net B_GAUCHE: now also TP1.2

Commit message: Schéma vérifié
Parts:
- renumbered J4 to J11, J5 to J12, TP1 to TP7, TP2 to TP8
Connections:
- no-connect marks 0 -> 4
Other:
- note removed: "Bien mettre dans le bon sens dans le PCB"
- company: (none) -> CRINSA
- title: (none) -> Carte Principale
- moved on the sheet: J11, J12, R10, R7, R8, R9, TP7, TP8, U2

Commit message: Avancée PCB
Parts:
- J8: renamed from J11; footprint Connector_PinHeader_2.54mm:PinHeader_1x08_P2.54mm_Vertical -> Connector_Molex:Molex_KK-254_AE-6410-08A_1x08_P2.54mm_Vertical
- J9: renamed from J12; footprint Connector_PinHeader_2.54mm:PinHeader_1x08_P2.54mm_Vertical -> Connector_Molex:Molex_KK-254_AE-6410-08A_1x08_P2.54mm_Vertical
- R6: renamed from R7; footprint Resistor_THT:R_Axial_DIN0207_L6.3mm_D2.5mm_P10.16mm_Horizontal -> Resistor_SMD:R_1210_3225Metric_Pad1.30x2.65mm_HandSolder
- R7: renamed from R8; footprint Resistor_THT:R_Axial_DIN0207_L6.3mm_D2.5mm_P10.16mm_Horizontal -> Resistor_SMD:R_1210_3225Metric_Pad1.30x2.65mm_HandSolder
- R8: renamed from R9; footprint Resistor_THT:R_Axial_DIN0207_L6.3mm_D2.5mm_P10.16mm_Horizontal -> Resistor_SMD:R_1210_3225Metric_Pad1.30x2.65mm_HandSolder
- R9: renamed from R10; footprint Resistor_THT:R_Axial_DIN0207_L6.3mm_D2.5mm_P10.16mm_Horizontal -> Resistor_SMD:R_1210_3225Metric_Pad1.30x2.65mm_HandSolder
- renumbered TP7 to TP6, TP8 to TP7
Changed lines of the file:
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@@
 		(dnp no)
 		(fields_autoplaced yes)
-		(property "Reference" "#PWR040"
+		(property "Reference" "#PWR034"
 			(at 125.73 97.79 0)
 			(effects
@@
 			(project "Carte-Principale"
 				(path "/88b0dd29-ac24-4c5d-804c-fc642ecf6263/a2923913-7939-4f75-8694-93f1ab74a018"
-					(reference "#PWR040")
+					(reference "#PWR034")
 					(unit 1)
 				)
@@
 		(dnp no)
 		(fields_autoplaced yes)
-		(property "Reference" "TP8"
+		(property "Reference" "TP7"
 			(at 40.64 77.4699 90)
 			(effects
@@
 			(project "Carte-Principale"
 				(path "/88b0dd29-ac24-4c5d-804c-fc642ecf6263/a2923913-7939-4f75-8694-93f1ab74a018"
-					(reference "TP8")
+					(reference "TP7")
 					(unit 1)
 				)
@@
 		(dnp no)
 		(fields_autoplaced yes)
-		(property "Reference" "#PWR033"
+		(property "Reference" "#PWR027"
 			(at 125.73 36.83 0)
 			(effects
@@
 			(project "Carte-Principale"
 				(path "/88b0dd29-ac24-4c5d-804c-fc642ecf6263/a2923913-7939-4f75-8694-93f1ab74a018"
-					(reference "#PWR033")
+					(reference "#PWR027")
 					(unit 1)
 				)
@@
 		(dnp no)
 		(fields_autoplaced yes)
-		(property "Reference" "J12"
+		(property "Reference" "J9"
 			(at 143.51 81.2801 0)
 			(effects
@@
 			)
 		)
-		(property "Footprint" "Connector_PinHeader_2.54mm:PinHeader_1x08_P2.54mm_Vertical"
+		(property "Footprint" "Connector_Molex:Molex_KK-254_AE-6410-08A_1x08_P2.54mm_Vertical"
 			(at 142.24 78.74 0)
 			(effects
@@
 			(project "Carte-Principale"
 				(path "/88b0dd29-ac24-4c5d-804c-fc642ecf6263/a2923913-7939-4f75-8694-93f1ab74a018"
-					(reference "J12")
+					(reference "J9")
 					(unit 1)
 				)
@@
 		(dnp no)
 		(fields_autoplaced yes)
-		(property "Reference" "TP7"
+		(property "Reference" "TP6"
 			(at 40.64 49.5299 90)
 			(effects
@@
 			(project "Carte-Principale"
 				(path "/88b0dd29-ac24-4c5d-804c-fc642ecf6263/a2923913-7939-4f75-8694-93f1ab74a018"
-					(reference "TP7")
+					(reference "TP6")
 					(unit 1)
 				)
@@
 		(dnp no)
 		(fields_autoplaced yes)
-		(property "Reference" "#PWR038"
+		(property "Reference" "#PWR032"
 			(at 125.73 74.93 0)
 			(effects
@@
 			(project "Carte-Principale"
 				(path "/88b0dd29-ac24-4c5d-804c-fc642ecf6263/a2923913-7939-4f75-8694-93f1ab74a018"
-					(reference "#PWR038")
+					(reference "#PWR032")
 					(unit 1)
 				)
@@
 		(dnp no)
 		(fields_autoplaced yes)
-		(property "Reference" "R9"
+		(property "Reference" "R8"
 			(at 88.9 73.6599 0)
 			(effects
@@
 			)
 		)
-		(property "Footprint" "Resistor_THT:R_Axial_DIN0207_L6.3mm_D2.5mm_P10.16mm_Horizontal"
+		(property "Footprint" "Resistor_SMD:R_1210_3225Metric_Pad1.30x2.65mm_HandSolder"
 			(at 86.36 74.93 0)
 			(effects
@@
 			(project "Carte-Principale"
 				(path "/88b0dd29-ac24-4c5d-804c-fc642ecf6263/a2923913-7939-4f75-8694-93f1ab74a018"
-					(reference "R9")
+					(reference "R8")
 					(unit 1)
 				)
@@
 		(dnp no)
 		(fields_autoplaced yes)
-		(property "Reference" "R8"
+		(property "Reference" "R7"
 			(at 88.9 53.3399 0)
 			(effects
@@
 			)
 		)
-		(property "Footprint" "Resistor_THT:R_Axial_DIN0207_L6.3mm_D2.5mm_P10.16mm_Horizontal"
+		(property "Footprint" "Resistor_SMD:R_1210_3225Metric_Pad1.30x2.65mm_HandSolder"
 			(at 86.36 54.61 0)
 			(effects
@@
 			(project "Carte-Principale"
 				(path "/88b0dd29-ac24-4c5d-804c-fc642ecf6263/a2923913-7939-4f75-8694-93f1ab74a018"
-					(reference "R8")
+					(reference "R7")
 					(unit 1)
 				)
@@
 		(on_board yes)
 		(dnp no)
-		(property "Reference" "#PWR036"
+		(property "Reference" "#PWR030"
 			(at 93.98 62.23 0)
 			(effects
@@
 			(project "Carte-Principale"
 				(path "/88b0dd29-ac24-4c5d-804c-fc642ecf6263/a2923913-7939-4f75-8694-93f1ab74a018"
-					(reference "#PWR036")
+					(reference "#PWR030")
 					(unit 1)
 				)
@@
 		(dnp no)
 		(fields_autoplaced yes)
-		(property "Reference" "#PWR034"
+		(property "Reference" "#PWR028"
 			(at 72.39 31.75 0)
 			(effects
@@
 			(project "Carte-Principale"
 				(path "/88b0dd29-ac24-4c5d-804c-fc642ecf6263/a2923913-7939-4f75-8694-93f1ab74a018"
-					(reference "#PWR034")
+					(reference "#PWR028")
 					(unit 1)
 				)
@@
 		(dnp no)
 		(fields_autoplaced yes)
-		(property "Reference" "J11"
+		(property "Reference" "J8"
 			(at 143.51 43.1801 0)
 			(effects
@@
 			)
 		)
-		(property "Footprint" "Connector_PinHeader_2.54mm:PinHeader_1x08_P2.54mm_Vertical"
+		(property "Footprint" "Connector_Molex:Molex_KK-254_AE-6410-08A_1x08_P2.54mm_Vertical"
 			(at 142.24 40.64 0)
 			(effects
@@
 			(project "Carte-Principale"
 				(path "/88b0dd29-ac24-4c5d-804c-fc642ecf6263/a2923913-7939-4f75-8694-93f1ab74a018"
-					(reference "J11")
+					(reference "J8")
 					(unit 1)
 				)
@@
 		(dnp no)
 		(fields_autoplaced yes)
-		(property "Reference" "R7"
+		(property "Reference" "R6"
 			(at 88.9 45.7199 0)
 			(effects
@@
 			)
 		)
-		(property "Footprint" "Resistor_THT:R_Axial_DIN0207_L6.3mm_D2.5mm_P10.16mm_Horizontal"
+		(property "Footprint" "Resistor_SMD:R_1210_3225Metric_Pad1.30x2.65mm_HandSolder"
 			(at 86.36 46.99 0)
 			(effects
@@
 			(project "Carte-Principale"
 				(path "/88b0dd29-ac24-4c5d-804c-fc642ecf6263/a2923913-7939-4f75-8694-93f1ab74a018"
-					(reference "R7")
+					(reference "R6")
 					(unit 1)
 				)
@@
 		(on_board yes)
 		(dnp no)
-		(property "Reference" "#PWR037"
+		(property "Reference" "#PWR031"
 			(at 83.82 67.31 0)
 			(effects
@@
 			(project "Carte-Principale"
 				(path "/88b0dd29-ac24-4c5d-804c-fc642ecf6263/a2923913-7939-4f75-8694-93f1ab74a018"
-					(reference "#PWR037")
+					(reference "#PWR031")
 					(unit 1)
 				)
@@
 		(dnp no)
 		(fields_autoplaced yes)
-		(property "Reference" "#PWR039"
+		(property "Reference" "#PWR033"
 			(at 72.39 87.63 0)
 			(effects
@@
 			(project "Carte-Principale"
 				(path "/88b0dd29-ac24-4c5d-804c-fc642ecf6263/a2923913-7939-4f75-8694-93f1ab74a018"
-					(reference "#PWR039")
+					(reference "#PWR033")
 					(unit 1)
 				)
@@
 		(dnp no)
 		(fields_autoplaced yes)
-		(property "Reference" "R10"
+		(property "Reference" "R9"
 			(at 88.9 81.2799 0)
 			(effects
@@
 			)
 		)
-		(property "Footprint" "Resistor_THT:R_Axial_DIN0207_L6.3mm_D2.5mm_P10.16mm_Horizontal"
+		(property "Footprint" "Resistor_SMD:R_1210_3225Metric_Pad1.30x2.65mm_HandSolder"
 			(at 86.36 82.55 0)
 			(effects
@@
 			(project "Carte-Principale"
 				(path "/88b0dd29-ac24-4c5d-804c-fc642ecf6263/a2923913-7939-4f75-8694-93f1ab74a018"
-					(reference "R10")
+					(reference "R9")
 					(unit 1)
 				)
@@
 		(dnp no)
 		(fields_autoplaced yes)
-		(property "Reference" "#PWR035"
+		(property "Reference" "#PWR029"
 			(at 125.73 59.69 0)
 			(effects
@@
 			(project "Carte-Principale"
 				(path "/88b0dd29-ac24-4c5d-804c-fc642ecf6263/a2923913-7939-4f75-8694-93f1ab74a018"
-					(reference "#PWR035")
-					(unit 1)
-				)
+					(reference "#PWR029")
+					(unit 1)
+				)

Commit message: avancée
Parts:
- renumbered J8 to J12, J9 to J7, R9 to R27, R6 to R28, R8 to R29, R7 to R30, TP6 to TP8, TP7 to TP9, U2 to U3
Changed lines of the file:
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@@
 		(dnp no)
 		(fields_autoplaced yes)
-		(property "Reference" "TP7"
+		(property "Reference" "TP9"
 			(at 40.64 77.4699 90)
 			(effects
@@
 			(project "Carte-Principale"
 				(path "/88b0dd29-ac24-4c5d-804c-fc642ecf6263/a2923913-7939-4f75-8694-93f1ab74a018"
-					(reference "TP7")
+					(reference "TP9")
 					(unit 1)
 				)
@@
 		(dnp no)
 		(fields_autoplaced yes)
-		(property "Reference" "J9"
+		(property "Reference" "J7"
 			(at 143.51 81.2801 0)
 			(effects
@@
 			(project "Carte-Principale"
 				(path "/88b0dd29-ac24-4c5d-804c-fc642ecf6263/a2923913-7939-4f75-8694-93f1ab74a018"
-					(reference "J9")
+					(reference "J7")
 					(unit 1)
 				)
@@
 		(dnp no)
 		(fields_autoplaced yes)
-		(property "Reference" "TP6"
+		(property "Reference" "TP8"
 			(at 40.64 49.5299 90)
 			(effects
@@
 			(project "Carte-Principale"
 				(path "/88b0dd29-ac24-4c5d-804c-fc642ecf6263/a2923913-7939-4f75-8694-93f1ab74a018"
-					(reference "TP6")
+					(reference "TP8")
 					(unit 1)
 				)
@@
 		(dnp no)
 		(fields_autoplaced yes)
-		(property "Reference" "R8"
+		(property "Reference" "R29"
 			(at 88.9 73.6599 0)
 			(effects
@@
 			(project "Carte-Principale"
 				(path "/88b0dd29-ac24-4c5d-804c-fc642ecf6263/a2923913-7939-4f75-8694-93f1ab74a018"
-					(reference "R8")
+					(reference "R29")
 					(unit 1)
 				)
@@
 		(dnp no)
 		(fields_autoplaced yes)
-		(property "Reference" "R7"
+		(property "Reference" "R30"
 			(at 88.9 53.3399 0)
 			(effects
@@
 			(project "Carte-Principale"
 				(path "/88b0dd29-ac24-4c5d-804c-fc642ecf6263/a2923913-7939-4f75-8694-93f1ab74a018"
-					(reference "R7")
+					(reference "R30")
 					(unit 1)
 				)
@@
 		(dnp no)
 		(fields_autoplaced yes)
-		(property "Reference" "J8"
+		(property "Reference" "J12"
 			(at 143.51 43.1801 0)
 			(effects
@@
 			(project "Carte-Principale"
 				(path "/88b0dd29-ac24-4c5d-804c-fc642ecf6263/a2923913-7939-4f75-8694-93f1ab74a018"
-					(reference "J8")
+					(reference "J12")
 					(unit 1)
 				)
@@
 		(dnp no)
 		(fields_autoplaced yes)
-		(property "Reference" "R6"
+		(property "Reference" "R28"
 			(at 88.9 45.7199 0)
 			(effects
@@
 			(project "Carte-Principale"
 				(path "/88b0dd29-ac24-4c5d-804c-fc642ecf6263/a2923913-7939-4f75-8694-93f1ab74a018"
-					(reference "R6")
+					(reference "R28")
 					(unit 1)
 				)
@@
 		(dnp no)
 		(fields_autoplaced yes)
-		(property "Reference" "R9"
+		(property "Reference" "R27"
 			(at 88.9 81.2799 0)
 			(effects
@@
 			(project "Carte-Principale"
 				(path "/88b0dd29-ac24-4c5d-804c-fc642ecf6263/a2923913-7939-4f75-8694-93f1ab74a018"
-					(reference "R9")
+					(reference "R27")
 					(unit 1)
 				)
@@
 		(dnp no)
 		(fields_autoplaced yes)
-		(property "Reference" "U2"
+		(property "Reference" "U3"
 			(at 75.4065 36.83 0)
 			(effects
@@
 			(project "Carte-Principale"
 				(path "/88b0dd29-ac24-4c5d-804c-fc642ecf6263/a2923913-7939-4f75-8694-93f1ab74a018"
-					(reference "U2")
-					(unit 1)
-				)
+					(reference "U3")
+					(unit 1)
+				)

Commit message: Final pcb modification
Parts:
- renumbered J12 to J13, J7 to J8, R30 to R28, R28 to R30
Changed lines of the file:
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@@
 		(dnp no)
 		(fields_autoplaced yes)
-		(property "Reference" "J7"
+		(property "Reference" "J8"
 			(at 143.51 81.2801 0)
 			(effects
@@
 			(project "Carte-Principale"
 				(path "/88b0dd29-ac24-4c5d-804c-fc642ecf6263/a2923913-7939-4f75-8694-93f1ab74a018"
-					(reference "J7")
+					(reference "J8")
 					(unit 1)
 				)
@@
 		(dnp no)
 		(fields_autoplaced yes)
-		(property "Reference" "R30"
+		(property "Reference" "R28"
 			(at 88.9 53.3399 0)
 			(effects
@@
 			(project "Carte-Principale"
 				(path "/88b0dd29-ac24-4c5d-804c-fc642ecf6263/a2923913-7939-4f75-8694-93f1ab74a018"
-					(reference "R30")
+					(reference "R28")
 					(unit 1)
 				)
@@
 		(dnp no)
 		(fields_autoplaced yes)
-		(property "Reference" "J12"
+		(property "Reference" "J13"
 			(at 143.51 43.1801 0)
 			(effects
@@
 			(project "Carte-Principale"
 				(path "/88b0dd29-ac24-4c5d-804c-fc642ecf6263/a2923913-7939-4f75-8694-93f1ab74a018"
-					(reference "J12")
+					(reference "J13")
 					(unit 1)
 				)
@@
 		(dnp no)
 		(fields_autoplaced yes)
-		(property "Reference" "R28"
+		(property "Reference" "R30"
 			(at 88.9 45.7199 0)
 			(effects
@@
 			(project "Carte-Principale"
 				(path "/88b0dd29-ac24-4c5d-804c-fc642ecf6263/a2923913-7939-4f75-8694-93f1ab74a018"
-					(reference "R28")
-					(unit 1)
-				)
+					(reference "R30")
+					(unit 1)
+				)

Commit message: Cartes élec à refaire et TODO
Parts:
- added C7: 0.1µ, Capacitor_SMD:C_1210_3225Metric_Pad1.33x2.70mm_HandSolder, symbol Device:C_Small
- J13, J8: footprint Connector_Molex:Molex_KK-254_AE-6410-08A_1x08_P2.54mm_Vertical -> Connector_JST:JST_XH_B8B-XH-A_1x08_P2.50mm_Vertical
Connections:
- net +3.3V: now also C7.1
- net GND: now also C7.2
Changed lines of the file:
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@@
+		(color 0 0 0 0)
+	)
+	(junction
+		(at 72.39 93.98)
+		(diameter 0)
 		(color 0 0 0 0)
 	)
@@
 	(wire
 		(pts
+			(xy 77.47 99.06) (xy 77.47 101.6)
+		)
+		(stroke
+			(width 0)
+			(type default)
+		)
+	)
+	(wire
+		(pts
 			(xy 87.63 62.23) (xy 85.09 62.23)
 		)
@@
 	(wire
 		(pts
+			(xy 72.39 93.98) (xy 72.39 90.17)
+		)
+		(stroke
+			(width 0)
+			(type default)
+		)
+	)
+	(wire
+		(pts
 			(xy 137.16 33.02) (xy 125.73 33.02)
 		)
@@
 	(wire
 		(pts
-			(xy 72.39 91.44) (xy 72.39 90.17)
+			(xy 72.39 96.52) (xy 72.39 93.98)
 		)
 		(stroke
@@
 		(pts
 			(xy 95.25 85.09) (xy 86.36 85.09)
+		)
+		(stroke
+			(width 0)
+			(type default)
+		)
+	)
+	(wire
+		(pts
+			(xy 72.39 93.98) (xy 77.47 93.98)
 		)
 		(stroke
@@
 			)
 		)
-		(property "Footprint" "Connector_Molex:Molex_KK-254_AE-6410-08A_1x08_P2.54mm_Vertical"
+		(property "Footprint" "Connector_JST:JST_XH_B8B-XH-A_1x08_P2.50mm_Vertical"
 			(at 142.24 78.74 0)
 			(effects
@@
 				(path "/88b0dd29-ac24-4c5d-804c-fc642ecf6263/a2923913-7939-4f75-8694-93f1ab74a018"
 					(reference "TP8")
+					(unit 1)
+				)
+			)
+		)
+	)
+	(symbol
+		(lib_id "power:GND")
+		(at 77.47 101.6 0)
+		(unit 1)
+		(exclude_from_sim no)
+		(in_bom yes)
+		(on_board yes)
+		(dnp no)
+		(fields_autoplaced yes)
+		(property "Reference" "#PWR011"
+			(at 77.47 107.95 0)
+			(effects
+				(font
+					(size 1.27 1.27)
+				)
+				(hide yes)
+			)
+		)
+		(property "Value" "GND"
+			(at 77.47 106.68 0)
+			(effects
+				(font
+					(size 1.27 1.27)
+				)
+			)
+		)
+		(property "Footprint" ""
+			(at 77.47 101.6 0)
+			(effects
+				(font
+					(size 1.27 1.27)
+				)
+				(hide yes)
+			)
+		)
+		(property "Datasheet" ""
+			(at 77.47 101.6 0)
+			(effects
+				(font
+					(size 1.27 1.27)
+				)
+				(hide yes)
+			)
+		)
+		(property "Description" "Power symbol creates a global label with name \"GND\" , ground"
+			(at 77.47 101.6 0)
+			(effects
+				(font
+					(size 1.27 1.27)
+				)
+				(hide yes)
+			)
+		)
+		(pin "1"
+		)
+		(instances
+			(project "Carte-Principale"
+				(path "/88b0dd29-ac24-4c5d-804c-fc642ecf6263/a2923913-7939-4f75-8694-93f1ab74a018"
+					(reference "#PWR011")
 					(unit 1)
 				)
@@
 			)
 		)
-		(property "Footprint" "Connector_Molex:Molex_KK-254_AE-6410-08A_1x08_P2.54mm_Vertical"
+		(property "Footprint" "Connector_JST:JST_XH_B8B-XH-A_1x08_P2.50mm_Vertical"
 			(at 142.24 40.64 0)
 			(effects
@@
 	(symbol
 		(lib_id "power:+3.3V")
-		(at 72.39 91.44 180)
+		(at 72.39 96.52 180)
 		(unit 1)
 		(exclude_from_sim no)
@@
 		(fields_autoplaced yes)
 		(property "Reference" "#PWR033"
-			(at 72.39 87.63 0)
+			(at 72.39 92.71 0)
 			(effects
 				(font
@@
 		)
 		(property "Value" "+3.3V"
+			(at 72.39 101.6 0)
+			(effects
+				(font
+					(size 1.27 1.27)
+				)
+			)
+		)
+		(property "Footprint" ""
 			(at 72.39 96.52 0)
 			(effects
@@
 					(size 1.27 1.27)
 				)
-			)
-		)
-		(property "Footprint" ""
-			(at 72.39 91.44 0)
-			(effects
-				(font
-					(size 1.27 1.27)
-				)
 				(hide yes)
 			)
 		)
 		(property "Datasheet" ""
-			(at 72.39 91.44 0)
+			(at 72.39 96.52 0)
 			(effects
 				(font
@@
 		)
 		(property "Description" "Power symbol creates a global label with name \"+3.3V\""
-			(at 72.39 91.44 0)
+			(at 72.39 96.52 0)
 			(effects
 				(font
@@
 					(unit 1)
 				)
+			)
+		)
+	)
+	(symbol
+		(lib_id "Device:C_Small")
+		(at 77.47 96.52 0)
+		(unit 1)
+		(exclude_from_sim no)
+		(in_bom yes)
+		(on_board yes)
+		(dnp no)
+		(fields_autoplaced yes)
+		(property "Reference" "C7"
+			(at 80.01 95.2562 0)
+			(effects
+				(font
+					(size 1.27 1.27)
+				)
+				(justify left)
+			)
+		)
+		(property "Value" "0.1µ"
+			(at 80.01 97.7962 0)
+			(effects
+				(font
+					(size 1.27 1.27)
+				)
+				(justify left)
+			)
+		)
+		(property "Footprint" "Capacitor_SMD:C_1210_3225Metric_Pad1.33x2.70mm_HandSolder"
+			(at 77.47 96.52 0)
+			(effects
+				(font
+					(size 1.27 1.27)
+				)
+				(hide yes)
+			)
+		)
+		(property "Datasheet" "~"
+			(at 77.47 96.52 0)
+			(effects
+				(font
+					(size 1.27 1.27)
+				)
+				(hide yes)
+			)
+		)
+		(property "Description" "Unpolarized capacitor, small symbol"
+			(at 77.47 96.52 0)
+			(effects
+				(font
+					(size 1.27 1.27)
+				)
+				(hide yes)
+			)
+		)
+		(pin "2"
+		)
+		(pin "1"
+		)
+		(instances
+			(project "Carte-Principale"
+				(path "/88b0dd29-ac24-4c5d-804c-fc642ecf6263/a2923913-7939-4f75-8694-93f1ab74a018"
+					(reference "C7")
+					(unit 1)
+				)
