File: Carte-Principale/encodeurs.kicad_sch (KiCad schematic)
At the start: 10 parts, among them J13 Encodeur_G, J8 Encodeur_D, U3 AM26LV32xD

Commit message: FInal
Other:
- note added: "Comme les années précédentes"
Changed lines of the file:
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@@
+		)
+	)
+	(text "Comme les années précédentes"
+		(exclude_from_sim no)
+		(at 72.39 29.21 0)
+		(effects
+			(font
+				(size 1.27 1.27)
+			)
 		)
 	)

Commit message: abcdefgh
Other:
- company: CRINSA -> CRINSA - Boris HILKENS
Changed lines of the file:
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@@
 	(title_block
 		(title "Carte Principale")
-		(date "2024-08-12")
-		(company "CRINSA")
+		(date "2024-12-27")
+		(rev "V1")
+		(company "CRINSA - Boris HILKENS")
 		(comment 1 "Carte de contrôle pour le robot")
 	)
