File: Carte-Principale/interface.kicad_sch (KiCad schematic)
At the start: 0 parts

Commit message: Rajout écran
Parts:
- added J7: LCD_TFT, symbol Connector:Conn_01x14_Pin
- added J8: LCD_SD, symbol Connector:Conn_01x04_Pin
- added R33, R35, R36, R37: 10K, symbol Device:R_Small
- added R34, R38, R39, R40: x, symbol Device:R_Small
- added R42, R43, R44, R45: 10k, symbol Device:R
- added SW1: Rouge, symbol Switch:SW_Push_LED
- added SW2: Bleu, symbol Switch:SW_Push_LED
- added SW3: Jaune, symbol Switch:SW_Push_LED
- added SW4: Selector1, symbol Switch:SW_SPDT
- added SW5: Selector2, symbol Switch:SW_SPDT
- added SW6: Vert, symbol Switch:SW_Push_LED
Connections:
- new net: R40.1, SW1.4 (A)
- new net: R39.1, SW6.4 (A)
- new net: R38.1, SW3.4 (A)
- new net: R34.1, SW2.4 (A)
- new net +5V: J7.1 (Pin_1), R33.2, R35.2, R36.2, R37.2, SW4.2 (B), SW5.2 (B)
- new net Bleu_LED: R34.2
- new net Bleu_SW: R33.1, SW2.2
- new net CLK_SD: J8.4 (Pin_4)
- new net CS_LCD: J7.3 (Pin_3)
- new net CS_SD: J8.1 (Pin_1)
- new net DC_LCD: J7.5 (Pin_5)
- new net GND: J7.2 (Pin_2), R42.2, R43.2, R44.2, R45.2, SW1.1, SW1.3 (K), SW2.1, SW2.3 (K), SW3.1, SW3.3 (K), SW6.1, SW6.3 (K)
- new net Jaune_LED: R38.2
- new net Jaune_SW: R35.1, SW3.2
- new net LED_LCD: J7.8 (Pin_8)
- new net MISO_LCD: J7.9 (Pin_9)
- new net MISO_SD: J8.3 (Pin_3)
- new net MOSI_LCD: J7.6 (Pin_6)
- new net MOSI_SD: J8.2 (Pin_2)
- new net RESET_LCD: J7.4 (Pin_4)
- new net Rouge_LED: R40.2
- new net Rouge_SW: R37.1, SW1.2
- new net SCK_LCD: J7.7 (Pin_7)
- new net Selector1_1: R45.1, SW4.1 (A)
- new net Selector1_2: R44.1, SW4.3 (C)
- new net Selector2_1: R42.1, SW5.1 (A)
- new net Selector2_2: R43.1, SW5.3 (C)
- new net T_CLK_LCD: J7.10 (Pin_10)
- new net T_CS_LCD: J7.11 (Pin_11)
- new net T_DIN_LCD: J7.12 (Pin_12)
- new net T_DO_LCD: J7.13 (Pin_13)
- new net T_IRQ_LCD: J7.14 (Pin_14)
- new net Vert_LED: R39.2
- new net Vert_SW: R36.1, SW6.2

Commit message: wiring
Parts:
- removed R34, R38, R39, R40: x, symbol Device:R_Small
- removed R42, R43, R44, R45: 10k, symbol Device:R
- removed SW4: Selector1, symbol Switch:SW_SPDT
- removed SW5: Selector2, symbol Switch:SW_SPDT
- added Q2, Q3, Q4, Q5: BSS138, Package_TO_SOT_SMD:SOT-23, symbol Transistor_FET:BSS138
- added R11, R13, R15, R17: 10k, Resistor_SMD:R_1206_3216Metric_Pad1.30x1.75mm_HandSolder, symbol Device:R_Small
- J11: renamed from J7; footprint (none) -> Connector_PinSocket_2.54mm:PinSocket_1x14_P2.54mm_Vertical
- J12: renamed from J8; footprint (none) -> Connector_PinSocket_2.54mm:PinSocket_1x04_P2.54mm_Vertical
- R12: renamed from R36; footprint (none) -> Resistor_SMD:R_1206_3216Metric_Pad1.30x1.75mm_HandSolder
- R14: renamed from R35; footprint (none) -> Resistor_SMD:R_1206_3216Metric_Pad1.30x1.75mm_HandSolder
- R16: renamed from R33; footprint (none) -> Resistor_SMD:R_1206_3216Metric_Pad1.30x1.75mm_HandSolder
- R18: renamed from R37; footprint (none) -> Resistor_SMD:R_1206_3216Metric_Pad1.30x1.75mm_HandSolder
- SW2: renamed from SW6; footprint (none) -> Connector_PinHeader_2.54mm:PinHeader_1x04_P2.54mm_Vertical
- SW3: footprint (none) -> Connector_PinHeader_2.54mm:PinHeader_1x04_P2.54mm_Vertical
- SW4: renamed from SW2; footprint (none) -> Connector_PinHeader_2.54mm:PinHeader_1x04_P2.54mm_Vertical
- SW5: renamed from SW1; footprint (none) -> Connector_PinHeader_2.54mm:PinHeader_1x04_P2.54mm_Vertical
Connections:
- net LED_LCD is gone; now on net +5V: J11.8 (Pin_8)
- net +5V: now also SW2.4 (A), SW3.4 (A), SW4.4 (A), SW5.4 (A)
- net Bleu_LED: now also Q4.1 (G), R15.2
- net GND: now also Q2.2 (S), Q3.2 (S), Q4.2 (S), Q5.2 (S), R11.1, R13.1, R15.1, R17.1; no longer SW2.3 (K), SW3.3 (K), SW4.3 (K), SW5.3 (K)
- net Jaune_LED: now also Q3.1 (G), R13.2
- net Rouge_LED: now also Q5.1 (G), R17.2
- net Vert_LED: now also Q2.1 (G), R11.2
- net CLK_SD renamed SCK_SD
- net T_CLK_LCD renamed T_SCK_LCD
- net T_DIN_LCD renamed T_MISO_LCD
- net T_DO_LCD renamed T_MOSI_LCD
- new net: Q3.3 (D), SW3.3 (K)
- new net: Q4.3 (D), SW4.3 (K)
- new net: Q5.3 (D), SW5.3 (K)
- new net: Q2.3 (D), SW2.3 (K)
Other:
- moved on the sheet: R12, R14, R16, R18, SW2, SW3, SW4, SW5

Commit message: Schéma vérifié
Parts:
- R11, R12, R13, R14, R15, R16, R17, R18: footprint Resistor_SMD:R_1206_3216Metric_Pad1.30x1.75mm_HandSolder -> Resistor_SMD:R_1210_3225Metric_Pad1.30x2.65mm_HandSolder
- SW2, SW3, SW4, SW5: footprint Connector_PinHeader_2.54mm:PinHeader_1x04_P2.54mm_Vertical -> Connector_Molex:Molex_KK-254_AE-6410-04A_1x04_P2.54mm_Vertical
- renumbered J11 to J18, J12 to J19
Connections:
- net +5V: no longer J18.1 (Pin_1), J18.8 (Pin_8)
- new net +3.3V: J18.1 (Pin_1), J18.8 (Pin_8)
Other:
- company: (none) -> CRINSA
- title: (none) -> Carte Principale
- moved on the sheet: J18, J19, Q2, Q3, Q4, Q5, R11, R12, R13, R14, R15, R16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

Commit message: Avancée PCB
Parts:
- renumbered J18 to J14, J19 to J15, R11 to R27, R12 to R28, R13 to R29, R14 to R30, R15 to R31, R16 to R32, R17 to R33, R18 to R34, SW2 to SW1, SW3 to SW2, SW4 to SW3, SW5 to SW4
Changed lines of the file:
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@@
 		(dnp no)
 		(fields_autoplaced yes)
-		(property "Reference" "#PWR058"
+		(property "Reference" "#PWR084"
 			(at 53.34 50.8 0)
 			(effects
@@
 			(project "Carte-Principale"
 				(path "/88b0dd29-ac24-4c5d-804c-fc642ecf6263/d641269b-1187-4929-99a2-e1e683ab1f5a"
-					(reference "#PWR058")
+					(reference "#PWR084")
 					(unit 1)
 				)
@@
 		(dnp no)
 		(fields_autoplaced yes)
-		(property "Reference" "R14"
+		(property "Reference" "R30"
 			(at 82.55 45.72 90)
 			(effects
@@
 			(project "Carte-Principale"
 				(path "/88b0dd29-ac24-4c5d-804c-fc642ecf6263/d641269b-1187-4929-99a2-e1e683ab1f5a"
-					(reference "R14")
+					(reference "R30")
 					(unit 1)
 				)
@@
 		(dnp no)
 		(fields_autoplaced yes)
-		(property "Reference" "R17"
+		(property "Reference" "R33"
 			(at 35.56 77.4699 0)
 			(effects
@@
 			(project "Carte-Principale"
 				(path "/88b0dd29-ac24-4c5d-804c-fc642ecf6263/d641269b-1187-4929-99a2-e1e683ab1f5a"
-					(reference "R17")
+					(reference "R33")
 					(unit 1)
 				)
@@
 		(dnp no)
 		(fields_autoplaced yes)
-		(property "Reference" "R12"
+		(property "Reference" "R28"
 			(at 82.55 30.48 90)
 			(effects
@@
 			(project "Carte-Principale"
 				(path "/88b0dd29-ac24-4c5d-804c-fc642ecf6263/d641269b-1187-4929-99a2-e1e683ab1f5a"
-					(reference "R12")
+					(reference "R28")
 					(unit 1)
 				)
@@
 		(dnp no)
 		(fields_autoplaced yes)
-		(property "Reference" "#PWR062"
+		(property "Reference" "#PWR088"
 			(at 138.43 67.31 0)
 			(effects
@@
 			(project "Carte-Principale"
 				(path "/88b0dd29-ac24-4c5d-804c-fc642ecf6263/d641269b-1187-4929-99a2-e1e683ab1f5a"
-					(reference "#PWR062")
+					(reference "#PWR088")
 					(unit 1)
 				)
@@
 		(dnp no)
 		(fields_autoplaced yes)
-		(property "Reference" "#PWR055"
+		(property "Reference" "#PWR081"
 			(at 53.34 35.56 0)
 			(effects
@@
 			(project "Carte-Principale"
 				(path "/88b0dd29-ac24-4c5d-804c-fc642ecf6263/d641269b-1187-4929-99a2-e1e683ab1f5a"
-					(reference "#PWR055")
+					(reference "#PWR081")
 					(unit 1)
 				)
@@
 		(dnp no)
 		(fields_autoplaced yes)
-		(property "Reference" "R16"
+		(property "Reference" "R32"
 			(at 82.55 60.96 90)
 			(effects
@@
 			(project "Carte-Principale"
 				(path "/88b0dd29-ac24-4c5d-804c-fc642ecf6263/d641269b-1187-4929-99a2-e1e683ab1f5a"
-					(reference "R16")
+					(reference "R32")
 					(unit 1)
 				)
@@
 		(dnp no)
 		(fields_autoplaced yes)
-		(property "Reference" "R18"
+		(property "Reference" "R34"
 			(at 82.55 76.2 90)
 			(effects
@@
 			(project "Carte-Principale"
 				(path "/88b0dd29-ac24-4c5d-804c-fc642ecf6263/d641269b-1187-4929-99a2-e1e683ab1f5a"
-					(reference "R18")
+					(reference "R34")
 					(unit 1)
 				)
@@
 		(dnp no)
 		(fields_autoplaced yes)
-		(property "Reference" "R13"
+		(property "Reference" "R29"
 			(at 35.56 46.9899 0)
 			(effects
@@
 			(project "Carte-Principale"
 				(path "/88b0dd29-ac24-4c5d-804c-fc642ecf6263/d641269b-1187-4929-99a2-e1e683ab1f5a"
-					(reference "R13")
+					(reference "R29")
 					(unit 1)
 				)
@@
 		(dnp no)
 		(fields_autoplaced yes)
-		(property "Reference" "SW3"
+		(property "Reference" "SW2"
 			(at 66.04 60.96 0)
 			(effects
@@
 			(project "Carte-Principale"
 				(path "/88b0dd29-ac24-4c5d-804c-fc642ecf6263/d641269b-1187-4929-99a2-e1e683ab1f5a"
-					(reference "SW3")
+					(reference "SW2")
 					(unit 1)
 				)
@@
 		(dnp no)
 		(fields_autoplaced yes)
-		(property "Reference" "#PWR059"
+		(property "Reference" "#PWR085"
 			(at 148.59 52.07 0)
 			(effects
@@
 			(project "Carte-Principale"
 				(path "/88b0dd29-ac24-4c5d-804c-fc642ecf6263/d641269b-1187-4929-99a2-e1e683ab1f5a"
-					(reference "#PWR059")
+					(reference "#PWR085")
 					(unit 1)
 				)
@@
 		(on_board yes)
 		(dnp no)
-		(property "Reference" "#PWR056"
+		(property "Reference" "#PWR082"
 			(at 33.02 45.72 0)
 			(effects
@@
 			(project "Carte-Principale"
 				(path "/88b0dd29-ac24-4c5d-804c-fc642ecf6263/d641269b-1187-4929-99a2-e1e683ab1f5a"
-					(reference "#PWR056")
+					(reference "#PWR082")
 					(unit 1)
 				)
@@
 		(on_board yes)
 		(dnp no)
-		(property "Reference" "#PWR065"
+		(property "Reference" "#PWR091"
 			(at 33.02 91.44 0)
 			(effects
@@
 			(project "Carte-Principale"
 				(path "/88b0dd29-ac24-4c5d-804c-fc642ecf6263/d641269b-1187-4929-99a2-e1e683ab1f5a"
-					(reference "#PWR065")
+					(reference "#PWR091")
 					(unit 1)
 				)
@@
 		(dnp no)
 		(fields_autoplaced yes)
-		(property "Reference" "J19"
+		(property "Reference" "J15"
 			(at 173.355 59.69 0)
 			(effects
@@
 			(project "Carte-Principale"
 				(path "/88b0dd29-ac24-4c5d-804c-fc642ecf6263/d641269b-1187-4929-99a2-e1e683ab1f5a"
-					(reference "J19")
+					(reference "J15")
 					(unit 1)
 				)
@@
 		(dnp no)
 		(fields_autoplaced yes)
-		(property "Reference" "J18"
+		(property "Reference" "J14"
 			(at 132.715 44.45 0)
 			(effects
@@
 			(project "Carte-Principale"
 				(path "/88b0dd29-ac24-4c5d-804c-fc642ecf6263/d641269b-1187-4929-99a2-e1e683ab1f5a"
-					(reference "J18")
+					(reference "J14")
 					(unit 1)
 				)
@@
 		(dnp no)
 		(fields_autoplaced yes)
-		(property "Reference" "#PWR057"
+		(property "Reference" "#PWR083"
 			(at 138.43 49.53 0)
 			(effects
@@
 			(project "Carte-Principale"
 				(path "/88b0dd29-ac24-4c5d-804c-fc642ecf6263/d641269b-1187-4929-99a2-e1e683ab1f5a"
-					(reference "#PWR057")
+					(reference "#PWR083")
 					(unit 1)
 				)
@@
 		(dnp no)
 		(fields_autoplaced yes)
-		(property "Reference" "#PWR064"
+		(property "Reference" "#PWR090"
 			(at 53.34 81.28 0)
 			(effects
@@
 			(project "Carte-Principale"
 				(path "/88b0dd29-ac24-4c5d-804c-fc642ecf6263/d641269b-1187-4929-99a2-e1e683ab1f5a"
-					(reference "#PWR064")
+					(reference "#PWR090")
 					(unit 1)
 				)
@@
 		(on_board yes)
 		(dnp no)
-		(property "Reference" "#PWR060"
+		(property "Reference" "#PWR086"
 			(at 33.02 60.96 0)
 			(effects
@@
 			(project "Carte-Principale"
 				(path "/88b0dd29-ac24-4c5d-804c-fc642ecf6263/d641269b-1187-4929-99a2-e1e683ab1f5a"
-					(reference "#PWR060")
+					(reference "#PWR086")
 					(unit 1)
 				)
@@
 		(dnp no)
 		(fields_autoplaced yes)
-		(property "Reference" "R11"
+		(property "Reference" "R27"
 			(at 35.56 31.7499 0)
 			(effects
@@
 			(project "Carte-Principale"
 				(path "/88b0dd29-ac24-4c5d-804c-fc642ecf6263/d641269b-1187-4929-99a2-e1e683ab1f5a"
-					(reference "R11")
+					(reference "R27")
 					(unit 1)
 				)
@@
 		(dnp no)
 		(fields_autoplaced yes)
-		(property "Reference" "SW5"
+		(property "Reference" "SW4"
 			(at 66.04 91.44 0)
 			(effects
@@
 			(project "Carte-Principale"
 				(path "/88b0dd29-ac24-4c5d-804c-fc642ecf6263/d641269b-1187-4929-99a2-e1e683ab1f5a"
-					(reference "SW5")
+					(reference "SW4")
 					(unit 1)
 				)
@@
 		(dnp no)
 		(fields_autoplaced yes)
-		(property "Reference" "SW4"
+		(property "Reference" "SW3"
 			(at 66.04 76.2 0)
 			(effects
@@
 			(project "Carte-Principale"
 				(path "/88b0dd29-ac24-4c5d-804c-fc642ecf6263/d641269b-1187-4929-99a2-e1e683ab1f5a"
-					(reference "SW4")
+					(reference "SW3")
 					(unit 1)
 				)
@@
 		(dnp no)
 		(fields_autoplaced yes)
-		(property "Reference" "#PWR061"
+		(property "Reference" "#PWR087"
 			(at 53.34 66.04 0)
 			(effects
@@
 			(project "Carte-Principale"
 				(path "/88b0dd29-ac24-4c5d-804c-fc642ecf6263/d641269b-1187-4929-99a2-e1e683ab1f5a"
-					(reference "#PWR061")
+					(reference "#PWR087")
 					(unit 1)
 				)
@@
 		(dnp no)
 		(fields_autoplaced yes)
-		(property "Reference" "SW2"
+		(property "Reference" "SW1"
 			(at 66.04 45.72 0)
 			(effects
@@
 			(project "Carte-Principale"
 				(path "/88b0dd29-ac24-4c5d-804c-fc642ecf6263/d641269b-1187-4929-99a2-e1e683ab1f5a"
-					(reference "SW2")
+					(reference "SW1")
 					(unit 1)
 				)
@@
 		(on_board yes)
 		(dnp no)
-		(property "Reference" "#PWR063"
+		(property "Reference" "#PWR089"
 			(at 33.02 76.2 0)
 			(effects
@@
 			(project "Carte-Principale"
 				(path "/88b0dd29-ac24-4c5d-804c-fc642ecf6263/d641269b-1187-4929-99a2-e1e683ab1f5a"
-					(reference "#PWR063")
+					(reference "#PWR089")
 					(unit 1)
 				)
@@
 		(dnp no)
 		(fields_autoplaced yes)
-		(property "Reference" "R15"
+		(property "Reference" "R31"
 			(at 35.56 62.2299 0)
 			(effects
@@
 			(project "Carte-Principale"
 				(path "/88b0dd29-ac24-4c5d-804c-fc642ecf6263/d641269b-1187-4929-99a2-e1e683ab1f5a"
-					(reference "R15")
+					(reference "R31")
 					(unit 1)
 				)
@@
 		(dnp no)
 		(fields_autoplaced yes)
-		(property "Reference" "#PWR054"
+		(property "Reference" "#PWR080"
 			(at 87.63 33.02 0)
 			(effects
@@
 			(project "Carte-Principale"
 				(path "/88b0dd29-ac24-4c5d-804c-fc642ecf6263/d641269b-1187-4929-99a2-e1e683ab1f5a"
-					(reference "#PWR054")
-					(unit 1)
-				)
+					(reference "#PWR080")
+					(unit 1)
+				)

Commit message: avancée
Parts:
- renumbered J14 to J21, J15 to J22, Q3 to Q2, Q2 to Q3, R31 to R10, R29 to R11, R33 to R12, R32 to R31, R30 to R32, R28 to R33, R27 to R9, SW3 to SW1, SW4 to SW2, SW2 to SW3, SW1 to SW4
Changed lines of the file:
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@@
 		(dnp no)
 		(fields_autoplaced yes)
-		(property "Reference" "R30"
+		(property "Reference" "R32"
 			(at 82.55 45.72 90)
 			(effects
@@
 			(project "Carte-Principale"
 				(path "/88b0dd29-ac24-4c5d-804c-fc642ecf6263/d641269b-1187-4929-99a2-e1e683ab1f5a"
-					(reference "R30")
+					(reference "R32")
 					(unit 1)
 				)
@@
 		(on_board yes)
 		(dnp no)
-		(property "Reference" "Q3"
+		(property "Reference" "Q2"
 			(at 41.91 57.15 90)
 			(effects
@@
 			(project "Carte-Principale"
 				(path "/88b0dd29-ac24-4c5d-804c-fc642ecf6263/d641269b-1187-4929-99a2-e1e683ab1f5a"
-					(reference "Q3")
+					(reference "Q2")
 					(unit 1)
 				)
@@
 		(dnp no)
 		(fields_autoplaced yes)
-		(property "Reference" "R33"
+		(property "Reference" "R12"
 			(at 35.56 77.4699 0)
 			(effects
@@
 			(project "Carte-Principale"
 				(path "/88b0dd29-ac24-4c5d-804c-fc642ecf6263/d641269b-1187-4929-99a2-e1e683ab1f5a"
-					(reference "R33")
+					(reference "R12")
 					(unit 1)
 				)
@@
 		(dnp no)
 		(fields_autoplaced yes)
-		(property "Reference" "R28"
+		(property "Reference" "R33"
 			(at 82.55 30.48 90)
 			(effects
@@
 			(project "Carte-Principale"
 				(path "/88b0dd29-ac24-4c5d-804c-fc642ecf6263/d641269b-1187-4929-99a2-e1e683ab1f5a"
-					(reference "R28")
+					(reference "R33")
 					(unit 1)
 				)
@@
 		(dnp no)
 		(fields_autoplaced yes)
-		(property "Reference" "R32"
+		(property "Reference" "R31"
 			(at 82.55 60.96 90)
 			(effects
@@
 			(project "Carte-Principale"
 				(path "/88b0dd29-ac24-4c5d-804c-fc642ecf6263/d641269b-1187-4929-99a2-e1e683ab1f5a"
-					(reference "R32")
+					(reference "R31")
 					(unit 1)
 				)
@@
 		(dnp no)
 		(fields_autoplaced yes)
-		(property "Reference" "R29"
+		(property "Reference" "R11"
 			(at 35.56 46.9899 0)
 			(effects
@@
 			(project "Carte-Principale"
 				(path "/88b0dd29-ac24-4c5d-804c-fc642ecf6263/d641269b-1187-4929-99a2-e1e683ab1f5a"
-					(reference "R29")
+					(reference "R11")
 					(unit 1)
 				)
@@
 		(dnp no)
 		(fields_autoplaced yes)
-		(property "Reference" "SW2"
+		(property "Reference" "SW3"
 			(at 66.04 60.96 0)
 			(effects
@@
 			(project "Carte-Principale"
 				(path "/88b0dd29-ac24-4c5d-804c-fc642ecf6263/d641269b-1187-4929-99a2-e1e683ab1f5a"
-					(reference "SW2")
+					(reference "SW3")
 					(unit 1)
 				)
@@
 		(dnp no)
 		(fields_autoplaced yes)
-		(property "Reference" "J15"
+		(property "Reference" "J22"
 			(at 173.355 59.69 0)
 			(effects
@@
 			(project "Carte-Principale"
 				(path "/88b0dd29-ac24-4c5d-804c-fc642ecf6263/d641269b-1187-4929-99a2-e1e683ab1f5a"
-					(reference "J15")
+					(reference "J22")
 					(unit 1)
 				)
@@
 		(dnp no)
 		(fields_autoplaced yes)
-		(property "Reference" "J14"
+		(property "Reference" "J21"
 			(at 132.715 44.45 0)
 			(effects
@@
 			(project "Carte-Principale"
 				(path "/88b0dd29-ac24-4c5d-804c-fc642ecf6263/d641269b-1187-4929-99a2-e1e683ab1f5a"
-					(reference "J14")
+					(reference "J21")
 					(unit 1)
 				)
@@
 		(dnp no)
 		(fields_autoplaced yes)
-		(property "Reference" "R27"
+		(property "Reference" "R9"
 			(at 35.56 31.7499 0)
 			(effects
@@
 			(project "Carte-Principale"
 				(path "/88b0dd29-ac24-4c5d-804c-fc642ecf6263/d641269b-1187-4929-99a2-e1e683ab1f5a"
-					(reference "R27")
+					(reference "R9")
 					(unit 1)
 				)
@@
 		(dnp no)
 		(fields_autoplaced yes)
-		(property "Reference" "SW4"
+		(property "Reference" "SW2"
 			(at 66.04 91.44 0)
 			(effects
@@
 			(project "Carte-Principale"
 				(path "/88b0dd29-ac24-4c5d-804c-fc642ecf6263/d641269b-1187-4929-99a2-e1e683ab1f5a"
-					(reference "SW4")
+					(reference "SW2")
 					(unit 1)
 				)
@@
 		(dnp no)
 		(fields_autoplaced yes)
-		(property "Reference" "SW3"
+		(property "Reference" "SW1"
 			(at 66.04 76.2 0)
 			(effects
@@
 			(project "Carte-Principale"
 				(path "/88b0dd29-ac24-4c5d-804c-fc642ecf6263/d641269b-1187-4929-99a2-e1e683ab1f5a"
-					(reference "SW3")
+					(reference "SW1")
 					(unit 1)
 				)
@@
 		(dnp no)
 		(fields_autoplaced yes)
-		(property "Reference" "SW1"
+		(property "Reference" "SW4"
 			(at 66.04 45.72 0)
 			(effects
@@
 			(project "Carte-Principale"
 				(path "/88b0dd29-ac24-4c5d-804c-fc642ecf6263/d641269b-1187-4929-99a2-e1e683ab1f5a"
-					(reference "SW1")
+					(reference "SW4")
 					(unit 1)
 				)
@@
 		(on_board yes)
 		(dnp no)
-		(property "Reference" "Q2"
+		(property "Reference" "Q3"
 			(at 41.91 41.91 90)
 			(effects
@@
 			(project "Carte-Principale"
 				(path "/88b0dd29-ac24-4c5d-804c-fc642ecf6263/d641269b-1187-4929-99a2-e1e683ab1f5a"
-					(reference "Q2")
+					(reference "Q3")
 					(unit 1)
 				)
@@
 		(dnp no)
 		(fields_autoplaced yes)
-		(property "Reference" "R31"
+		(property "Reference" "R10"
 			(at 35.56 62.2299 0)
 			(effects
@@
 			(project "Carte-Principale"
 				(path "/88b0dd29-ac24-4c5d-804c-fc642ecf6263/d641269b-1187-4929-99a2-e1e683ab1f5a"
-					(reference "R31")
-					(unit 1)
-				)
+					(reference "R10")
+					(unit 1)
+				)

Commit message: Final pcb modification
Parts:
- renumbered J21 to J16, J22 to J17, Q3 to Q2, Q2 to Q3, R11 to R10, R9 to R11, R10 to R9, SW2 to SW1, SW1 to SW2
Changed lines of the file:
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@@
 		(on_board yes)
 		(dnp no)
-		(property "Reference" "Q2"
+		(property "Reference" "Q3"
 			(at 41.91 57.15 90)
 			(effects
@@
 			(project "Carte-Principale"
 				(path "/88b0dd29-ac24-4c5d-804c-fc642ecf6263/d641269b-1187-4929-99a2-e1e683ab1f5a"
-					(reference "Q2")
+					(reference "Q3")
 					(unit 1)
 				)
@@
 		(dnp no)
 		(fields_autoplaced yes)
-		(property "Reference" "R11"
+		(property "Reference" "R10"
 			(at 35.56 46.9899 0)
 			(effects
@@
 			(project "Carte-Principale"
 				(path "/88b0dd29-ac24-4c5d-804c-fc642ecf6263/d641269b-1187-4929-99a2-e1e683ab1f5a"
-					(reference "R11")
+					(reference "R10")
 					(unit 1)
 				)
@@
 		(dnp no)
 		(fields_autoplaced yes)
-		(property "Reference" "J22"
+		(property "Reference" "J17"
 			(at 173.355 59.69 0)
 			(effects
@@
 			(project "Carte-Principale"
 				(path "/88b0dd29-ac24-4c5d-804c-fc642ecf6263/d641269b-1187-4929-99a2-e1e683ab1f5a"
-					(reference "J22")
+					(reference "J17")
 					(unit 1)
 				)
@@
 		(dnp no)
 		(fields_autoplaced yes)
-		(property "Reference" "J21"
+		(property "Reference" "J16"
 			(at 132.715 44.45 0)
 			(effects
@@
 			(project "Carte-Principale"
 				(path "/88b0dd29-ac24-4c5d-804c-fc642ecf6263/d641269b-1187-4929-99a2-e1e683ab1f5a"
-					(reference "J21")
+					(reference "J16")
 					(unit 1)
 				)
@@
 		(dnp no)
 		(fields_autoplaced yes)
-		(property "Reference" "R9"
+		(property "Reference" "R11"
 			(at 35.56 31.7499 0)
 			(effects
@@
 			(project "Carte-Principale"
 				(path "/88b0dd29-ac24-4c5d-804c-fc642ecf6263/d641269b-1187-4929-99a2-e1e683ab1f5a"
-					(reference "R9")
+					(reference "R11")
 					(unit 1)
 				)
@@
 		(dnp no)
 		(fields_autoplaced yes)
-		(property "Reference" "SW2"
+		(property "Reference" "SW1"
 			(at 66.04 91.44 0)
 			(effects
@@
 			(project "Carte-Principale"
 				(path "/88b0dd29-ac24-4c5d-804c-fc642ecf6263/d641269b-1187-4929-99a2-e1e683ab1f5a"
-					(reference "SW2")
+					(reference "SW1")
 					(unit 1)
 				)
@@
 		(dnp no)
 		(fields_autoplaced yes)
-		(property "Reference" "SW1"
+		(property "Reference" "SW2"
 			(at 66.04 76.2 0)
 			(effects
@@
 			(project "Carte-Principale"
 				(path "/88b0dd29-ac24-4c5d-804c-fc642ecf6263/d641269b-1187-4929-99a2-e1e683ab1f5a"
-					(reference "SW1")
+					(reference "SW2")
 					(unit 1)
 				)
@@
 		(on_board yes)
 		(dnp no)
-		(property "Reference" "Q3"
+		(property "Reference" "Q2"
 			(at 41.91 41.91 90)
 			(effects
@@
 			(project "Carte-Principale"
 				(path "/88b0dd29-ac24-4c5d-804c-fc642ecf6263/d641269b-1187-4929-99a2-e1e683ab1f5a"
-					(reference "Q3")
+					(reference "Q2")
 					(unit 1)
 				)
@@
 		(dnp no)
 		(fields_autoplaced yes)
-		(property "Reference" "R10"
+		(property "Reference" "R9"
 			(at 35.56 62.2299 0)
 			(effects
@@
 			(project "Carte-Principale"
 				(path "/88b0dd29-ac24-4c5d-804c-fc642ecf6263/d641269b-1187-4929-99a2-e1e683ab1f5a"
-					(reference "R10")
-					(unit 1)
-				)
+					(reference "R9")
+					(unit 1)
+				)

Commit message: Cartes élec à refaire et TODO
Parts:
- removed J16: LCD_TFT, Connector_PinSocket_2.54mm:PinSocket_1x14_P2.54mm_Vertical, symbol Connector:Conn_01x14_Pin
- removed J17: LCD_SD, Connector_PinSocket_2.54mm:PinSocket_1x04_P2.54mm_Vertical, symbol Connector:Conn_01x04_Pin
- SW1, SW2, SW3, SW4: footprint Connector_Molex:Molex_KK-254_AE-6410-04A_1x04_P2.54mm_Vertical -> Connector_JST:JST_XH_B4B-XH-A_1x04_P2.50mm_Vertical
