File: Carte-Principale/interface.kicad_sch (KiCad schematic)
At the start: 16 parts, among them Q2 BSS138, Q3 BSS138, Q4 BSS138, Q5 BSS138, SW1 Rouge, SW2 Bleu, SW3 Jaune, SW4 Vert

Commit message: FInal
Parts:
- added BZ1: Buzzer, Buzzer_Beeper:Buzzer_12x9.5RM7.6, symbol Device:Buzzer
- added J21: I2C Screen, Connector_JST:JST_XH_B4B-XH-A_1x04_P2.50mm_Vertical, symbol Connector:Conn_01x04_Pin
- added Q1: BC817, Package_TO_SOT_SMD:SOT-23, symbol Transistor_BJT:BC817
- added R2: R, Resistor_SMD:R_1206_3216Metric_Pad1.30x1.75mm_HandSolder, symbol Device:R
Connections:
- net +5V: now also BZ1.1 (+), J21.1 (Pin_1)
- net GND: now also J21.4 (Pin_4), Q1.2 (E)
- new net: BZ1.2 (-), Q1.3 (C)
- new net: Q1.1 (B), R2.2
- new net Buzzer: R2.1
- new net LCD_SCK: J21.3 (Pin_3)
- new net LCD_SDA: J21.2 (Pin_2)

Commit message: abcdefgh
Parts:
- R2: footprint Resistor_SMD:R_1206_3216Metric_Pad1.30x1.75mm_HandSolder -> Resistor_SMD:R_1210_3225Metric_Pad1.30x2.65mm_HandSolder
Other:
- company: CRINSA -> CRINSA - Boris HILKENS
Changed lines of the file:
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@@
 	(title_block
 		(title "Carte Principale")
-		(date "2024-08-12")
-		(company "CRINSA")
+		(date "2024-12-27")
+		(rev "V1")
+		(company "CRINSA - Boris HILKENS")
 		(comment 1 "Carte de contrôle pour le robot")
 	)
@@
 			)
 		)
-		(property "Footprint" "Resistor_SMD:R_1206_3216Metric_Pad1.30x1.75mm_HandSolder"
+		(property "Footprint" "Resistor_SMD:R_1210_3225Metric_Pad1.30x2.65mm_HandSolder"
 			(at 132.08 42.418 90)
 			(effects
