File: Carte-Principale/Carte-Principale.kicad_pcb (KiCad board)
At the start: 2 copper layers, 1 part, among them U1 NUCLEOH723ZG

Commit message: wiring
Parts:
- added C1: 0.1uF, Capacitor_SMD:C_1206_3216Metric_Pad1.33x1.80mm_HandSolder, F.Cu at (123.0, 42.8)
- added C2: 100n, Capacitor_SMD:C_1206_3216Metric_Pad1.33x1.80mm_HandSolder, F.Cu at (159.0, 92.0)
- added C3: 100n, Capacitor_SMD:C_1206_3216Metric_Pad1.33x1.80mm_HandSolder, F.Cu at (159.0, 95.4)
- added C4: 100n, Capacitor_SMD:C_1206_3216Metric_Pad1.33x1.80mm_HandSolder, F.Cu at (159.0, 98.7)
- added C5: 100n, Capacitor_SMD:C_1206_3216Metric_Pad1.33x1.80mm_HandSolder, F.Cu at (159.0, 102.1)
- added D1: 3V3, LED_SMD:LED_2010_5025Metric_Pad1.52x2.65mm_HandSolder, F.Cu at (148.0, 140.0)
- added D2: 5VA, LED_SMD:LED_2010_5025Metric_Pad1.52x2.65mm_HandSolder, F.Cu at (148.0, 144.3)
- added D3: 5V, LED_SMD:LED_2010_5025Metric_Pad1.52x2.65mm_HandSolder, F.Cu at (148.0, 148.6)
- added D4: 12VA, LED_SMD:LED_2010_5025Metric_Pad1.52x2.65mm_HandSolder, F.Cu at (148.0, 152.9)
- added D5: 12V, LED_SMD:LED_2010_5025Metric_Pad1.52x2.65mm_HandSolder, F.Cu at (148.0, 157.2)
- added DRV1: ~, DRV8844:DRV8844_BREAKOUT_BOARD, F.Cu at (141.4, 83.0)
- added J1: 12V, TerminalBlock:TerminalBlock_bornier-2_P5.08mm, F.Cu at (135.8, 142.4)
- added J10: I2C_Sensors, Connector_PinSocket_2.54mm:PinSocket_1x04_P2.54mm_Vertical, F.Cu at (160.8, 110.4)
- added J11: LCD_TFT, Connector_PinSocket_2.54mm:PinSocket_1x14_P2.54mm_Vertical, F.Cu at (134.9, 34.9)
- added J12: LCD_SD, Connector_PinSocket_2.54mm:PinSocket_1x04_P2.54mm_Vertical, F.Cu at (150.3, 47.2)
- added J2: 12VA, TerminalBlock:TerminalBlock_bornier-2_P5.08mm, F.Cu at (135.8, 151.4)
- added J3: 5V, TerminalBlock:TerminalBlock_bornier-2_P5.08mm, F.Cu at (135.8, 160.5)
- added J4: Encodeur_G, Connector_PinHeader_2.54mm:PinHeader_1x08_P2.54mm_Vertical, F.Cu at (134.9, 110.4)
- added J5: Encodeur_D, Connector_PinHeader_2.54mm:PinHeader_1x08_P2.54mm_Vertical, F.Cu at (139.5, 110.4)
- added J6: Moteur_Gauche, TerminalBlock:TerminalBlock_bornier-2_P5.08mm, F.Cu at (153.4, 76.8)
- added J7: Moteur_Droit, TerminalBlock:TerminalBlock_bornier-2_P5.08mm, F.Cu at (153.4, 85.8)
- added J8: PCA9685, Connector_PinSocket_2.54mm:PinSocket_1x03_P2.54mm_Vertical, F.Cu at (165.4, 110.4)
- added J9: AX12, Connector_PinSocket_2.54mm:PinSocket_1x03_P2.54mm_Vertical, F.Cu at (170.0, 110.4)
- added Q2: BSS138, Package_TO_SOT_SMD:SOT-23, F.Cu at (145.6, 47.2)
- added Q3: BSS138, Package_TO_SOT_SMD:SOT-23, F.Cu at (145.6, 51.9)
- added Q4: BSS138, Package_TO_SOT_SMD:SOT-23, F.Cu at (145.6, 56.5)
- added Q5: BSS138, Package_TO_SOT_SMD:SOT-23, F.Cu at (145.6, 61.1)
- added R1: 10K, Resistor_SMD:R_1206_3216Metric_Pad1.30x1.75mm_HandSolder, F.Cu at (154.9, 139.5)
- added R10: 100, Resistor_THT:R_Axial_DIN0207_L6.3mm_D2.5mm_P10.16mm_Horizontal, F.Cu at (143.4, 122.2)
- added R11: 10k, Resistor_SMD:R_1206_3216Metric_Pad1.30x1.75mm_HandSolder, F.Cu at (140.1, 34.2)
- added R12: 10K, Resistor_SMD:R_1206_3216Metric_Pad1.30x1.75mm_HandSolder, F.Cu at (140.1, 37.5)
- added R13: 10k, Resistor_SMD:R_1206_3216Metric_Pad1.30x1.75mm_HandSolder, F.Cu at (140.1, 40.8)
- added R14: 10K, Resistor_SMD:R_1206_3216Metric_Pad1.30x1.75mm_HandSolder, F.Cu at (140.1, 44.1)
- added R15: 10k, Resistor_SMD:R_1206_3216Metric_Pad1.30x1.75mm_HandSolder, F.Cu at (140.1, 47.4)
- added R16: 10K, Resistor_SMD:R_1206_3216Metric_Pad1.30x1.75mm_HandSolder, F.Cu at (140.1, 50.7)
- added R17: 10k, Resistor_SMD:R_1206_3216Metric_Pad1.30x1.75mm_HandSolder, F.Cu at (140.1, 54.0)
- added R18: 10K, Resistor_SMD:R_1206_3216Metric_Pad1.30x1.75mm_HandSolder, F.Cu at (140.1, 57.3)
- added R2: R, Resistor_SMD:R_1206_3216Metric_Pad1.30x1.75mm_HandSolder, F.Cu at (154.9, 142.8)
- added R3: R, Resistor_SMD:R_1206_3216Metric_Pad1.30x1.75mm_HandSolder, F.Cu at (154.9, 146.1)
- added R4: R, Resistor_SMD:R_1206_3216Metric_Pad1.30x1.75mm_HandSolder, F.Cu at (154.9, 149.4)
- added R5: R, Resistor_SMD:R_1206_3216Metric_Pad1.30x1.75mm_HandSolder, F.Cu at (154.9, 152.7)
- added R6: R, Resistor_SMD:R_1206_3216Metric_Pad1.30x1.75mm_HandSolder, F.Cu at (154.9, 156.0)
- added R7: 100, Resistor_THT:R_Axial_DIN0207_L6.3mm_D2.5mm_P10.16mm_Horizontal, F.Cu at (143.4, 110.1)
- added R8: 100, Resistor_THT:R_Axial_DIN0207_L6.3mm_D2.5mm_P10.16mm_Horizontal, F.Cu at (143.4, 114.1)
- added R9: 100, Resistor_THT:R_Axial_DIN0207_L6.3mm_D2.5mm_P10.16mm_Horizontal, F.Cu at (143.4, 118.2)
- added SW1: RESET, Button_Switch_THT:SW_PUSH_6mm, F.Cu at (122.0, 34.6)
- added SW2: Vert, Connector_PinHeader_2.54mm:PinHeader_1x04_P2.54mm_Vertical, F.Cu at (145.4, 34.9)
- added SW3: Jaune, Connector_PinHeader_2.54mm:PinHeader_1x04_P2.54mm_Vertical, F.Cu at (150.1, 34.9)
- added SW4: Bleu, Connector_PinHeader_2.54mm:PinHeader_1x04_P2.54mm_Vertical, F.Cu at (154.7, 34.9)
- added SW5: Rouge, Connector_PinHeader_2.54mm:PinHeader_1x04_P2.54mm_Vertical, F.Cu at (159.4, 34.9)
- added TP1: Test_Gauche, TestPoint:TestPoint_2Pads_Pitch2.54mm_Drill0.8mm, F.Cu at (152.1, 125.9)
- added TP2: Test_Droit, TestPoint:TestPoint_2Pads_Pitch2.54mm_Drill0.8mm, F.Cu at (152.1, 129.3)
- added TP3: Test_PWM, TestPoint:TestPoint_2Pads_Pitch2.54mm_Drill0.8mm, F.Cu at (134.4, 95.4)
- added TP4: Test_DIR, TestPoint:TestPoint_2Pads_Pitch2.54mm_Drill0.8mm, F.Cu at (134.4, 98.7)
- added U2: AM26LV32xD, Package_SO:SOIC-16_3.9x9.9mm_P1.27mm, F.Cu at (146.1, 130.1)
- added U3: 74LVC1G3157, Package_TO_SOT_SMD:SOT-363_SC-70-6_Handsoldering, F.Cu at (153.1, 92.3)
- added U4: 74LVC1G3157, Package_TO_SOT_SMD:SOT-363_SC-70-6_Handsoldering, F.Cu at (153.1, 96.3)
- added U5: 74LVC1G3157, Package_TO_SOT_SMD:SOT-363_SC-70-6_Handsoldering, F.Cu at (153.1, 100.2)
- added U6: 74LVC1G3157, Package_TO_SOT_SMD:SOT-363_SC-70-6_Handsoldering, F.Cu at (153.1, 104.1)
- moved U1 63.1 mm to (84.2, 101.2), turned to 0 degrees
Connections:
- U1 pad CN10_10: unconnected-(U1F-D3/TIMER_A_PWM3-PadCN10_10) -> /PE13
- U1 pad CN10_11: unconnected-(U1F-A8/ADC_C_IN-PadCN10_11) -> /Encodeur_Droit_A
- U1 pad CN10_12: unconnected-(U1F-D2/IO-PadCN10_12) -> /PG14
- U1 pad CN10_13: unconnected-(U1F-D26/QSPI_CS-PadCN10_13) -> /PG6
- U1 pad CN10_14: unconnected-(U1F-D1/USART_A_TX-PadCN10_14) -> /I2C1_SCL
- U1 pad CN10_15: unconnected-(U1F-D27/QSPI_CLK-PadCN10_15) -> /PB2
- U1 pad CN10_16: unconnected-(U1F-D0/USART_A_RX-PadCN10_16) -> /I2C1_SDA
- U1 pad CN10_17: Net-(U1F-GND_CN10-PadCN10_17) -> GND
- U1 pad CN10_18: unconnected-(U1F-D42/TIMER_A_PWM1N-PadCN10_18) -> /PE8
- U1 pad CN10_19: unconnected-(U1F-D28/QSPI_BK1_IO3-PadCN10_19) -> /PD13
- U1 pad CN10_2: unconnected-(U1F-D7/IO-PadCN10_2) -> /PG12
- U1 pad CN10_20: unconnected-(U1F-D41/TIMER_A_ETR-PadCN10_20) -> /PE7
- U1 pad CN10_21: unconnected-(U1F-D29/QSPI_BK1_IO1-PadCN10_21) -> /PD12
- U1 pad CN10_22: Net-(U1F-GND_CN10-PadCN10_17) -> GND
- U1 pad CN10_23: unconnected-(U1F-D30/QSPI_BK1_IO0-PadCN10_23) -> /PD11
- U1 pad CN10_24: unconnected-(U1F-D40/TIMER_A_PWM2N-PadCN10_24) -> /PE10
- U1 pad CN10_25: unconnected-(U1F-D31/QSPI_BK1_IO2-PadCN10_25) -> /PE2
- U1 pad CN10_26: unconnected-(U1F-D39/TIMER_A_PWM3N-PadCN10_26) -> /PE12
- U1 pad CN10_27: Net-(U1F-GND_CN10-PadCN10_17) -> GND
- U1 pad CN10_28: unconnected-(U1F-D38/TIMER_A_BKIN2-PadCN10_28) -> /PE6
- U1 pad CN10_29: unconnected-(U1F-D32/TIMER_C_PWM1-PadCN10_29) -> /PA0
- U1 pad CN10_3: unconnected-(U1F-AGND_CN10-PadCN10_3) -> GND
- U1 pad CN10_30: unconnected-(U1F-D37/TIMER_A_BKIN1-PadCN10_30) -> /PE15
- U1 pad CN10_31: unconnected-(U1F-D33/TIMER_D_PWM1-PadCN10_31) -> /PB0
- U1 pad CN10_32: unconnected-(U1F-D36/TIMER_C_PWM2-PadCN10_32) -> /PB10
- U1 pad CN10_34: unconnected-(U1F-D35/TIMER_C_PWM3-PadCN10_34) -> /PB11
- U1 pad CN10_4: unconnected-(U1F-D6/TIMER_A_PWM1-PadCN10_4) -> /PE9
- U1 pad CN10_5: Net-(U1F-GND_CN10-PadCN10_17) -> GND
- U1 pad CN10_6: unconnected-(U1F-D5/TIMER_A_PWM2-PadCN10_6) -> /PE11
- U1 pad CN10_7: unconnected-(U1F-A6/ADC_A_IN-PadCN10_7) -> /PF4
- U1 pad CN10_8: unconnected-(U1F-D4/IO-PadCN10_8) -> /PE14
- U1 pad CN10_9: unconnected-(U1F-A7/ADC_B_IN-PadCN10_9) -> /PF5
- U1 pad CN7_1: unconnected-(U1E-D16/I2S_A_MCK-PadCN7_1) -> /PC6
- U1 pad CN7_10: unconnected-(U1E-D13/SPI_A_SCK-PadCN7_10) -> /PA5
- U1 pad CN7_11: unconnected-(U1E-D21/I2S_B_MCK-PadCN7_11) -> /PC7
- U1 pad CN7_12: unconnected-(U1E-D12/SPI_A_MISO-PadCN7_12) -> /PA6
- U1 pad CN7_13: unconnected-(U1E-D22/I2S_B_SD/SPI_B_MOSI-PadCN7_13) -> /PB5
- U1 pad CN7_14: unconnected-(U1E-D11/SPI_A_MOSI/TIM_E_PWM1-PadCN7_14) -> /PB5
- U1 pad CN7_15: unconnected-(U1E-D23/I2S_B_CK/SPI_B_SCK-PadCN7_15) -> /PB3
- U1 pad CN7_16: unconnected-(U1E-D10/SPI_A_CS/TIM_B_PWM3-PadCN7_16) -> /PD14
- U1 pad CN7_17: unconnected-(U1E-D24/SPI_B_NSS-PadCN7_17) -> /PA4
- U1 pad CN7_18: unconnected-(U1E-D9/TIMER_B_PWM2-PadCN7_18) -> /PD15
- U1 pad CN7_19: unconnected-(U1E-D25/SPI_B_MISO-PadCN7_19) -> /PB4
- U1 pad CN7_2: unconnected-(U1E-D15/I2C_A_SCL-PadCN7_2) -> /PB8
- U1 pad CN7_20: unconnected-(U1E-D8/IO-PadCN7_20) -> /PF3
- U1 pad CN7_3: unconnected-(U1E-D17/I2S_A_SD-PadCN7_3) -> /PB15
- U1 pad CN7_4: unconnected-(U1E-D14/I2C_A_SDA-PadCN7_4) -> /PB9
- U1 pad CN7_5: unconnected-(U1E-D18/I2S_A_CK-PadCN7_5) -> /PB13
- U1 pad CN7_7: unconnected-(U1E-D19/I2S_A_WS-PadCN7_7) -> /PB12
- U1 pad CN7_8: unconnected-(U1E-GND_CN7-PadCN7_8) -> GND
- U1 pad CN7_9: unconnected-(U1E-D20/I2S_B_WS-PadCN7_9) -> /PA15
- U1 pad CN8_10: unconnected-(U1C-D47/SDMMC_CK-PadCN8_10) -> /PC12
- U1 pad CN8_11: Net-(U1C-GND_CN8-PadCN8_11) -> GND
- U1 pad CN8_12: unconnected-(U1C-D48/SDMMC_CMD-PadCN8_12) -> /PD2
- U1 pad CN8_13: Net-(U1C-GND_CN8-PadCN8_11) -> GND
- U1 pad CN8_14: unconnected-(U1C-D49/IO-PadCN8_14) -> /PF2
- U1 pad CN8_16: unconnected-(U1C-D50/IO-PadCN8_16) -> /PG3
- U1 pad CN8_2: unconnected-(U1C-D43/SDMMC_D0-PadCN8_2) -> /PC8
- U1 pad CN8_4: unconnected-(U1C-D44/SDMMC_D1/I2S_A_CKIN-PadCN8_4) -> /I2C3_SDA
- U1 pad CN8_5: unconnected-(U1C-NRST_CN8-PadCN8_5) -> /NRST
- U1 pad CN8_6: unconnected-(U1C-D45/SDMMC_D2-PadCN8_6) -> /PC10
- U1 pad CN8_7: unconnected-(U1C-3V3_CN8-PadCN8_7) -> +3V3
- U1 pad CN8_8: unconnected-(U1C-D46/SDMMC_D3-PadCN8_8) -> /PC11
- U1 pad CN9_1: unconnected-(U1D-A0/ADC12_INP15-PadCN9_1) -> /AX12_RX
- U1 pad CN9_10: unconnected-(U1D-D55/USART_B_CTS-PadCN9_10) -> /PD3
- U1 pad CN9_11: unconnected-(U1D-A5/ADC3_INP6/I2C1_SCL-PadCN9_11) -> /PF10
- U1 pad CN9_12: Net-(U1D-GND_CN9-PadCN9_12) -> GND
- U1 pad CN9_13: unconnected-(U1D-D72/COMP1_INP-PadCN9_13) -> /PB2
- U1 pad CN9_14: unconnected-(U1D-D56/SAI_A_MCLK-PadCN9_14) -> /PE2
- U1 pad CN9_15: unconnected-(U1D-D71/COMP2_INP-PadCN9_15) -> /PE9
- U1 pad CN9_16: unconnected-(U1D-D57/SAI_A_FS-PadCN9_16) -> /PE4
- U1 pad CN9_17: unconnected-(U1D-D70/I2C_B_SMBA-PadCN9_17) -> /PF2
- U1 pad CN9_18: unconnected-(U1D-D58/SAI_A_SCK-PadCN9_18) -> /PE5
- U1 pad CN9_19: unconnected-(U1D-D69/I2C_B_SCL-PadCN9_19) -> /I2C2_SCL
- U1 pad CN9_2: unconnected-(U1D-D51/USART_B_SCLK-PadCN9_2) -> /PD7
- U1 pad CN9_20: unconnected-(U1D-D59/SAI_A_SD-PadCN9_20) -> /PE6
- U1 pad CN9_21: unconnected-(U1D-D68/I2C_B_SDA-PadCN9_21) -> /I2C2_SDA
- U1 pad CN9_22: unconnected-(U1D-D60/SAI_B_SD-PadCN9_22) -> /PE3
- U1 pad CN9_23: Net-(U1D-GND_CN9-PadCN9_12) -> GND
- U1 pad CN9_24: unconnected-(U1D-D61/SAI_B_SCK-PadCN9_24) -> /PF8
- U1 pad CN9_25: unconnected-(U1D-D67/CAN_RX-PadCN9_25) -> /PD0
- U1 pad CN9_26: unconnected-(U1D-D62/SAI_B_MCLK-PadCN9_26) -> /Encodeur_Droit_B
- U1 pad CN9_27: unconnected-(U1D-D66/CAN_TX-PadCN9_27) -> /PD1
- U1 pad CN9_28: unconnected-(U1D-D63/SAI_B_FS-PadCN9_28) -> /PF9
- U1 pad CN9_29: unconnected-(U1D-D65/IO-PadCN9_29) -> /PG0
- U1 pad CN9_3: unconnected-(U1D-A1/ADC123_INP10-PadCN9_3) -> /PC0
- U1 pad CN9_30: unconnected-(U1D-D64/IO-PadCN9_30) -> /PG1
- U1 pad CN9_4: unconnected-(U1D-D52/USART_B_RX-PadCN9_4) -> /PD6
- U1 pad CN9_5: unconnected-(U1D-A2/ADC12_INP13-PadCN9_5) -> /PC3
- U1 pad CN9_6: unconnected-(U1D-D53/USART_B_TX-PadCN9_6) -> /AX12_RX
- U1 pad CN9_7: unconnected-(U1D-A3/ADC12_INP5-PadCN9_7) -> /PB1
- U1 pad CN9_8: unconnected-(U1D-D54/USART_B_RTS-PadCN9_8) -> /PD4
- U1 pad CN9_9: unconnected-(U1D-A4/ADC123_INP12/I2C1_SDA-PadCN9_9) -> /PC2

Commit message: Schéma vérifié
Parts:
- added F1: 1.3A, Fuse:Fuse_2010_5025Metric_Pad1.52x2.65mm_HandSolder, F.Cu at (218.4, 46.7)
- added F2: 2A, Fuse:Fuse_2010_5025Metric_Pad1.52x2.65mm_HandSolder, F.Cu at (210.4, 86.4)
- added F3: 5A, Fuse:Fuse_2010_5025Metric_Pad1.52x2.65mm_HandSolder, F.Cu at (210.4, 90.6)
- added F4: 5A, Fuse:Fuse_2010_5025Metric_Pad1.52x2.65mm_HandSolder, F.Cu at (210.4, 94.8)
- added H1: MountingHole, MountingHole:MountingHole_3.2mm_M3, F.Cu at (210.5, 48.5)
- added H2: MountingHole, MountingHole:MountingHole_3.2mm_M3, F.Cu at (210.5, 56.5)
- added H3: MountingHole, MountingHole:MountingHole_3.2mm_M3, F.Cu at (210.5, 64.4)
- added H4: MountingHole, MountingHole:MountingHole_3.2mm_M3, F.Cu at (210.5, 72.4)
- added J13: Moteur_Gauche, TerminalBlock:TerminalBlock_bornier-2_P5.08mm, F.Cu at (227.5, 49.1)
- added J14: Moteur_Droit, TerminalBlock:TerminalBlock_bornier-2_P5.08mm, F.Cu at (227.5, 58.1)
- added J15: PCA9685, Connector_Molex:Molex_KK-254_AE-6410-06A_1x06_P2.54mm_Vertical, F.Cu at (226.6, 68.6)
- added J16: AX12, Connector_Molex:Molex_KK-254_AE-6410-03A_1x03_P2.54mm_Vertical, F.Cu at (238.8, 76.5)
- added J17: I2C_Sensors, Connector_Molex:Molex_KK-254_AE-6410-04A_1x04_P2.54mm_Vertical, F.Cu at (226.6, 76.5)
- added J18: LCD_TFT, Connector_PinSocket_2.54mm:PinSocket_1x14_P2.54mm_Vertical, F.Cu at (197.7, 46.9)
- added J19: LCD_SD, Connector_PinSocket_2.54mm:PinSocket_1x04_P2.54mm_Vertical, F.Cu at (202.3, 46.9)
- added Q1: IRF630, Package_TO_SOT_THT:TO-220-3_Vertical, F.Cu at (209.8, 82.3)
- added TP10: Test_DIR, TestPoint:TestPoint_2Pads_Pitch2.54mm_Drill0.8mm, F.Cu at (237.6, 49.6)
- added TP5: 12VA, Connector_Pin:Pin_D1.0mm_L10.0mm, F.Cu at (216.3, 86.3)
- added TP6: 12V, Connector_Pin:Pin_D1.0mm_L10.0mm, F.Cu at (216.3, 90.4)
- added TP7: Test_Gauche, TestPoint:TestPoint_2Pads_Pitch2.54mm_Drill0.8mm, F.Cu at (226.1, 84.0)
- added TP8: Test_Droit, TestPoint:TestPoint_2Pads_Pitch2.54mm_Drill0.8mm, F.Cu at (226.1, 87.4)
- added TP9: Test_PWM, TestPoint:TestPoint_2Pads_Pitch2.54mm_Drill0.8mm, F.Cu at (237.6, 46.2)
- C1, C2, C3, C4, C5: footprint Capacitor_SMD:C_1206_3216Metric_Pad1.33x1.80mm_HandSolder -> Capacitor_SMD:C_1210_3225Metric_Pad1.33x2.70mm_HandSolder
- J1: value 12V -> Serial; footprint TerminalBlock:TerminalBlock_bornier-2_P5.08mm -> Connector_Molex:Molex_KK-254_AE-6410-03A_1x03_P2.54mm_Vertical
- J10: value I2C_Sensors -> 5V; footprint Connector_PinSocket_2.54mm:PinSocket_1x04_P2.54mm_Vertical -> Connector_AMASS:AMASS_XT30U-M_1x02_P5.0mm_Vertical
- J11: value LCD_TFT -> Encodeur_G; footprint Connector_PinSocket_2.54mm:PinSocket_1x14_P2.54mm_Vertical -> Connector_PinHeader_2.54mm:PinHeader_1x08_P2.54mm_Vertical
- J12: value LCD_SD -> Encodeur_D; footprint Connector_PinSocket_2.54mm:PinSocket_1x04_P2.54mm_Vertical -> Connector_PinHeader_2.54mm:PinHeader_1x08_P2.54mm_Vertical
- J2: value 12VA -> PA; footprint TerminalBlock:TerminalBlock_bornier-2_P5.08mm -> Connector_Molex:Molex_KK-254_AE-6410-05A_1x05_P2.54mm_Vertical
- J3: value 5V -> PG; footprint TerminalBlock:TerminalBlock_bornier-2_P5.08mm -> Connector_Molex:Molex_KK-254_AE-6410-08A_1x08_P2.54mm_Vertical
- J4: value Encodeur_G -> SPI2; footprint Connector_PinHeader_2.54mm:PinHeader_1x08_P2.54mm_Vertical -> Connector_Molex:Molex_KK-254_AE-6410-04A_1x04_P2.54mm_Vertical
- J5: value Encodeur_D -> SPI3; footprint Connector_PinHeader_2.54mm:PinHeader_1x08_P2.54mm_Vertical -> Connector_Molex:Molex_KK-254_AE-6410-04A_1x04_P2.54mm_Vertical
- J6: value Moteur_Gauche -> I2C2; footprint TerminalBlock:TerminalBlock_bornier-2_P5.08mm -> Connector_Molex:Molex_KK-254_AE-6410-03A_1x03_P2.54mm_Vertical
- J7: value Moteur_Droit -> I2C3; footprint TerminalBlock:TerminalBlock_bornier-2_P5.08mm -> Connector_Molex:Molex_KK-254_AE-6410-03A_1x03_P2.54mm_Vertical
- J8: value PCA9685 -> 12V; footprint Connector_PinSocket_2.54mm:PinSocket_1x03_P2.54mm_Vertical -> Connector_AMASS:AMASS_XT60-M_1x02_P7.20mm_Vertical
- J9: value AX12 -> 12VA; footprint Connector_PinSocket_2.54mm:PinSocket_1x03_P2.54mm_Vertical -> Connector_AMASS:AMASS_XT60-M_1x02_P7.20mm_Vertical
- R1, R11, R12, R13, R14, R15, R16, R17, R18, R2, R3, R4, R5, R6: footprint Resistor_SMD:R_1206_3216Metric_Pad1.30x1.75mm_HandSolder -> Resistor_SMD:R_1210_3225Metric_Pad1.30x2.65mm_HandSolder
- SW2, SW3, SW4, SW5: footprint Connector_PinHeader_2.54mm:PinHeader_1x04_P2.54mm_Vertical -> Connector_Molex:Molex_KK-254_AE-6410-04A_1x04_P2.54mm_Vertical
- TP1: value Test_Gauche -> GND; footprint TestPoint:TestPoint_2Pads_Pitch2.54mm_Drill0.8mm -> Connector_Pin:Pin_D1.0mm_L10.0mm
- TP2: value Test_Droit -> 3V3; footprint TestPoint:TestPoint_2Pads_Pitch2.54mm_Drill0.8mm -> Connector_Pin:Pin_D1.0mm_L10.0mm
- TP3: value Test_PWM -> 5VA; footprint TestPoint:TestPoint_2Pads_Pitch2.54mm_Drill0.8mm -> Connector_Pin:Pin_D1.0mm_L10.0mm
- TP4: value Test_DIR -> 5V; footprint TestPoint:TestPoint_2Pads_Pitch2.54mm_Drill0.8mm -> Connector_Pin:Pin_D1.0mm_L10.0mm
- moved J4 33.4 mm to (165.1, 124.7)
- moved J10 30.9 mm to (190.5, 102.1)
- moved DRV1 28.0 mm to (118.1, 67.3)
- moved J5 25.7 mm to (165.1, 112.8)
- moved J9 24.1 mm to (188.1, 126.2)
- moved J8 23.4 mm to (188.6, 112.8)
- moved SW3 21.0 mm to (168.1, 45.7)
- moved U1 19.4 mm to (66.5, 93.1)
- moved J7 16.3 mm to (169.7, 84.6)
- moved SW5 16.2 mm to (175.5, 33.0)
- moved C1 14.2 mm to (121.2, 28.7), turned to 90 degrees
- moved SW1 14.2 mm to (110.5, 26.4)
- moved J1 13.9 mm to (121.9, 143.3)
- moved SW4 13.0 mm to (160.3, 23.1)
- moved J2 12.9 mm to (122.9, 152.8)
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Connections:
- C2 pad 2: +5V -> +3.3V
- C3 pad 2: +5V -> +3.3V
- C4 pad 2: +5V -> +3.3V
- C5 pad 2: +5V -> +3.3V
- J1 pad 2: +12V -> /DEBUG_TX
- J10 pad 2: /I2C1_SCL -> Net-(J10-Pin_2)
- J11 pad 2: GND -> /Encodeurs/Z+_GAUCHE
- J11 pad 3: /PE0 -> /Encodeurs/Z-_GAUCHE
- J11 pad 4: /PE4 -> /Encodeurs/B-_GAUCHE
- J11 pad 5: /PE5 -> /Encodeurs/B+_GAUCHE
- J11 pad 6: /PD7 -> /Encodeurs/A+_GAUCHE
- J11 pad 7: /PA5 -> /Encodeurs/A-_GAUCHE
- J11 pad 8: +5V -> GND
- J12 pad 1: /PE3 -> +5V
- J12 pad 2: /PD7 -> /Encodeurs/Z+_DROITE
- J12 pad 3: /PA6 -> /Encodeurs/Z-_DROITE
- J12 pad 4: /PA5 -> /Encodeurs/B-_DROITE
- J2 pad 2: +12VA -> /PA12
- J3 pad 2: +5V -> /PG15
- J4 pad 1: +5V -> GND
- J4 pad 2: /Encodeurs/Z+_GAUCHE -> /PC3
- J4 pad 3: /Encodeurs/Z-_GAUCHE -> /PC2
- J4 pad 4: /Encodeurs/B-_GAUCHE -> /PB10
- J5 pad 1: +5V -> GND
- J5 pad 2: /Encodeurs/Z+_DROITE -> /PB2
- J5 pad 3: /Encodeurs/Z-_DROITE -> /PC11
- J5 pad 4: /Encodeurs/B-_DROITE -> /PC10
- J6 pad 1: /Moteurs/MOTOR1A -> GND
- J6 pad 2: /Moteurs/MOTOR1B -> /I2C2_SDA
- J7 pad 1: /Moteurs/MOTOR2A -> GND
- J7 pad 2: /Moteurs/MOTOR2B -> /I2C3_SDA
- J8 pad 2: /I2C1_SCL -> Net-(J8-Pin_2)
- J9 pad 2: +12VA -> Net-(J9-Pin_2)
- TP1 pad 1: /Encodeur_Gauche_A -> GND
- TP2 pad 1: /Encodeur_Droit_A -> +3.3V
- TP3 pad 1: /PE9 -> +5VA
- TP4 pad 1: /PF5 -> +5V
- U1 pad CN10_31: /PB0 -> unconnected-(U1F-D33/TIMER_D_PWM1-PadCN10_31)
- U1 pad CN10_33: unconnected-(U1F-D34/TIMER_B_ETR-PadCN10_33) -> /PE0
- U1 pad CN11_16: +3V3 -> Net-(U1A-3V3)
- U1 pad CN12_27: /PB4 -> unconnected-(U1B-PB4-PadCN12_27)
- U1 pad CN7_15: /PB3 -> unconnected-(U1E-D23/I2S_B_CK/SPI_B_SCK-PadCN7_15)
- U1 pad CN7_19: /PB4 -> unconnected-(U1E-D25/SPI_B_MISO-PadCN7_19)
- U1 pad CN8_14: /PF2 -> /PG2
- U3 pad 5: +5V -> +3.3V
- U4 pad 5: +5V -> +3.3V
- U5 pad 5: +5V -> +3.3V
- U6 pad 5: +5V -> +3.3V

Commit message: Avancée PCB
Parts:
- removed F4: 5A, Fuse:Fuse_2010_5025Metric_Pad1.52x2.65mm_HandSolder
- removed J16: AX12, Connector_Molex:Molex_KK-254_AE-6410-03A_1x03_P2.54mm_Vertical
- removed J17: I2C_Sensors, Connector_Molex:Molex_KK-254_AE-6410-04A_1x04_P2.54mm_Vertical
- removed J18: LCD_TFT, Connector_PinSocket_2.54mm:PinSocket_1x14_P2.54mm_Vertical
- removed J19: LCD_SD, Connector_PinSocket_2.54mm:PinSocket_1x04_P2.54mm_Vertical
- removed SW5: Rouge, Connector_Molex:Molex_KK-254_AE-6410-04A_1x04_P2.54mm_Vertical
- removed TP10: Test_DIR, TestPoint:TestPoint_2Pads_Pitch2.54mm_Drill0.8mm
- added C6: x, Capacitor_THT:CP_Radial_D8.0mm_P3.50mm, F.Cu at (189.2, 45.7)
- added D6: LED, LED_SMD:LED_2010_5025Metric_Pad1.52x2.65mm_HandSolder, F.Cu at (140.5, 100.1)
- added D7: LED, LED_SMD:LED_2010_5025Metric_Pad1.52x2.65mm_HandSolder, F.Cu at (136.2, 100.1)
- added M1: Motor_Servo, Connector_PinHeader_2.54mm:PinHeader_1x03_P2.54mm_Vertical, F.Cu at (140.3, 44.5)
- added M10: Motor_Servo, Connector_PinHeader_2.54mm:PinHeader_1x03_P2.54mm_Vertical, F.Cu at (170.8, 44.5)
- added M11: Motor_Servo, Connector_PinHeader_2.54mm:PinHeader_1x03_P2.54mm_Vertical, F.Cu at (153.0, 44.5)
- added M12: Motor_Servo, Connector_PinHeader_2.54mm:PinHeader_1x03_P2.54mm_Vertical, F.Cu at (155.6, 44.5)
- added M13: Motor_Servo, Connector_PinHeader_2.54mm:PinHeader_1x03_P2.54mm_Vertical, F.Cu at (158.1, 44.5)
- added M2: Motor_Servo, Connector_PinHeader_2.54mm:PinHeader_1x03_P2.54mm_Vertical, F.Cu at (160.7, 44.5)
- added M3: Motor_Servo, Connector_PinHeader_2.54mm:PinHeader_1x03_P2.54mm_Vertical, F.Cu at (142.9, 44.5)
- added M4: Motor_Servo, Connector_PinHeader_2.54mm:PinHeader_1x03_P2.54mm_Vertical, F.Cu at (163.2, 44.5)
- added M5: Motor_Servo, Connector_PinHeader_2.54mm:PinHeader_1x03_P2.54mm_Vertical, F.Cu at (145.4, 44.5)
- added M6: Motor_Servo, Connector_PinHeader_2.54mm:PinHeader_1x03_P2.54mm_Vertical, F.Cu at (165.7, 44.5)
- added M7: Motor_Servo, Connector_PinHeader_2.54mm:PinHeader_1x03_P2.54mm_Vertical, F.Cu at (148.0, 44.5)
- added M8: Motor_Servo, Connector_PinHeader_2.54mm:PinHeader_1x03_P2.54mm_Vertical, F.Cu at (168.3, 44.5)
- added M9: Motor_Servo, Connector_PinHeader_2.54mm:PinHeader_1x03_P2.54mm_Vertical, F.Cu at (150.5, 44.5)
- added R19: 220, LED_SMD:LED_1210_3225Metric_Pad1.42x2.65mm_HandSolder, F.Cu at (147.3, 83.8)
- added R20: 220, LED_SMD:LED_1210_3225Metric_Pad1.42x2.65mm_HandSolder, F.Cu at (143.5, 83.8)
- added R21: 220, LED_SMD:LED_1210_3225Metric_Pad1.42x2.65mm_HandSolder, F.Cu at (139.7, 83.8)
- added R22: 220, LED_SMD:LED_1210_3225Metric_Pad1.42x2.65mm_HandSolder, F.Cu at (135.9, 83.8)
- added R23: 220, LED_SMD:LED_1210_3225Metric_Pad1.42x2.65mm_HandSolder, F.Cu at (132.1, 83.8)
- added R24: x, LED_SMD:LED_1210_3225Metric_Pad1.42x2.65mm_HandSolder, F.Cu at (141.9, 128.3)
- added R25: x, LED_SMD:LED_1210_3225Metric_Pad1.42x2.65mm_HandSolder, F.Cu at (137.6, 128.3)
- added R26: x, LED_SMD:LED_1210_3225Metric_Pad1.42x2.65mm_HandSolder, F.Cu at (133.3, 128.3)
- added R27: 10k, Resistor_SMD:R_1210_3225Metric_Pad1.30x2.65mm_HandSolder, F.Cu at (94.3, 105.4)
- added R28: 10K, Resistor_SMD:R_1210_3225Metric_Pad1.30x2.65mm_HandSolder, B.Cu at (94.0, 104.1)
- added R29: 10k, Resistor_SMD:R_1210_3225Metric_Pad1.30x2.65mm_HandSolder, F.Cu at (94.3, 109.2)
- added R30: 10K, Resistor_SMD:R_1210_3225Metric_Pad1.30x2.65mm_HandSolder, B.Cu at (94.0, 108.8)
- added R31: 10k, Resistor_SMD:R_1210_3225Metric_Pad1.30x2.65mm_HandSolder, F.Cu at (94.3, 113.0)
- added R32: 10K, Resistor_SMD:R_1210_3225Metric_Pad1.30x2.65mm_HandSolder, B.Cu at (94.0, 113.9)
- added R33: 10k, Resistor_SMD:R_1210_3225Metric_Pad1.30x2.65mm_HandSolder, F.Cu at (94.3, 116.8)
- added R34: 10K, Resistor_SMD:R_1210_3225Metric_Pad1.30x2.65mm_HandSolder, B.Cu at (94.0, 119.0)
- added U7: PCA9685PW, Package_SO:TSSOP-28_4.4x9.7mm_P0.65mm, F.Cu at (123.5, 81.6)
- C1: value 0.1uF -> 100n
- C5: value 100n -> 10u
- D5: value 12V -> LED
- F2: value 2A -> 5A
- J10: value 5V -> Moteur_Gauche; footprint Connector_AMASS:AMASS_XT30U-M_1x02_P5.0mm_Vertical -> TerminalBlock:TerminalBlock_bornier-2_P5.08mm
- J11: value Encodeur_G -> Moteur_Droit; footprint Connector_PinHeader_2.54mm:PinHeader_1x08_P2.54mm_Vertical -> TerminalBlock:TerminalBlock_bornier-2_P5.08mm
- J12: value Encodeur_D -> AX12; footprint Connector_PinHeader_2.54mm:PinHeader_1x08_P2.54mm_Vertical -> Connector_Molex:Molex_KK-254_AE-6410-03A_1x03_P2.54mm_Vertical
- J13: value Moteur_Gauche -> I2C_Sensors; footprint TerminalBlock:TerminalBlock_bornier-2_P5.08mm -> Connector_Molex:Molex_KK-254_AE-6410-04A_1x04_P2.54mm_Vertical
- J14: value Moteur_Droit -> LCD_TFT; footprint TerminalBlock:TerminalBlock_bornier-2_P5.08mm -> Connector_PinSocket_2.54mm:PinSocket_1x14_P2.54mm_Vertical; moved to B.Cu
- J15: value PCA9685 -> LCD_SD; footprint Connector_Molex:Molex_KK-254_AE-6410-06A_1x06_P2.54mm_Vertical -> Connector_PinSocket_2.54mm:PinSocket_1x04_P2.54mm_Vertical; moved to B.Cu
- J2: value PA -> SPI2; footprint Connector_Molex:Molex_KK-254_AE-6410-05A_1x05_P2.54mm_Vertical -> Connector_Molex:Molex_KK-254_AE-6410-04A_1x04_P2.54mm_Vertical
- J3: value PG -> SPI3; footprint Connector_Molex:Molex_KK-254_AE-6410-08A_1x08_P2.54mm_Vertical -> Connector_Molex:Molex_KK-254_AE-6410-04A_1x04_P2.54mm_Vertical
- J4: value SPI2 -> I2C2; footprint Connector_Molex:Molex_KK-254_AE-6410-04A_1x04_P2.54mm_Vertical -> Connector_Molex:Molex_KK-254_AE-6410-03A_1x03_P2.54mm_Vertical
- J5: value SPI3 -> I2C3; footprint Connector_Molex:Molex_KK-254_AE-6410-04A_1x04_P2.54mm_Vertical -> Connector_Molex:Molex_KK-254_AE-6410-03A_1x03_P2.54mm_Vertical
- J6: value I2C2 -> 12VA; footprint Connector_Molex:Molex_KK-254_AE-6410-03A_1x03_P2.54mm_Vertical -> Connector_AMASS:AMASS_XT60-M_1x02_P7.20mm_Vertical
- J7: value I2C3 -> 5V; footprint Connector_Molex:Molex_KK-254_AE-6410-03A_1x03_P2.54mm_Vertical -> Connector_AMASS:AMASS_XT30U-M_1x02_P5.0mm_Vertical
- J8: value 12V -> Encodeur_G; footprint Connector_AMASS:AMASS_XT60-M_1x02_P7.20mm_Vertical -> Connector_Molex:Molex_KK-254_AE-6410-08A_1x08_P2.54mm_Vertical
- J9: value 12VA -> Encodeur_D; footprint Connector_AMASS:AMASS_XT60-M_1x02_P7.20mm_Vertical -> Connector_Molex:Molex_KK-254_AE-6410-08A_1x08_P2.54mm_Vertical
- R10: value 100 -> 220; footprint Resistor_THT:R_Axial_DIN0207_L6.3mm_D2.5mm_P10.16mm_Horizontal -> LED_SMD:LED_1210_3225Metric_Pad1.42x2.65mm_HandSolder
- R11, R15, R17: value 10k -> 220; footprint Resistor_SMD:R_1210_3225Metric_Pad1.30x2.65mm_HandSolder -> LED_SMD:LED_1210_3225Metric_Pad1.42x2.65mm_HandSolder
- R12, R14, R16, R18: value 10K -> 220; footprint Resistor_SMD:R_1210_3225Metric_Pad1.30x2.65mm_HandSolder -> LED_SMD:LED_1210_3225Metric_Pad1.42x2.65mm_HandSolder
- R13: footprint Resistor_SMD:R_1210_3225Metric_Pad1.30x2.65mm_HandSolder -> LED_SMD:LED_1210_3225Metric_Pad1.42x2.65mm_HandSolder
- R6: value R -> 100
- R7, R8, R9: footprint Resistor_THT:R_Axial_DIN0207_L6.3mm_D2.5mm_P10.16mm_Horizontal -> Resistor_SMD:R_1210_3225Metric_Pad1.30x2.65mm_HandSolder
- SW1: value RESET -> Vert; footprint Button_Switch_THT:SW_PUSH_6mm -> Connector_Molex:Molex_KK-254_AE-6410-04A_1x04_P2.54mm_Vertical
- SW2: value Vert -> Jaune
- SW3: value Jaune -> Bleu
- SW4: value Bleu -> Rouge
- TP6: value 12V -> Test_Gauche; footprint Connector_Pin:Pin_D1.0mm_L10.0mm -> TestPoint:TestPoint_2Pads_Pitch2.54mm_Drill0.8mm
- TP7: value Test_Gauche -> Test_Droit
- TP8: value Test_Droit -> Test_PWM
- TP9: value Test_PWM -> Test_DIR
- moved H4 157.3 mm to (63.5, 128.3)
- moved H3 149.4 mm to (63.5, 38.1)
- moved TP9 148.8 mm to (88.9, 49.5), turned to 90 degrees
- moved TP8 147.2 mm to (83.8, 49.5), turned to 90 degrees
- moved Q1 146.6 mm to (63.5, 91.1)
- moved TP5 142.0 mm to (76.3, 63.0)
- moved TP7 132.1 mm to (98.6, 49.5), turned to 90 degrees
- moved J15 131.9 mm to (95.3, 82.5), turned to 180 degrees
- moved F3 130.9 mm to (81.3, 111.8), turned to -90 degrees
- moved F2 130.0 mm to (81.3, 101.6), turned to -90 degrees
- moved TP6 127.8 mm to (95.2, 49.5), turned to 90 degrees
- moved J10 121.2 mm to (87.6, 38.1), turned to 180 degrees
- moved D1 118.6 mm to (69.8, 50.8)
- moved D2 118.6 mm to (69.8, 55.1)
- moved D3 118.6 mm to (69.8, 59.4)
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Connections:
- C1 pad 1: /NRST -> GND
- C1 pad 2: GND -> +3.3V
- C5 pad 2: +3.3V -> +5V
- D5 pad 2: Net-(D5-A) -> /Actionneurs + sensors/PWM13
- F1 pad 2: +3V3 -> +3.3V
- F2 pad 1: Net-(J8-Pin_2) -> Net-(J6-Pin_2)
- F2 pad 2: +12V -> +12VA
- F3 pad 1: Net-(J9-Pin_2) -> Net-(J7-Pin_2)
- F3 pad 2: +12VA -> +5V
- J10 pad 1: GND -> /Moteurs/MOTOR1A
- J10 pad 2: Net-(J10-Pin_2) -> /Moteurs/MOTOR1B
- J11 pad 1: +5V -> /Moteurs/MOTOR2A
- J11 pad 2: /Encodeurs/Z+_GAUCHE -> /Moteurs/MOTOR2B
- J12 pad 1: +5V -> GND
- J12 pad 2: /Encodeurs/Z+_DROITE -> +12VA
- J12 pad 3: /Encodeurs/Z-_DROITE -> /AX12_RX
- J13 pad 1: /Moteurs/MOTOR1A -> GND
- J13 pad 2: /Moteurs/MOTOR1B -> /I2C1_SCL
- J14 pad 1: /Moteurs/MOTOR2A -> +3.3V
- J14 pad 2: /Moteurs/MOTOR2B -> GND
- J15 pad 1: +5VA -> /PE3
- J15 pad 2: +5V -> /PD7
- J15 pad 3: /I2C1_SDA -> /PA6
- J15 pad 4: /I2C1_SCL -> /PA5
- J2 pad 2: /PA12 -> /PC3
- J2 pad 3: /PA11 -> /PC2
- J2 pad 4: /PA10 -> /PB10
- J3 pad 2: /PG15 -> /PB2
- J3 pad 3: /PG10 -> /PC11
- J3 pad 4: /PG9 -> /PC10
- J4 pad 2: /PC3 -> /I2C2_SDA
- J4 pad 3: /PC2 -> /I2C2_SCL
- J5 pad 2: /PB2 -> /I2C3_SDA
- J5 pad 3: /PC11 -> /I2C3_SCL
- J6 pad 2: /I2C2_SDA -> Net-(J6-Pin_2)
- J7 pad 2: /I2C3_SDA -> Net-(J7-Pin_2)
- J8 pad 1: GND -> +5V
- J8 pad 2: Net-(J8-Pin_2) -> /Encodeurs/Z+_GAUCHE
- J9 pad 1: GND -> +5V
- J9 pad 2: Net-(J9-Pin_2) -> /Encodeurs/Z+_DROITE
- R10 pad 1: /Encodeurs/A-_DROITE -> Net-(U7-LED0)
- R10 pad 2: /Encodeurs/A+_DROITE -> /Actionneurs + sensors/PWM0
- R11 pad 1: GND -> Net-(U7-LED1)
- R11 pad 2: /PE8 -> /Actionneurs + sensors/PWM1
- R12 pad 1: /PF15 -> Net-(U7-LED2)
- R12 pad 2: +5V -> /Actionneurs + sensors/PWM2
- R13 pad 1: GND -> Net-(U7-~{OE})
- R13 pad 2: /PE7 -> GND
- R14 pad 1: /PF14 -> Net-(U7-LED3)
- R14 pad 2: +5V -> /Actionneurs + sensors/PWM3
- R15 pad 1: GND -> Net-(U7-LED4)
- R15 pad 2: /PG1 -> /Actionneurs + sensors/PWM4
- R16 pad 1: /PF13 -> Net-(U7-LED5)
- R16 pad 2: +5V -> /Actionneurs + sensors/PWM5
- R17 pad 1: GND -> Net-(U7-LED6)
- R17 pad 2: /PB1 -> /Actionneurs + sensors/PWM6
- R18 pad 1: /PG0 -> Net-(U7-LED7)
- R18 pad 2: +5V -> /Actionneurs + sensors/PWM7
- R6 pad 1: +12V -> /Encodeurs/B-_GAUCHE
- R6 pad 2: Net-(D5-A) -> /Encodeurs/B+_GAUCHE
- R7 pad 1: /Encodeurs/B-_GAUCHE -> /Encodeurs/A-_GAUCHE
- R7 pad 2: /Encodeurs/B+_GAUCHE -> /Encodeurs/A+_GAUCHE
- R8 pad 1: /Encodeurs/A-_GAUCHE -> /Encodeurs/B-_DROITE
- R8 pad 2: /Encodeurs/A+_GAUCHE -> /Encodeurs/B+_DROITE
- R9 pad 1: /Encodeurs/B-_DROITE -> /Encodeurs/A-_DROITE
- R9 pad 2: /Encodeurs/B+_DROITE -> /Encodeurs/A+_DROITE
- SW1 pad 2: /NRST -> /PF15
- SW2 pad 2: /PF15 -> /PF14
- SW2 pad 3: Net-(Q2-D) -> Net-(Q3-D)
- SW3 pad 2: /PF14 -> /PF13
- SW3 pad 3: Net-(Q3-D) -> Net-(Q4-D)
- SW4 pad 2: /PF13 -> /PG0
- SW4 pad 3: Net-(Q4-D) -> Net-(Q5-D)
- TP6 pad 1: +12V -> /Encodeur_Gauche_A
- TP7 pad 1: /Encodeur_Gauche_A -> /Encodeur_Droit_A
- TP7 pad 2: /Encodeur_Gauche_B -> /Encodeur_Droit_B
- TP8 pad 1: /Encodeur_Droit_A -> /PE9
- TP8 pad 2: /Encodeur_Droit_B -> /PE11
- TP9 pad 1: /PE9 -> /PF5
- TP9 pad 2: /PE11 -> /PF4
- U1 pad CN11_1: /PC10 -> unconnected-(U1A-PC10-PadCN11_1)
- U1 pad CN11_14: /NRST -> unconnected-(U1A-NRST-PadCN11_14)
- U1 pad CN11_17: /PA15 -> unconnected-(U1A-PA15-PadCN11_17)
- U1 pad CN11_2: /PC11 -> unconnected-(U1A-PC11-PadCN11_2)
- U1 pad CN11_28: /PA0 -> unconnected-(U1A-PA0-PadCN11_28)
- U1 pad CN11_3: /PC12 -> unconnected-(U1A-PC12-PadCN11_3)
- U1 pad CN11_32: /PA4 -> unconnected-(U1A-PA4-PadCN11_32)
- U1 pad CN11_35: /PC2 -> unconnected-(U1A-PC2-PadCN11_35)
- U1 pad CN11_37: /PC3 -> unconnected-(U1A-PC3-PadCN11_37)
- U1 pad CN11_38: /PC0 -> unconnected-(U1A-PC0-PadCN11_38)
- U1 pad CN11_39: /PD4 -> unconnected-(U1A-PD4-PadCN11_39)
- U1 pad CN11_4: /PD2 -> unconnected-(U1A-PD2-PadCN11_4)
- U1 pad CN11_40: /PD3 -> unconnected-(U1A-PD3-PadCN11_40)
- U1 pad CN11_42: /PG2 -> unconnected-(U1A-PG2-PadCN11_42)
- U1 pad CN11_43: /PD6 -> unconnected-(U1A-PD6-PadCN11_43)
- U1 pad CN11_44: /PG3 -> unconnected-(U1A-PG3-PadCN11_44)
- U1 pad CN11_45: /PD7 -> unconnected-(U1A-PD7-PadCN11_45)
- U1 pad CN11_46: /PE2 -> unconnected-(U1A-PE2-PadCN11_46)
- U1 pad CN11_47: /PE3 -> unconnected-(U1A-PE3-PadCN11_47)
- U1 pad CN11_48: /PE4 -> unconnected-(U1A-PE4-PadCN11_48)
- U1 pad CN11_50: /PE5 -> unconnected-(U1A-PE5-PadCN11_50)
- U1 pad CN11_52: /PF2 -> unconnected-(U1A-PF2-PadCN11_52)
- U1 pad CN11_54: /PF8 -> unconnected-(U1A-PF8-PadCN11_54)
- U1 pad CN11_55: /PD1 -> unconnected-(U1A-PD1-PadCN11_55)
- U1 pad CN11_56: /PF9 -> unconnected-(U1A-PF9-PadCN11_56)
- U1 pad CN11_57: /PD0 -> unconnected-(U1A-PD0-PadCN11_57)
- U1 pad CN11_58: /PG1 -> unconnected-(U1A-PG1-PadCN11_58)
- U1 pad CN11_59: /PG0 -> unconnected-(U1A-PG0-PadCN11_59)
- U1 pad CN11_62: /PE6 -> unconnected-(U1A-PE6-PadCN11_62)
- U1 pad CN11_63: /PG9 -> unconnected-(U1A-PG9-PadCN11_63)
- U1 pad CN11_64: /PG15 -> unconnected-(U1A-PG15-PadCN11_64)
- U1 pad CN11_65: /PG12 -> unconnected-(U1A-PG12-PadCN11_65)
- U1 pad CN11_66: /PG10 -> unconnected-(U1A-PG10-PadCN11_66)
- U1 pad CN12_11: /PA5 -> unconnected-(U1B-PA5-PadCN12_11)
- U1 pad CN12_12: /PA12 -> unconnected-(U1B-PA12-PadCN12_12)
- U1 pad CN12_13: /PA6 -> unconnected-(U1B-PA6-PadCN12_13)
- U1 pad CN12_14: /PA11 -> unconnected-(U1B-PA11-PadCN12_14)
- U1 pad CN12_16: /PB12 -> unconnected-(U1B-PB12-PadCN12_16)
- U1 pad CN12_18: /PB11 -> unconnected-(U1B-PB11-PadCN12_18)
- U1 pad CN12_19: /PC7 -> unconnected-(U1B-PC7-PadCN12_19)
- U1 pad CN12_2: /PC8 -> unconnected-(U1B-PC8-PadCN12_2)
- U1 pad CN12_21: /PA9 -> unconnected-(U1B-PA9-PadCN12_21)
- U1 pad CN12_22: /PB2 -> unconnected-(U1B-PB2-PadCN12_22)
- U1 pad CN12_24: /PB1 -> unconnected-(U1B-PB1-PadCN12_24)
- U1 pad CN12_25: /PB10 -> unconnected-(U1B-PB10-PadCN12_25)
- U1 pad CN12_26: /PB15 -> unconnected-(U1B-PB15-PadCN12_26)
- U1 pad CN12_28: /PB14 -> unconnected-(U1B-PB14-PadCN12_28)
- U1 pad CN12_29: /PB5 -> unconnected-(U1B-PB5-PadCN12_29)
- U1 pad CN12_3: /PB8 -> unconnected-(U1B-PB8-PadCN12_3)
- U1 pad CN12_30: /PB13 -> unconnected-(U1B-PB13-PadCN12_30)
- U1 pad CN12_33: /PA10 -> unconnected-(U1B-PA10-PadCN12_33)
- U1 pad CN12_36: /PF5 -> unconnected-(U1B-PF5-PadCN12_36)
- U1 pad CN12_38: /PF4 -> unconnected-(U1B-PF4-PadCN12_38)
- U1 pad CN12_4: /PC6 -> unconnected-(U1B-PC6-PadCN12_4)
- U1 pad CN12_40: /PE8 -> unconnected-(U1B-PE8-PadCN12_40)
- U1 pad CN12_41: /PD13 -> unconnected-(U1B-PD13-PadCN12_41)
- U1 pad CN12_42: /PF10 -> unconnected-(U1B-PF10-PadCN12_42)
- U1 pad CN12_43: /PD12 -> unconnected-(U1B-PD12-PadCN12_43)
- U1 pad CN12_44: /PE7 -> unconnected-(U1B-PE7-PadCN12_44)
- U1 pad CN12_45: /PD11 -> unconnected-(U1B-PD11-PadCN12_45)
- U1 pad CN12_46: /PD14 -> unconnected-(U1B-PD14-PadCN12_46)
- U1 pad CN12_47: /PE10 -> unconnected-(U1B-PE10-PadCN12_47)
- U1 pad CN12_48: /PD15 -> unconnected-(U1B-PD15-PadCN12_48)
- U1 pad CN12_49: /PE12 -> unconnected-(U1B-PE12-PadCN12_49)
- U1 pad CN12_5: /PB9 -> unconnected-(U1B-PB9-PadCN12_5)
- U1 pad CN12_50: /PF14 -> unconnected-(U1B-PF14-PadCN12_50)
- U1 pad CN12_51: /PE14 -> unconnected-(U1B-PE14-PadCN12_51)
- U1 pad CN12_52: /PE9 -> unconnected-(U1B-PE9-PadCN12_52)
- U1 pad CN12_53: /PE15 -> unconnected-(U1B-PE15-PadCN12_53)
- U1 pad CN12_55: /PE13 -> unconnected-(U1B-PE13-PadCN12_55)
- U1 pad CN12_56: /PE11 -> unconnected-(U1B-PE11-PadCN12_56)
- U1 pad CN12_57: /PF13 -> unconnected-(U1B-PF13-PadCN12_57)
- U1 pad CN12_58: /PF3 -> unconnected-(U1B-PF3-PadCN12_58)
- U1 pad CN12_60: /PF15 -> unconnected-(U1B-PF15-PadCN12_60)
- U1 pad CN12_61: /PG14 -> unconnected-(U1B-PG14-PadCN12_61)
- U1 pad CN12_64: /PE0 -> unconnected-(U1B-PE0-PadCN12_64)
- U1 pad CN12_66: /PG8 -> unconnected-(U1B-PG8-PadCN12_66)
- U1 pad CN12_68: /PG5 -> unconnected-(U1B-PG5-PadCN12_68)
- U1 pad CN12_69: /PG4 -> unconnected-(U1B-PG4-PadCN12_69)
- U1 pad CN12_70: /PG6 -> unconnected-(U1B-PG6-PadCN12_70)
- U1 pad CN8_5: /NRST -> unconnected-(U1C-NRST_CN8-PadCN8_5)
- U1 pad CN8_7: +3V3 -> Net-(U1A-3V3)
Routing:
- added copper zone on B.Cu, net GND
- added copper zone on F.Cu, net GND
Other:
- board outline added: 152.4 x 101.6 mm
