File: Carte-Principale/Carte-Principale.kicad_pcb (KiCad board)
At the start: 2 copper layers, 152.4 x 101.6 mm, 108 parts, among them J1 Serial, J10 Moteur_Gauche, J11 Moteur_Droit, J12 AX12, J13 I2C_Sensors, J14 LCD_TFT, J15 LCD_SD, J2 SPI2, J3 SPI3, J4 I2C2, J5 I2C3, J6 12VA, J7 5V, J8 Encodeur_G, J9 Encodeur_D, M1 Motor_Servo, M10 Motor_Servo, M11 Motor_Servo, M12 Motor_Servo, M13 Motor_Servo, M2 Motor_Servo, M3 Motor_Servo, M4 Motor_Servo, M5 Motor_Servo, M6 Motor_Servo, M7 Motor_Servo, M8 Motor_Servo, M9 Motor_Servo, Q1 IRF630, Q2 BSS138, Q3 BSS138, Q4 BSS138, Q5 BSS138, SW1 Vert, SW2 Jaune, SW3 Bleu, SW4 Rouge, U1 NUCLEOH723ZG, U2 AM26LV32xD, U3 74LVC1G3157, U4 74LVC1G3157, U5 74LVC1G3157, U6 74LVC1G3157, U7 PCA9685PW

Commit message: avancée
Parts:
- removed the J3 at (154.9, 128.3)
- removed the J4 at (188.0, 128.3)
- added G***: LOGO, LOGO, F.Cu at (67.0, 47.0)
- added G0: LOGO, LOGO, F.Cu at (170.0, 133.0)
- added J10: SPI3, Connector_Molex:Molex_KK-254_AE-6410-04A_1x04_P2.54mm_Vertical, F.Cu at (120.5, 129.5)
- added J8: I2C2, Connector_Molex:Molex_KK-254_AE-6410-04A_1x04_P2.54mm_Vertical, F.Cu at (133.2, 129.5)
- added J9: GPIO, Connector_Molex:Molex_KK-254_AE-6410-04A_1x04_P2.54mm_Vertical, F.Cu at (120.5, 138.4)
- added kibuzzard-1: G***, kibuzzard-66C08CAE, F.Cu at (72.4, 55.9)
- added kibuzzard-10: G***, kibuzzard-66C08EB4, F.Cu at (102.0, 144.1)
- added kibuzzard-11: G***, kibuzzard-66C46925, F.Cu at (129.4, 144.1)
- added kibuzzard-13: G***, kibuzzard-66C08BB8, F.Cu at (141.0, 31.8)
- added kibuzzard-14: G***, kibuzzard-66C08BD9, F.Cu at (171.4, 31.8)
- added kibuzzard-15: G***, kibuzzard-66C34407, F.Cu at (165.8, 49.8)
- added kibuzzard-16: G***, kibuzzard-66C3440D, F.Cu at (165.8, 44.8)
- added kibuzzard-17: G***, kibuzzard-66C0927B, F.Cu at (189.0, 44.5)
- added kibuzzard-18: G***, kibuzzard-66C34414, F.Cu at (165.5, 47.3)
- added kibuzzard-19: G***, kibuzzard-66C3235E, F.Cu at (169.4, 144.0)
- added kibuzzard-2: G***, kibuzzard-66C08D4F, F.Cu at (67.9, 108.0)
- added kibuzzard-20: G***, kibuzzard-66C32535, F.Cu at (193.0, 31.8)
- added kibuzzard-21: G***, kibuzzard-66C09269, F.Cu at (191.5, 44.5)
- added kibuzzard-22: G***, kibuzzard-66C0929D, F.Cu at (194.0, 50.8)
- added kibuzzard-23: G***, kibuzzard-66C3253B, F.Cu at (207.9, 46.7)
- added kibuzzard-24: G***, kibuzzard-66C09293, F.Cu at (194.0, 48.3)
- added kibuzzard-25: G***, kibuzzard-66C091C7, B.Cu at (193.0, 33.0)
- added kibuzzard-26: G***, kibuzzard-66C0922C, B.Cu at (207.2, 47.0)
- added kibuzzard-27: G***, kibuzzard-66C091DE, B.Cu at (171.4, 33.0)
- added kibuzzard-28: G***, kibuzzard-66C091DE, B.Cu at (141.0, 33.0)
- added kibuzzard-29: G***, kibuzzard-66C09378, B.Cu at (129.4, 134.0)
- added kibuzzard-3: G***, kibuzzard-66C08D66, F.Cu at (68.6, 118.7)
- added kibuzzard-30: G***, kibuzzard-66C09044, B.Cu at (116.7, 134.0)
- added kibuzzard-31: G***, kibuzzard-66C09044, B.Cu at (116.7, 142.9)
- added kibuzzard-32: G***, kibuzzard-66C090AC, B.Cu at (96.5, 33.0)
- added kibuzzard-33: G***, kibuzzard-66C09018, B.Cu at (102.0, 134.0)
- added kibuzzard-34: G***, kibuzzard-66C09018, B.Cu at (102.0, 142.9)
- added kibuzzard-35: G***, kibuzzard-66C090AC, B.Cu at (84.5, 33.0)
- added kibuzzard-36: G***, kibuzzard-66C08FE4, B.Cu at (87.0, 134.0)
- added kibuzzard-37: G***, kibuzzard-66C08FE4, B.Cu at (74.3, 134.0)
- added kibuzzard-38: G***, kibuzzard-66C08FE4, B.Cu at (87.0, 142.9)
- added kibuzzard-39: G***, kibuzzard-66C08FE4, B.Cu at (74.3, 142.9)
- added kibuzzard-4: G***, kibuzzard-66C08EFC, F.Cu at (80.6, 144.1)
- added kibuzzard-5: G***, kibuzzard-66C08F7C, F.Cu at (95.9, 31.8)
- added kibuzzard-6: G***, kibuzzard-66C09269, F.Cu at (99.0, 45.4)
- added kibuzzard-66C478F6: G***, kibuzzard-66C478F6, F.Cu at (84.5, 108.5)
- added kibuzzard-66C48662: G***, kibuzzard-66C48662, F.Cu at (116.7, 144.1)
- added kibuzzard-7: G***, kibuzzard-66C0927B, F.Cu at (96.5, 45.4)
- added kibuzzard-8: G***, kibuzzard-66C092E0, F.Cu at (93.3, 49.2)
- added kibuzzard-9: G***, kibuzzard-66C092F4, F.Cu at (93.3, 51.8)
- C3, C4, U5: moved to B.Cu
- C5: renamed from C1; moved to B.Cu
- C6: renamed from C2; moved to B.Cu
- J11: renamed from J2; value SPI2 -> GPIO
- J5: value I2C3 -> UART_Debug; footprint Connector_Molex:Molex_KK-254_AE-6410-03A_1x03_P2.54mm_Vertical -> Connector_Molex:Molex_KK-254_AE-6410-04A_1x04_P2.54mm_Vertical
- J6: renamed from J1; value Serial -> UART; footprint Connector_Molex:Molex_KK-254_AE-6410-03A_1x03_P2.54mm_Vertical -> Connector_Molex:Molex_KK-254_AE-6410-04A_1x04_P2.54mm_Vertical
- R16: renamed from R19; footprint LED_SMD:LED_1210_3225Metric_Pad1.42x2.65mm_HandSolder -> Resistor_SMD:R_1210_3225Metric_Pad1.30x2.65mm_HandSolder
- R18: renamed from R17; footprint LED_SMD:LED_1210_3225Metric_Pad1.42x2.65mm_HandSolder -> Resistor_SMD:R_1210_3225Metric_Pad1.30x2.65mm_HandSolder
- R19: renamed from R16; footprint LED_SMD:LED_1210_3225Metric_Pad1.42x2.65mm_HandSolder -> Resistor_SMD:R_1210_3225Metric_Pad1.30x2.65mm_HandSolder
- R2: renamed from R24; footprint LED_SMD:LED_1210_3225Metric_Pad1.42x2.65mm_HandSolder -> Resistor_SMD:R_1210_3225Metric_Pad1.30x2.65mm_HandSolder
- R20: renamed from R18; footprint LED_SMD:LED_1210_3225Metric_Pad1.42x2.65mm_HandSolder -> Resistor_SMD:R_1210_3225Metric_Pad1.30x2.65mm_HandSolder
- R22: renamed from R15; footprint LED_SMD:LED_1210_3225Metric_Pad1.42x2.65mm_HandSolder -> Resistor_SMD:R_1210_3225Metric_Pad1.30x2.65mm_HandSolder
- R23: footprint LED_SMD:LED_1210_3225Metric_Pad1.42x2.65mm_HandSolder -> Resistor_SMD:R_1210_3225Metric_Pad1.30x2.65mm_HandSolder
- R24: renamed from R22; footprint LED_SMD:LED_1210_3225Metric_Pad1.42x2.65mm_HandSolder -> Resistor_SMD:R_1210_3225Metric_Pad1.30x2.65mm_HandSolder
- R25: renamed from R20; footprint LED_SMD:LED_1210_3225Metric_Pad1.42x2.65mm_HandSolder -> Resistor_SMD:R_1210_3225Metric_Pad1.30x2.65mm_HandSolder
- R26: renamed from R21; footprint LED_SMD:LED_1210_3225Metric_Pad1.42x2.65mm_HandSolder -> Resistor_SMD:R_1210_3225Metric_Pad1.30x2.65mm_HandSolder
- R27: renamed from R9; moved to B.Cu
- R28: renamed from R6; moved to B.Cu
- R29: renamed from R8; moved to B.Cu
- R30: renamed from R7; moved to B.Cu
- R5: renamed from R25; footprint LED_SMD:LED_1210_3225Metric_Pad1.42x2.65mm_HandSolder -> Resistor_SMD:R_1210_3225Metric_Pad1.30x2.65mm_HandSolder
- R6: renamed from R26; footprint LED_SMD:LED_1210_3225Metric_Pad1.42x2.65mm_HandSolder -> Resistor_SMD:R_1210_3225Metric_Pad1.30x2.65mm_HandSolder
- TP6: value Test_Gauche -> Test_PWM
- TP7: value Test_Droit -> Test_DIR
- TP8: value Test_PWM -> Test_Gauche
- TP9: value Test_DIR -> Test_Droit
- U3: renamed from U2; moved to B.Cu
- U4: renamed from U6; moved to B.Cu
- U6: renamed from U4; moved to B.Cu
- U7: renamed from U3; moved to B.Cu
- moved TP8 105.1 mm to (189.0, 50.8)
- moved C1 104.8 mm to (84.5, 50.4), turned to 90 degrees
- moved TP9 102.6 mm to (191.5, 50.8)
- moved J6 92.9 mm to (105.8, 138.4)
- moved D2 84.3 mm to (63.5, 77.8), turned to 0 degrees
- moved D3 81.3 mm to (63.5, 74.1), turned to 0 degrees
- moved D1 78.6 mm to (63.5, 70.2), turned to 0 degrees
- moved J5 72.0 mm to (105.8, 129.5)
- moved R2 70.1 mm to (87.0, 84.8), turned to 180 degrees
- moved R5 69.2 mm to (87.0, 81.1), turned to 180 degrees
- moved R6 68.7 mm to (87.0, 77.5), turned to 180 degrees
- moved SW2 51.2 mm to (78.1, 138.4)
- moved R23 47.0 mm to (178.5, 76.2), turned to 90 degrees
- moved R29 39.8 mm to (171.2, 49.5)
- moved R24 39.8 mm to (175.0, 76.2), turned to 90 degrees
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- renumbered C6 to C1, C5 to C2, D7 to D1, D5 to D2, D6 to D3, D3 to D4, D2 to D5, D1 to D6, D4 to D7, F3 to F1, F1 to F3, H3 to H1, H4 to H2, H1 to H3, H2 to H4, J10 to J1, J8 to J12, J13 to J17, J6 to J2, J12 to J20, J14 to J21, J15 to J22, J7 to J3, J11 to J4, J9 to J7, M2 to M10, M8 to M11, M11 to M13, M7 to M2, M5 to M4, M9 to M5, M4 to M6, M13 to M7, M10 to M8, M6 to M9, Q3 to Q2, Q2 to Q3, R2 to R1, R31 to R10, R29 to R11, R33 to R12, R12 to R13, R10 to R14, R11 to R15, R14 to R17, R13 to R21, R5 to R3, R32 to R31, R30 to R32, R28 to R33, R3 to R4, R1 to R7, R4 to R8, R27 to R9, SW3 to SW1, SW4 to SW2, SW2 to SW3, SW1 to SW4, TP2 to TP1, TP4 to TP2, TP1 to TP3, TP3 to TP4, U7 to U1, U1 to U2
Connections:
- DRV1 pad EN1: /PF8 -> /PB13
- DRV1 pad EN2: /PF9 -> /PB15
- DRV1 pad FLT: /PE6 -> /PB12
- DRV1 pad RST: /PF10 -> /PA15
- F3 pad 1: Net-(U1A-3V3) -> Net-(U2C-3V3_CN8)
- J11 pad 1: GND -> /PD3
- J11 pad 2: /PC3 -> /PD6
- J11 pad 3: /PC2 -> /PF7
- J11 pad 4: /PB10 -> /PF9
- J5 pad 1: GND -> /DEBUG_RX
- J5 pad 2: /I2C3_SDA -> /DEBUG_TX
- J5 pad 3: /I2C3_SCL -> +5V
- J6 pad 1: GND -> /PC7
- J6 pad 2: /DEBUG_TX -> /PC6
- J6 pad 3: /DEBUG_RX -> +5V
- Q2 pad 1: /PE7 -> /PG2
- Q3 pad 1: /PE8 -> /PD5
- Q4 pad 1: /PG1 -> /PG3
- Q5 pad 1: /PB1 -> /PC9
- R10 pad 2: /PG1 -> /PG3
- R11 pad 2: /PE7 -> /PG2
- R12 pad 2: /PB1 -> /PC9
- R31 pad 1: /PF13 -> /PC12
- R32 pad 1: /PF14 -> /PC8
- R33 pad 1: /PF15 -> /PD2
- R34 pad 1: /PG0 -> /PD4
- R9 pad 2: /PE8 -> /PD5
- SW1 pad 2: /PF13 -> /PC12
- SW2 pad 2: /PG0 -> /PD4
- SW3 pad 2: /PF14 -> /PC8
- SW4 pad 2: /PF15 -> /PD2
- TP6 pad 1: /Encodeur_Gauche_A -> /PE9
- TP6 pad 2: /Encodeur_Gauche_B -> /PE11
- TP7 pad 1: /Encodeur_Droit_A -> /PF5
- TP7 pad 2: /Encodeur_Droit_B -> /PF4
- TP8 pad 1: /PE9 -> /Encodeur_Gauche_A
- TP8 pad 2: /PE11 -> /Encodeur_Gauche_B
- TP9 pad 1: /PF5 -> /Encodeur_Droit_A
- TP9 pad 2: /PF4 -> /Encodeur_Droit_B
- U2 pad CN10_10: /PE13 -> unconnected-(U2F-D3/TIMER_A_PWM3-PadCN10_10)
- U2 pad CN10_11: /Encodeur_Droit_A -> /PF6
- U2 pad CN10_12: /PG14 -> unconnected-(U2F-D2/IO-PadCN10_12)
- U2 pad CN10_14: /I2C1_SCL -> unconnected-(U2F-D1/USART_A_TX-PadCN10_14)
- U2 pad CN10_15: /PB2 -> unconnected-(U2F-D27/QSPI_CLK-PadCN10_15)
- U2 pad CN10_16: /I2C1_SDA -> unconnected-(U2F-D0/USART_A_RX-PadCN10_16)
- U2 pad CN10_2: /PG12 -> unconnected-(U2F-D7/IO-PadCN10_2)
- U2 pad CN10_25: /PE2 -> unconnected-(U2F-D31/QSPI_BK1_IO2-PadCN10_25)
- U2 pad CN10_8: /PE14 -> unconnected-(U2F-D4/IO-PadCN10_8)
- U2 pad CN11_16: Net-(U1A-3V3) -> unconnected-(U2A-3V3-PadCN11_16)
- U2 pad CN11_51: /I2C2_SCL -> unconnected-(U2A-PF1-PadCN11_51)
- U2 pad CN11_53: /I2C2_SDA -> unconnected-(U2A-PF0-PadCN11_53)
- U2 pad CN12_1: /I2C3_SDA -> unconnected-(U2B-PC9-PadCN12_1)
- U2 pad CN12_23: /I2C3_SCL -> unconnected-(U2B-PA8-PadCN12_23)
- U2 pad CN7_13: /PB5 -> unconnected-(U2E-D22/I2S_B_SD/SPI_B_MOSI-PadCN7_13)
- U2 pad CN7_14: /PB5 -> unconnected-(U2E-D11/SPI_A_MOSI/TIM_E_PWM1-PadCN7_14)
- U2 pad CN7_16: /PD14 -> unconnected-(U2E-D10/SPI_A_CS/TIM_B_PWM3-PadCN7_16)
- U2 pad CN7_18: /PD15 -> unconnected-(U2E-D9/TIMER_B_PWM2-PadCN7_18)
- U2 pad CN7_2: /PB8 -> unconnected-(U2E-D15/I2C_A_SCL-PadCN7_2)
- U2 pad CN7_4: /PB9 -> unconnected-(U2E-D14/I2C_A_SDA-PadCN7_4)
- U2 pad CN8_4: /I2C3_SDA -> /PC9
- U2 pad CN8_7: Net-(U1A-3V3) -> Net-(U2C-3V3_CN8)
- U2 pad CN9_1: /AX12_RX -> unconnected-(U2D-A0/ADC12_INP15-PadCN9_1)
- U2 pad CN9_11: /PF10 -> unconnected-(U2D-A5/ADC3_INP6/I2C1_SCL-PadCN9_11)
- U2 pad CN9_15: /PE9 -> unconnected-(U2D-D71/COMP2_INP-PadCN9_15)
- U2 pad CN9_20: /PE6 -> unconnected-(U2D-D59/SAI_A_SD-PadCN9_20)
- U2 pad CN9_26: /Encodeur_Droit_B -> /PF7
- U2 pad CN9_3: /PC0 -> unconnected-(U2D-A1/ADC123_INP10-PadCN9_3)
- U2 pad CN9_5: /PC3 -> unconnected-(U2D-A2/ADC12_INP13-PadCN9_5)
- U2 pad CN9_6: /AX12_RX -> /PD5
- U2 pad CN9_7: /PB1 -> unconnected-(U2D-A3/ADC12_INP5-PadCN9_7)
- U2 pad CN9_9: /PC2 -> unconnected-(U2D-A4/ADC123_INP12/I2C1_SDA-PadCN9_9)
Routing:
- net +5V: track 0.00 -> 400.4 mm, vias 0 -> 4
- net +12VA: track 0.00 -> 245.0 mm
- net /AX12_RX: track 0.00 -> 187.9 mm, vias 0 -> 1
- net /I2C1_SDA: track 0.00 -> 186.8 mm, vias 0 -> 2
- net +5VA: track 0.00 -> 163.4 mm
- net /Encodeur_Droit_B: track 0.00 -> 135.2 mm, vias 0 -> 2
- net /Encodeur_Droit_A: track 0.00 -> 130.0 mm, vias 0 -> 2
- net +3.3V: track 0.00 -> 127.6 mm, vias 0 -> 2
- net /I2C1_SCL: track 0.00 -> 123.2 mm, vias 0 -> 1
- net /PD4: track 0.00 -> 101.3 mm, vias 0 -> 2
- net /PF3: track 0.00 -> 100.2 mm, vias 0 -> 1
- net /DEBUG_RX: track 0.00 -> 97.6 mm
- net /PF5: track 0.00 -> 91.3 mm, vias 0 -> 2
- net /PD1: track 0.00 -> 89.7 mm
- net /PC7: track 0.00 -> 84.0 mm, vias 0 -> 3
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Other:
- board size 152.4 x 101.6 mm -> 154.6 x 118.1 mm
- board text added: "12 11 10 9 8 7 6 5 4 3 2 1 0"
- board text added: "JLCJLCJLCJLC"

Commit message: Final pcb modification
Parts:
- removed the kibuzzard-31 at (116.7, 142.9)
- added J2: GND, Connector_PinHeader_2.54mm:PinHeader_1x04_P2.54mm_Vertical, F.Cu at (75.4, 40.2)
- added kibuzzard-32: G***, kibuzzard-66C60E06, B.Cu at (116.7, 142.9)
- added kibuzzard-33: G***, kibuzzard-66C60E22, B.Cu at (129.2, 142.8)
- added kibuzzard-66C837D2: G***, kibuzzard-66C837D2, F.Cu at (68.0, 74.0)
- renumbered C4 to C3, C3 to C4, C6 to C5, C5 to C6, D3 to D1, D1 to D3, D5 to D4, D4 to D5, F2 to F1, F1 to F2, G0 to G1, J9 to J10, J8 to J11, J11 to J12, J12 to J13, J17 to J14, J20 to J15, J21 to J16, J22 to J17, J2 to J3, J3 to J4, J4 to J5, J5 to J6, J6 to J7, J7 to J8, J10 to J9, M8 to M12, M4 to M2, M2 to M4, M7 to M6, M6 to M7, M12 to M8, Q3 to Q2, Q2 to Q3, R11 to R10, R9 to R11, R15 to R13, R13 to R14, R14 to R15, R20 to R16, R18 to R17, R22 to R18, R21 to R20, R17 to R21, R16 to R22, R26 to R25, R25 to R26, R30 to R28, R8 to R3, R28 to R30, R3 to R4, R7 to R6, R6 to R7, R4 to R8, R10 to R9, SW2 to SW1, SW1 to SW2, TP3 to TP2, TP2 to TP3, U7 to U6, U6 to U7, kibuzzard-8 to kibuzzard-10, kibuzzard-10 to kibuzzard-11, kibuzzard-66C48662 to kibuzzard-12, kibuzzard-11 to kibuzzard-13, kibuzzard-13 to kibuzzard-14, kibuzzard-14 to kibuzzard-15, kibuzzard-18 to kibuzzard-16, kibuzzard-16 to kibuzzard-17, kibuzzard-15 to kibuzzard-18, kibuzzard-17 to kibuzzard-19, kibuzzard-66C478F6 to kibuzzard-2, kibuzzard-19 to kibuzzard-20, kibuzzard-20 to kibuzzard-21, kibuzzard-24 to kibuzzard-22, kibuzzard-21 to kibuzzard-23, kibuzzard-22 to kibuzzard-24, kibuzzard-23 to kibuzzard-25, kibuzzard-25 to kibuzzard-26, kibuzzard-26 to kibuzzard-27, kibuzzard-27 to kibuzzard-28, kibuzzard-28 to kibuzzard-29, kibuzzard-2 to kibuzzard-3, kibuzzard-29 to kibuzzard-31, kibuzzard-32 to kibuzzard-34, kibuzzard-33 to kibuzzard-35, kibuzzard-34 to kibuzzard-36, kibuzzard-35 to kibuzzard-37, kibuzzard-37 to kibuzzard-38, kibuzzard-36 to kibuzzard-39, kibuzzard-3 to kibuzzard-4, kibuzzard-39 to kibuzzard-40, kibuzzard-38 to kibuzzard-41, kibuzzard-4 to kibuzzard-5, kibuzzard-5 to kibuzzard-6, kibuzzard-6 to kibuzzard-7, kibuzzard-7 to kibuzzard-8
Connections:
- J17 pad 1: /PE3 -> /PA4
Routing:
- net /PD7: track 0.00 -> 169.9 mm, vias 0 -> 1
- net /PA6: track 0.00 -> 139.6 mm, vias 0 -> 4
- net /PA5: track 0.00 -> 138.0 mm, vias 0 -> 2
- net +3.3V: track 127.6 -> 244.1 mm, vias 2 -> 3
- net /PG1: track 9.46 -> 77.5 mm
- net /PE2: track 0.00 -> 49.7 mm
- net /PE4: track 0.00 -> 49.6 mm
- net /PA4: track 0.00 -> 48.4 mm, vias 0 -> 2
- net /PE5: track 0.00 -> 47.2 mm
- net /PE0: track 0.00 -> 40.1 mm
- net /PF2: track 0.00 -> 38.8 mm
- net /PD1: track 89.7 -> 94.9 mm
- net +5V: track 400.4 -> 404.3 mm
- net /Encodeur_Gauche_A: track 46.9 -> 43.1 mm
- net /PF5: track 91.3 -> 93.4 mm
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
Commit message: Cartes élec à refaire et TODO
Parts:
- removed C1: x, Capacitor_THT:CP_Radial_D8.0mm_P3.50mm
- removed C2: 10u, Capacitor_SMD:C_1210_3225Metric_Pad1.33x2.70mm_HandSolder
- removed D1, D2, D3: LED, LED_SMD:LED_2010_5025Metric_Pad1.52x2.65mm_HandSolder
- removed D4: 5VA, LED_SMD:LED_2010_5025Metric_Pad1.52x2.65mm_HandSolder
- removed M1, M10, M11, M12, M13, M2, M3, M4, M5, M6, M7, M8, M9: Motor_Servo, Connector_PinHeader_2.54mm:PinHeader_1x03_P2.54mm_Vertical
- removed Q1: IRF630, Package_TO_SOT_THT:TO-220-3_Vertical
- removed R13, R14, R15, R21: 220, LED_SMD:LED_1210_3225Metric_Pad1.42x2.65mm_HandSolder
- removed R16, R17, R18, R19, R22, R23, R24, R25, R26: 220, Resistor_SMD:R_1210_3225Metric_Pad1.30x2.65mm_HandSolder
- removed R2, R5, R7: x, Resistor_SMD:R_1210_3225Metric_Pad1.30x2.65mm_HandSolder
- removed R20: 10k, LED_SMD:LED_1210_3225Metric_Pad1.42x2.65mm_HandSolder
- removed R6: 10K, Resistor_SMD:R_1210_3225Metric_Pad1.30x2.65mm_HandSolder
- removed R8: R, Resistor_SMD:R_1210_3225Metric_Pad1.30x2.65mm_HandSolder
- removed TP4: 5VA, Connector_Pin:Pin_D1.0mm_L10.0mm
- removed U1: PCA9685PW, Package_SO:TSSOP-28_4.4x9.7mm_P0.65mm
- removed kibuzzard-1: G***, kibuzzard-66C08CAE
- removed kibuzzard-15: G***, kibuzzard-66C08BD9
- removed kibuzzard-16: G***, kibuzzard-66C34414
- removed kibuzzard-17: G***, kibuzzard-66C3440D
- removed kibuzzard-18: G***, kibuzzard-66C34407
- removed kibuzzard-20: G***, kibuzzard-66C3235E
- removed kibuzzard-21: G***, kibuzzard-66C32535
- removed kibuzzard-25: G***, kibuzzard-66C3253B
- removed kibuzzard-6: G***, kibuzzard-66C08F7C
- removed kibuzzard-66C837D2: G***, kibuzzard-66C837D2
- added C7: 0.1µ, Capacitor_SMD:C_1210_3225Metric_Pad1.33x2.70mm_HandSolder, B.Cu at (168.5, 78.5)
- added J18: PCA9685, Connector_JST:JST_XH_B4B-XH-A_1x04_P2.50mm_Vertical, F.Cu at (178.9, 138.4)
- added J19: GPIO, Connector_JST:JST_XH_B4B-XH-A_1x04_P2.50mm_Vertical, F.Cu at (164.3, 138.4)
- added kibuzzard-66E9AA77: G***, kibuzzard-66E9AA77, B.Cu at (175.1, 141.9)
- added kibuzzard-66F08110: G***, kibuzzard-66F08110, F.Cu at (113.7, 32.0)
- added kibuzzard-66F08121: G***, kibuzzard-66F08121, F.Cu at (80.3, 45.0)
- added kibuzzard-66F082DD: G***, kibuzzard-66F082DD, B.Cu at (160.8, 142.5)
- added kibuzzard-66FDA353: G***, kibuzzard-66FDA353, F.Cu at (61.0, 70.6)
- added kibuzzard-66FEA7C0: G***, kibuzzard-66FEA7C0, F.Cu at (186.1, 31.8)
- added kibuzzard-66FEA7DC: G***, kibuzzard-66FEA7DC, F.Cu at (175.1, 144.1)
- added kibuzzard-66FEA7EE: G***, kibuzzard-66FEA7EE, F.Cu at (189.7, 144.1)
- added kibuzzard-66FEA7FA: G***, kibuzzard-66FEA7FA, F.Cu at (182.2, 128.9)
- J10, J11, J12, J14, J6, J7, J9, SW1, SW2, SW3, SW4: footprint Connector_Molex:Molex_KK-254_AE-6410-04A_1x04_P2.54mm_Vertical -> Connector_JST:JST_XH_B4B-XH-A_1x04_P2.50mm_Vertical
- J13, J8: footprint Connector_Molex:Molex_KK-254_AE-6410-08A_1x08_P2.54mm_Vertical -> Connector_JST:JST_XH_B8B-XH-A_1x08_P2.50mm_Vertical
- J15: footprint Connector_Molex:Molex_KK-254_AE-6410-03A_1x03_P2.54mm_Vertical -> Connector_JST:JST_XH_B3B-XH-A_1x03_P2.50mm_Vertical
- J16: value LCD_TFT -> GPIO; footprint Connector_PinSocket_2.54mm:PinSocket_1x14_P2.54mm_Vertical -> Connector_JST:JST_XH_B4B-XH-A_1x04_P2.50mm_Vertical; moved to F.Cu
- J17: value LCD_SD -> SMD_Conn; footprint Connector_PinSocket_2.54mm:PinSocket_1x04_P2.54mm_Vertical -> Connector_PinHeader_2.54mm:PinHeader_1x04_P2.54mm_Vertical_SMD_Pin1Right; moved to F.Cu
- moved kibuzzard-26 109.3 mm to (189.7, 142.2), turned to 90 degrees
- moved G1 106.7 mm to (72.6, 89.4), turned to -90 degrees
- moved J14 101.7 mm to (193.6, 138.4), turned to 180 degrees
- moved kibuzzard-27 92.1 mm to (175.1, 133.3), turned to 90 degrees
- moved J15 88.8 mm to (177.7, 129.5), turned to 180 degrees
- moved J17 72.2 mm to (157.3, 47.3), turned to -90 degrees
- moved J16 68.0 mm to (164.3, 129.5)
- moved J2 32.0 mm to (106.2, 48.8)
- moved D7 26.1 mm to (74.2, 39.3), turned to -90 degrees
- moved D5 23.7 mm to (78.2, 39.3), turned to -90 degrees
- moved G*** 20.9 mm to (86.6, 39.6), turned to 0 degrees
- moved D6 19.7 mm to (82.2, 39.3), turned to -90 degrees
- moved DRV1 17.7 mm to (132.0, 41.9)
- moved TP6 17.7 mm to (116.7, 51.8)
- moved TP7 17.7 mm to (116.7, 49.2)
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Connections:
- J16 pad 1: +3.3V -> /PD7
- J16 pad 2: GND -> /PE2
- J16 pad 3: /PE0 -> /PE5
- J17 pad 1: /PA4 -> /PE0
- J17 pad 2: /PD7 -> /PA4
- J17 pad 3: /PA6 -> /PA5
- J17 pad 4: /PA5 -> /PA6
Routing:
- net +5V: track 404.3 -> 0.00 mm, vias 4 -> 0
- net +12VA: track 245.0 -> 0.00 mm
- net +3.3V: track 244.1 -> 0.00 mm, vias 3 -> 0
- net /AX12_RX: track 187.9 -> 0.00 mm, vias 1 -> 0
- net /I2C1_SDA: track 187.2 -> 0.00 mm, vias 2 -> 0
- net /PD7: track 169.9 -> 0.00 mm, vias 1 -> 0
- net +5VA: track 163.4 -> 0.00 mm
- net /PA6: track 139.6 -> 0.00 mm, vias 4 -> 0
- net /PA5: track 138.0 -> 0.00 mm, vias 2 -> 0
- net /Encodeur_Droit_B: track 137.1 -> 0.00 mm, vias 2 -> 0
- net /Encodeur_Droit_A: track 131.8 -> 0.00 mm, vias 2 -> 0
- net /I2C1_SCL: track 121.5 -> 0.00 mm, vias 1 -> 0
- net /PD4: track 101.9 -> 0.00 mm, vias 2 -> 0
- net /PF3: track 100.2 -> 0.00 mm, vias 1 -> 0
- net /DEBUG_RX: track 97.6 -> 0.00 mm
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Other:
- board text removed: "12 11 10 9 8 7 6 5 4 3 2 1 0"

Commit message: FInal
Parts:
- removed J11: I2C2, Connector_JST:JST_XH_B4B-XH-A_1x04_P2.50mm_Vertical
- removed J12, J16, J19: GPIO, Connector_JST:JST_XH_B4B-XH-A_1x04_P2.50mm_Vertical
- removed J14: I2C_Sensors, Connector_JST:JST_XH_B4B-XH-A_1x04_P2.50mm_Vertical
- removed J17: SMD_Conn, Connector_PinHeader_2.54mm:PinHeader_1x04_P2.54mm_Vertical_SMD_Pin1Right
- removed kibuzzard-11: G***, kibuzzard-66C08EB4
- removed kibuzzard-12: G***, kibuzzard-66C48662
- removed kibuzzard-13: G***, kibuzzard-66C46925
- removed kibuzzard-14: G***, kibuzzard-66C08BB8
- removed kibuzzard-26: G***, kibuzzard-66C091C7
- removed kibuzzard-31: G***, kibuzzard-66C09378
- removed kibuzzard-32: G***, kibuzzard-66C60E06
- removed kibuzzard-33: G***, kibuzzard-66C60E22
- removed kibuzzard-36: G***, kibuzzard-66C09018
- removed kibuzzard-66E9AA77: G***, kibuzzard-66E9AA77
- removed kibuzzard-66F082DD: G***, kibuzzard-66F082DD
- removed kibuzzard-66FEA7C0: G***, kibuzzard-66FEA7C0
- removed kibuzzard-66FEA7DC: G***, kibuzzard-66FEA7DC
- removed kibuzzard-66FEA7EE: G***, kibuzzard-66FEA7EE
- removed kibuzzard-66FEA7FA: G***, kibuzzard-66FEA7FA
- removed kibuzzard-9: G***, kibuzzard-66C092F4
- added BZ1: Buzzer, Buzzer_Beeper:Buzzer_12x9.5RM7.6, F.Cu at (73.7, 47.6)
- added J21: I2C Screen, Connector_JST:JST_XH_B4B-XH-A_1x04_P2.50mm_Vertical, F.Cu at (164.5, 130.2)
- added Q1: BC817, Package_TO_SOT_SMD:SOT-23, F.Cu at (90.3, 57.4)
- added R2: R, Resistor_SMD:R_1206_3216Metric_Pad1.30x1.75mm_HandSolder, F.Cu at (89.5, 62.5)
- added kibuzzard-67547681: G***, kibuzzard-67547681, F.Cu at (145.7, 144.8)
- added kibuzzard-67548783: G***, kibuzzard-67548783, F.Cu at (184.8, 144.8)
- added kibuzzard-67548923: G***, kibuzzard-67548923, F.Cu at (205.7, 45.6)
- added kibuzzard-6754898D: G***, kibuzzard-6754898D, B.Cu at (160.7, 134.6)
- added kibuzzard-675489B9: G***, kibuzzard-675489B9, B.Cu at (160.6, 142.6)
- added kibuzzard-675489F8: G***, kibuzzard-675489F8, B.Cu at (184.8, 143.5)
- added kibuzzard-67548A22: G***, kibuzzard-67548A22, B.Cu at (184.8, 134.0)
- added kibuzzard-67548BCB: G***, kibuzzard-67548BCB, F.Cu at (160.7, 144.8)
- added kibuzzard-6757392E: G***, kibuzzard-6757392E, F.Cu at (121.7, 51.8)
- added kibuzzard-67573990: G***, kibuzzard-67573990, F.Cu at (169.5, 31.9)
- added kibuzzard-675739BC: G***, kibuzzard-675739BC, F.Cu at (169.5, 41.9)
- G1: moved to B.Cu
- J10: value GPIO -> Sensors; footprint Connector_JST:JST_XH_B4B-XH-A_1x04_P2.50mm_Vertical -> Connector_JST:JST_XH_B10B-XH-A_1x10_P2.50mm_Vertical
- J7: value UART -> GPIO; footprint Connector_JST:JST_XH_B4B-XH-A_1x04_P2.50mm_Vertical -> Connector_JST:JST_XH_B10B-XH-A_1x10_P2.50mm_Vertical
- moved kibuzzard-27 90.4 mm to (197.5, 45.8), turned to 0 degrees
- moved J15 84.6 mm to (200.8, 48.2), turned to 90 degrees
- moved J7 75.9 mm to (196.0, 130.2)
- moved G1 74.0 mm to (146.7, 88.9)
- moved J10 60.9 mm to (196.0, 139.1)
- moved R34 52.3 mm to (144.3, 104.7), turned to 90 degrees
- moved U6 52.0 mm to (146.7, 43.2), turned to 90 degrees
- moved C6 50.2 mm to (143.5, 53.0), turned to 90 degrees
- moved U7 47.3 mm to (143.5, 43.2), turned to 90 degrees
- moved R33 46.7 mm to (140.7, 104.7), turned to 90 degrees
- moved C5 45.3 mm to (139.7, 53.0), turned to 90 degrees
- moved R31 44.2 mm to (137.2, 104.7), turned to 90 degrees
- moved U5 42.7 mm to (140.3, 43.2), turned to 90 degrees
- moved C4 40.5 mm to (135.9, 53.0), turned to 90 degrees
- moved R32 39.8 mm to (133.6, 104.7), turned to 90 degrees
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Connections:
- J10 pad 1: /PF8 -> /I2C2_SCL
- J10 pad 2: /PG1 -> /I2C2_SDA
- J10 pad 3: /PG0 -> /PD1
- J10 pad 4: /PD1 -> /PE2
- J7 pad 1: /PC7 -> GND
- J7 pad 2: /PC6 -> /PE0
- J7 pad 3: +5V -> /PF8
- J7 pad 4: GND -> /PD6
- U2 pad CN10_11: /PF6 -> /Encodeur_Droit_A
- U2 pad CN11_11: /Encodeur_Droit_B -> unconnected-(U2A-PF7-PadCN11_11)
- U2 pad CN11_41: /AX12_RX -> unconnected-(U2A-PD5-PadCN11_41)
- U2 pad CN11_6: unconnected-(U2A-5V_EXT-PadCN11_6) -> +5V
- U2 pad CN11_9: /Encodeur_Droit_A -> unconnected-(U2A-PF6-PadCN11_9)
- U2 pad CN12_37: /AX12_RX -> unconnected-(U2B-PA3-PadCN12_37)
- U2 pad CN7_1: /PC6 -> /AX12_RX
- U2 pad CN7_11: /PC7 -> /AX12_RX
- U2 pad CN9_26: /PF7 -> /Encodeur_Droit_B
Routing:
- net +5V: track 0.00 -> 418.8 mm, vias 0 -> 1
- net +3.3V: track 0.00 -> 240.8 mm, vias 0 -> 7
- net +12VA: track 0.00 -> 213.3 mm
- net /PF3: track 0.00 -> 134.4 mm, vias 0 -> 2
- net /AX12_RX: track 0.00 -> 120.8 mm, vias 0 -> 2
- net /PA5: track 0.00 -> 112.2 mm
- net /DEBUG_TX: track 0.00 -> 110.5 mm, vias 0 -> 1
- net /PA4: track 0.00 -> 107.0 mm, vias 0 -> 3
- net /Encodeur_Droit_A: track 0.00 -> 105.1 mm, vias 0 -> 2
- net /Encodeur_Droit_B: track 0.00 -> 98.1 mm, vias 0 -> 1
- net /I2C1_SCL: track 0.00 -> 97.7 mm, vias 0 -> 1
- net /Encodeur_Gauche_A: track 0.00 -> 95.3 mm, vias 0 -> 2
- net /Encodeur_Gauche_B: track 0.00 -> 85.7 mm, vias 0 -> 1
- net /PA15: track 0.00 -> 84.2 mm, vias 0 -> 1
- net /Encodeurs/A+_DROITE: track 0.00 -> 76.1 mm
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Other:
- board size 154.6 x 118.1 mm -> 140 x 118.1 mm
