File: Carte-Principale/Moteurs.kicad_sch (KiCad schematic)
At the start: 0 parts

Commit message: Moteurs + Encodeurs
Parts:
- added C1, C2, C3, C4: 100n, symbol Device:C_Small
- added DRV1: ~, Carte moteur V1.0:DRV8844_BREAKOUT_BOARD, symbol drv8844_breackout_board_dip:DRV8844_BREACKOUT_BOARD_DIP
- added J1: Moteur_Gauche, symbol Connector:Screw_Terminal_01x02
- added J2: Moteur_Droit, symbol Connector:Screw_Terminal_01x02
- added U2, U3, U4, U5: 74LVC1G3157, Package_TO_SOT_SMD:SOT-363_SC-70-6_Handsoldering, symbol 74xGxx:74LVC1G3157
Connections:
- new net +12VA: DRV1.VMOT
- new net +5V: C1.2, C2.2, C3.2, C4.2, DRV1.SLP, U2.5 (VCC), U3.5 (VCC), U4.5 (VCC), U5.5 (VCC)
- new net DIR_MOTEUR_DROITE: U4.6, U5.6
- new net DIR_MOTEUR_GAUCHE: U2.6, U3.6
- new net EN_MOTEUR_DROIT: DRV1.EN2
- new net EN_MOTEUR_GAUCHE: DRV1.EN1
- new net FAULTDRV: DRV1.FLT
- new net GND: C1.1, C2.1, C3.1, C4.1, DRV1.GND, DRV1.GND1, U2.1, U2.2 (GND), U3.2 (GND), U3.3, U4.1, U4.2 (GND), U5.2 (GND), U5.3
- new net IN1: DRV1.IN1, U2.4
- new net IN2: DRV1.IN2, U3.4
- new net IN3: DRV1.IN3, U4.4
- new net IN4: DRV1.IN4, U5.4
- new net MOTOR1A: DRV1.1A, J1.1 (Pin_1)
- new net MOTOR1B: DRV1.1B, J1.2 (Pin_2)
- new net MOTOR2A: DRV1.2A, J2.1 (Pin_1)
- new net MOTOR2B: DRV1.2B, J2.2 (Pin_2)
- new net PWM_MOTEUR_DROITE: U4.3, U5.1
- new net PWM_MOTEUR_GAUCHE: U2.3, U3.1
- new net RSTDRV: DRV1.RST

Commit message: wiring
Parts:
- added TP3: Test_PWM, TestPoint:TestPoint_2Pads_Pitch2.54mm_Drill0.8mm, symbol Connector:TestPoint_2Pole
- added TP4: Test_DIR, TestPoint:TestPoint_2Pads_Pitch2.54mm_Drill0.8mm, symbol Connector:TestPoint_2Pole
- C2: renamed from C1; footprint (none) -> Capacitor_SMD:C_1206_3216Metric_Pad1.33x1.80mm_HandSolder
- C3: renamed from C2; footprint (none) -> Capacitor_SMD:C_1206_3216Metric_Pad1.33x1.80mm_HandSolder
- C4: renamed from C3; footprint (none) -> Capacitor_SMD:C_1206_3216Metric_Pad1.33x1.80mm_HandSolder
- C5: renamed from C4; footprint (none) -> Capacitor_SMD:C_1206_3216Metric_Pad1.33x1.80mm_HandSolder
- DRV1: footprint Carte moteur V1.0:DRV8844_BREAKOUT_BOARD -> DRV8844:DRV8844_BREAKOUT_BOARD
- J6: renamed from J1; footprint (none) -> TerminalBlock:TerminalBlock_bornier-2_P5.08mm
- J7: renamed from J2; footprint (none) -> TerminalBlock:TerminalBlock_bornier-2_P5.08mm
- renumbered U2 to U3, U3 to U4, U4 to U5, U5 to U6
Connections:
- net DIR_MOTEUR_DROITE: now also TP4.1
- net DIR_MOTEUR_GAUCHE: now also TP4.2
- net PWM_MOTEUR_DROITE renamed PWM_MOTEUR_DROITE_H
- net PWM_MOTEUR_DROITE_H: now also TP3.1
- net PWM_MOTEUR_GAUCHE renamed PWM_MOTEUR_GAUCHE_H
- net PWM_MOTEUR_GAUCHE_H: now also TP3.2

Commit message: Schéma vérifié
Parts:
- C2, C3, C4, C5: footprint Capacitor_SMD:C_1206_3216Metric_Pad1.33x1.80mm_HandSolder -> Capacitor_SMD:C_1210_3225Metric_Pad1.33x2.70mm_HandSolder
- renumbered J6 to J13, J7 to J14, TP4 to TP10, TP3 to TP9
Connections:
- net +5V: no longer C2.2, C3.2, C4.2, C5.2, U3.5 (VCC), U4.5 (VCC), U5.5 (VCC), U6.5 (VCC)
- new net +3.3V: C2.2, C3.2, C4.2, C5.2, U3.5 (VCC), U4.5 (VCC), U5.5 (VCC), U6.5 (VCC)
Other:
- company: (none) -> CRINSA
- title: (none) -> Carte Principale
- moved on the sheet: C2, C3, C4, C5, DRV1, J13, J14, TP10, TP9, U3A, U3B, U4A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

Commit message: Avancée PCB
Parts:
- renumbered C2 to C1, C3 to C2, C4 to C3, C5 to C4, J13 to J10, J14 to J11, TP9 to TP8, TP10 to TP9
Changed lines of the file:
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@@
 		(dnp no)
 		(fields_autoplaced yes)
-		(property "Reference" "#PWR044"
+		(property "Reference" "#PWR038"
 			(at 60.96 53.34 0)
 			(effects
@@
 			(project "Carte-Principale"
 				(path "/88b0dd29-ac24-4c5d-804c-fc642ecf6263/de945202-06d9-4619-881a-1edba2d78bfe"
-					(reference "#PWR044")
+					(reference "#PWR038")
 					(unit 1)
 				)
@@
 		(dnp no)
 		(fields_autoplaced yes)
-		(property "Reference" "#PWR047"
+		(property "Reference" "#PWR041"
 			(at 194.31 73.66 0)
 			(effects
@@
 			(project "Carte-Principale"
 				(path "/88b0dd29-ac24-4c5d-804c-fc642ecf6263/de945202-06d9-4619-881a-1edba2d78bfe"
-					(reference "#PWR047")
+					(reference "#PWR041")
 					(unit 1)
 				)
@@
 		(dnp no)
 		(fields_autoplaced yes)
-		(property "Reference" "#PWR046"
+		(property "Reference" "#PWR040"
 			(at 166.37 73.66 0)
 			(effects
@@
 			(project "Carte-Principale"
 				(path "/88b0dd29-ac24-4c5d-804c-fc642ecf6263/de945202-06d9-4619-881a-1edba2d78bfe"
-					(reference "#PWR046")
+					(reference "#PWR040")
 					(unit 1)
 				)
@@
 		(on_board yes)
 		(dnp no)
-		(property "Reference" "#PWR042"
+		(property "Reference" "#PWR036"
 			(at 111.76 41.91 0)
 			(effects
@@
 			(project "Carte-Principale"
 				(path "/88b0dd29-ac24-4c5d-804c-fc642ecf6263/de945202-06d9-4619-881a-1edba2d78bfe"
-					(reference "#PWR042")
+					(reference "#PWR036")
 					(unit 1)
 				)
@@
 		(dnp no)
 		(fields_autoplaced yes)
-		(property "Reference" "C5"
+		(property "Reference" "C4"
 			(at 175.2536 140.97 90)
 			(effects
@@
 			(project "Carte-Principale"
 				(path "/88b0dd29-ac24-4c5d-804c-fc642ecf6263/de945202-06d9-4619-881a-1edba2d78bfe"
-					(reference "C5")
+					(reference "C4")
 					(unit 1)
 				)
@@
 		(dnp no)
 		(fields_autoplaced yes)
-		(property "Reference" "#PWR043"
+		(property "Reference" "#PWR037"
 			(at 53.34 60.96 0)
 			(effects
@@
 			(project "Carte-Principale"
 				(path "/88b0dd29-ac24-4c5d-804c-fc642ecf6263/de945202-06d9-4619-881a-1edba2d78bfe"
-					(reference "#PWR043")
+					(reference "#PWR037")
 					(unit 1)
 				)
@@
 		(dnp no)
 		(fields_autoplaced yes)
-		(property "Reference" "C3"
+		(property "Reference" "C2"
 			(at 175.2536 99.06 90)
 			(effects
@@
 			(project "Carte-Principale"
 				(path "/88b0dd29-ac24-4c5d-804c-fc642ecf6263/de945202-06d9-4619-881a-1edba2d78bfe"
-					(reference "C3")
+					(reference "C2")
 					(unit 1)
 				)
@@
 		(dnp no)
 		(fields_autoplaced yes)
-		(property "Reference" "J14"
+		(property "Reference" "J11"
 			(at 185.42 45.7199 0)
 			(effects
@@
 			(project "Carte-Principale"
 				(path "/88b0dd29-ac24-4c5d-804c-fc642ecf6263/de945202-06d9-4619-881a-1edba2d78bfe"
-					(reference "J14")
+					(reference "J11")
 					(unit 1)
 				)
@@
 		(dnp no)
 		(fields_autoplaced yes)
-		(property "Reference" "#PWR041"
+		(property "Reference" "#PWR035"
 			(at 53.34 45.72 0)
 			(effects
@@
 			(project "Carte-Principale"
 				(path "/88b0dd29-ac24-4c5d-804c-fc642ecf6263/de945202-06d9-4619-881a-1edba2d78bfe"
-					(reference "#PWR041")
+					(reference "#PWR035")
 					(unit 1)
 				)
@@
 		(dnp no)
 		(fields_autoplaced yes)
-		(property "Reference" "#PWR045"
+		(property "Reference" "#PWR039"
 			(at 97.79 59.69 0)
 			(effects
@@
 			(project "Carte-Principale"
 				(path "/88b0dd29-ac24-4c5d-804c-fc642ecf6263/de945202-06d9-4619-881a-1edba2d78bfe"
-					(reference "#PWR045")
+					(reference "#PWR039")
 					(unit 1)
 				)
@@
 		(dnp no)
 		(fields_autoplaced yes)
-		(property "Reference" "C4"
+		(property "Reference" "C3"
 			(at 175.2536 120.65 90)
 			(effects
@@
 			(project "Carte-Principale"
 				(path "/88b0dd29-ac24-4c5d-804c-fc642ecf6263/de945202-06d9-4619-881a-1edba2d78bfe"
-					(reference "C4")
+					(reference "C3")
 					(unit 1)
 				)
@@
 		(dnp no)
 		(fields_autoplaced yes)
-		(property "Reference" "J13"
+		(property "Reference" "J10"
 			(at 185.42 38.0999 0)
 			(effects
@@
 			(project "Carte-Principale"
 				(path "/88b0dd29-ac24-4c5d-804c-fc642ecf6263/de945202-06d9-4619-881a-1edba2d78bfe"
-					(reference "J13")
+					(reference "J10")
 					(unit 1)
 				)
@@
 		(dnp no)
 		(fields_autoplaced yes)
-		(property "Reference" "C2"
+		(property "Reference" "C1"
 			(at 175.2536 77.47 90)
 			(effects
@@
 			(project "Carte-Principale"
 				(path "/88b0dd29-ac24-4c5d-804c-fc642ecf6263/de945202-06d9-4619-881a-1edba2d78bfe"
-					(reference "C2")
+					(reference "C1")
 					(unit 1)
 				)
@@
 		(dnp no)
 		(fields_autoplaced yes)
-		(property "Reference" "TP9"
+		(property "Reference" "TP8"
 			(at 105.41 99.0599 90)
 			(effects
@@
 			(project "Carte-Principale"
 				(path "/88b0dd29-ac24-4c5d-804c-fc642ecf6263/de945202-06d9-4619-881a-1edba2d78bfe"
-					(reference "TP9")
+					(reference "TP8")
 					(unit 1)
 				)
@@
 		(on_board yes)
 		(dnp no)
-		(property "Reference" "TP10"
+		(property "Reference" "TP9"
 			(at 53.34 105.41 90)
 			(effects
@@
 			(project "Carte-Principale"
 				(path "/88b0dd29-ac24-4c5d-804c-fc642ecf6263/de945202-06d9-4619-881a-1edba2d78bfe"
-					(reference "TP10")
-					(unit 1)
-				)
+					(reference "TP9")
+					(unit 1)
+				)

Commit message: avancée
Parts:
- renumbered C1 to C5, C2 to C6, J10 to J1, J11 to J4, TP8 to TP6, TP9 to TP7, U6 to U4, U4 to U6, U3 to U7
Changed lines of the file:
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@@
 		(dnp no)
 		(fields_autoplaced yes)
-		(property "Reference" "U3"
+		(property "Reference" "U7"
 			(at 82.55 60.96 0)
 			(effects
@@
 			(project "Carte-Principale"
 				(path "/88b0dd29-ac24-4c5d-804c-fc642ecf6263/de945202-06d9-4619-881a-1edba2d78bfe"
-					(reference "U3")
+					(reference "U7")
 					(unit 1)
 				)
@@
 		(dnp no)
 		(fields_autoplaced yes)
-		(property "Reference" "U4"
+		(property "Reference" "U6"
 			(at 175.26 87.63 90)
 			(effects
@@
 			(project "Carte-Principale"
 				(path "/88b0dd29-ac24-4c5d-804c-fc642ecf6263/de945202-06d9-4619-881a-1edba2d78bfe"
-					(reference "U4")
+					(reference "U6")
 					(unit 2)
 				)
@@
 		(dnp no)
 		(fields_autoplaced yes)
-		(property "Reference" "C2"
+		(property "Reference" "C6"
 			(at 175.2536 99.06 90)
 			(effects
@@
 			(project "Carte-Principale"
 				(path "/88b0dd29-ac24-4c5d-804c-fc642ecf6263/de945202-06d9-4619-881a-1edba2d78bfe"
-					(reference "C2")
+					(reference "C6")
 					(unit 1)
 				)
@@
 		(dnp no)
 		(fields_autoplaced yes)
-		(property "Reference" "J11"
+		(property "Reference" "J4"
 			(at 185.42 45.7199 0)
 			(effects
@@
 			(project "Carte-Principale"
 				(path "/88b0dd29-ac24-4c5d-804c-fc642ecf6263/de945202-06d9-4619-881a-1edba2d78bfe"
-					(reference "J11")
+					(reference "J4")
 					(unit 1)
 				)
@@
 		(dnp no)
 		(fields_autoplaced yes)
-		(property "Reference" "J10"
+		(property "Reference" "J1"
 			(at 185.42 38.0999 0)
 			(effects
@@
 			(project "Carte-Principale"
 				(path "/88b0dd29-ac24-4c5d-804c-fc642ecf6263/de945202-06d9-4619-881a-1edba2d78bfe"
-					(reference "J10")
+					(reference "J1")
 					(unit 1)
 				)
@@
 		(dnp no)
 		(fields_autoplaced yes)
-		(property "Reference" "U6"
+		(property "Reference" "U4"
 			(at 82.55 138.43 0)
 			(effects
@@
 			(project "Carte-Principale"
 				(path "/88b0dd29-ac24-4c5d-804c-fc642ecf6263/de945202-06d9-4619-881a-1edba2d78bfe"
-					(reference "U6")
+					(reference "U4")
 					(unit 1)
 				)
@@
 		(dnp no)
 		(fields_autoplaced yes)
-		(property "Reference" "U3"
+		(property "Reference" "U7"
 			(at 175.26 66.04 90)
 			(effects
@@
 			(project "Carte-Principale"
 				(path "/88b0dd29-ac24-4c5d-804c-fc642ecf6263/de945202-06d9-4619-881a-1edba2d78bfe"
-					(reference "U3")
+					(reference "U7")
 					(unit 2)
 				)
@@
 		(dnp no)
 		(fields_autoplaced yes)
-		(property "Reference" "U4"
+		(property "Reference" "U6"
 			(at 82.55 86.36 0)
 			(effects
@@
 			(project "Carte-Principale"
 				(path "/88b0dd29-ac24-4c5d-804c-fc642ecf6263/de945202-06d9-4619-881a-1edba2d78bfe"
-					(reference "U4")
+					(reference "U6")
 					(unit 1)
 				)
@@
 		(dnp no)
 		(fields_autoplaced yes)
-		(property "Reference" "C1"
+		(property "Reference" "C5"
 			(at 175.2536 77.47 90)
 			(effects
@@
 			(project "Carte-Principale"
 				(path "/88b0dd29-ac24-4c5d-804c-fc642ecf6263/de945202-06d9-4619-881a-1edba2d78bfe"
-					(reference "C1")
+					(reference "C5")
 					(unit 1)
 				)
@@
 		(dnp no)
 		(fields_autoplaced yes)
-		(property "Reference" "TP8"
+		(property "Reference" "TP6"
 			(at 105.41 99.0599 90)
 			(effects
@@
 			(project "Carte-Principale"
 				(path "/88b0dd29-ac24-4c5d-804c-fc642ecf6263/de945202-06d9-4619-881a-1edba2d78bfe"
-					(reference "TP8")
+					(reference "TP6")
 					(unit 1)
 				)
@@
 		(dnp no)
 		(fields_autoplaced yes)
-		(property "Reference" "U6"
+		(property "Reference" "U4"
 			(at 175.26 129.54 90)
 			(effects
@@
 			(project "Carte-Principale"
 				(path "/88b0dd29-ac24-4c5d-804c-fc642ecf6263/de945202-06d9-4619-881a-1edba2d78bfe"
-					(reference "U6")
+					(reference "U4")
 					(unit 2)
 				)
@@
 		(on_board yes)
 		(dnp no)
-		(property "Reference" "TP9"
+		(property "Reference" "TP7"
 			(at 53.34 105.41 90)
 			(effects
@@
 			(project "Carte-Principale"
 				(path "/88b0dd29-ac24-4c5d-804c-fc642ecf6263/de945202-06d9-4619-881a-1edba2d78bfe"
-					(reference "TP9")
-					(unit 1)
-				)
+					(reference "TP7")
+					(unit 1)
+				)

Commit message: Final pcb modification
Parts:
- renumbered C4 to C3, C3 to C4, C6 to C5, C5 to C6, J4 to J5, U7 to U6, U6 to U7
Changed lines of the file:
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@@
 		(dnp no)
 		(fields_autoplaced yes)
-		(property "Reference" "U7"
+		(property "Reference" "U6"
 			(at 82.55 60.96 0)
 			(effects
@@
 			(project "Carte-Principale"
 				(path "/88b0dd29-ac24-4c5d-804c-fc642ecf6263/de945202-06d9-4619-881a-1edba2d78bfe"
-					(reference "U7")
+					(reference "U6")
 					(unit 1)
 				)
@@
 		(dnp no)
 		(fields_autoplaced yes)
-		(property "Reference" "C4"
+		(property "Reference" "C3"
 			(at 175.2536 140.97 90)
 			(effects
@@
 			(project "Carte-Principale"
 				(path "/88b0dd29-ac24-4c5d-804c-fc642ecf6263/de945202-06d9-4619-881a-1edba2d78bfe"
-					(reference "C4")
+					(reference "C3")
 					(unit 1)
 				)
@@
 		(dnp no)
 		(fields_autoplaced yes)
-		(property "Reference" "U6"
+		(property "Reference" "U7"
 			(at 175.26 87.63 90)
 			(effects
@@
 			(project "Carte-Principale"
 				(path "/88b0dd29-ac24-4c5d-804c-fc642ecf6263/de945202-06d9-4619-881a-1edba2d78bfe"
-					(reference "U6")
+					(reference "U7")
 					(unit 2)
 				)
@@
 		(dnp no)
 		(fields_autoplaced yes)
-		(property "Reference" "C6"
+		(property "Reference" "C5"
 			(at 175.2536 99.06 90)
 			(effects
@@
 			(project "Carte-Principale"
 				(path "/88b0dd29-ac24-4c5d-804c-fc642ecf6263/de945202-06d9-4619-881a-1edba2d78bfe"
-					(reference "C6")
+					(reference "C5")
 					(unit 1)
 				)
@@
 		(dnp no)
 		(fields_autoplaced yes)
-		(property "Reference" "J4"
+		(property "Reference" "J5"
 			(at 185.42 45.7199 0)
 			(effects
@@
 			(project "Carte-Principale"
 				(path "/88b0dd29-ac24-4c5d-804c-fc642ecf6263/de945202-06d9-4619-881a-1edba2d78bfe"
-					(reference "J4")
+					(reference "J5")
 					(unit 1)
 				)
@@
 		(dnp no)
 		(fields_autoplaced yes)
-		(property "Reference" "C3"
+		(property "Reference" "C4"
 			(at 175.2536 120.65 90)
 			(effects
@@
 			(project "Carte-Principale"
 				(path "/88b0dd29-ac24-4c5d-804c-fc642ecf6263/de945202-06d9-4619-881a-1edba2d78bfe"
-					(reference "C3")
+					(reference "C4")
 					(unit 1)
 				)
@@
 		(dnp no)
 		(fields_autoplaced yes)
-		(property "Reference" "U7"
+		(property "Reference" "U6"
 			(at 175.26 66.04 90)
 			(effects
@@
 			(project "Carte-Principale"
 				(path "/88b0dd29-ac24-4c5d-804c-fc642ecf6263/de945202-06d9-4619-881a-1edba2d78bfe"
-					(reference "U7")
+					(reference "U6")
 					(unit 2)
 				)
@@
 		(dnp no)
 		(fields_autoplaced yes)
-		(property "Reference" "U6"
+		(property "Reference" "U7"
 			(at 82.55 86.36 0)
 			(effects
@@
 			(project "Carte-Principale"
 				(path "/88b0dd29-ac24-4c5d-804c-fc642ecf6263/de945202-06d9-4619-881a-1edba2d78bfe"
-					(reference "U6")
+					(reference "U7")
 					(unit 1)
 				)
@@
 		(dnp no)
 		(fields_autoplaced yes)
-		(property "Reference" "C5"
+		(property "Reference" "C6"
 			(at 175.2536 77.47 90)
 			(effects
@@
 			(project "Carte-Principale"
 				(path "/88b0dd29-ac24-4c5d-804c-fc642ecf6263/de945202-06d9-4619-881a-1edba2d78bfe"
-					(reference "C5")
-					(unit 1)
-				)
+					(reference "C6")
+					(unit 1)
+				)

Commit message: FInal
Other:
- note added: "Driver moteur du club robot (basé sur un drv8844)"
- note added: "Repris des années précédentes, marche bien"
- note added: "Switch des de direction des moteurs"
Changed lines of the file:
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@@
+		)
+	)
+	(text "Repris des années précédentes, marche bien"
+		(exclude_from_sim no)
+		(at 143.51 20.32 0)
+		(effects
+			(font
+				(size 5 5)
+			)
+		)
+	)
+	(text "Driver moteur du club robot (basé sur un drv8844)"
+		(exclude_from_sim no)
+		(at 97.79 31.75 0)
+		(effects
+			(font
+				(size 1.27 1.27)
+			)
+		)
+	)
+	(text "Switch des de direction des moteurs"
+		(exclude_from_sim no)
+		(at 120.65 73.66 0)
+		(effects
+			(font
+				(size 1.27 1.27)
+			)
 		)
 	)
@@
 		(on_board yes)
 		(dnp no)
-		(fields_autoplaced yes)
 		(property "Reference" "DRV1"
-			(at 96.52 30.48 0)
-			(effects
-				(font
+			(at 96.52 33.02 0)
+			(effects
+				(font
