File: Carte-Principale/Moteurs.kicad_sch (KiCad schematic)
At the start: 13 parts, among them J1 Moteur_Gauche, J5 Moteur_Droit, U4 74LVC1G3157, U5 74LVC1G3157, U6 74LVC1G3157, U7 74LVC1G3157

Commit message: abcdefgh
Other:
- company: CRINSA -> CRINSA - Boris HILKENS
Changed lines of the file:
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@@
 	(title_block
 		(title "Carte Principale")
-		(date "2024-08-12")
-		(company "CRINSA")
+		(date "2024-12-27")
+		(rev "V1")
+		(company "CRINSA - Boris HILKENS")
 		(comment 1 "Carte de contrôle pour le robot")
 	)
