File: Carte-Principale/Carte-Principale.kicad_sch (KiCad schematic)
At the start: 13 parts, among them J10 GPIO, J11 I2C2, J12 GPIO, J2 GND, J6 UART_Debug, J7 UART, J9 SPI3, U2 NUCLEOH723ZG

Commit message: Cartes élec à refaire et TODO
Parts:
- added J16, J19: GPIO, Connector_JST:JST_XH_B4B-XH-A_1x04_P2.50mm_Vertical, symbol Connector:Conn_01x04_Pin
- added J17: SMD_Conn, Connector_PinHeader_2.54mm:PinHeader_1x04_P2.54mm_Vertical_SMD_Pin1Right, symbol Connector:Conn_01x04_Pin
- J10, J11, J12, J6, J7, J9: footprint Connector_Molex:Molex_KK-254_AE-6410-04A_1x04_P2.54mm_Vertical -> Connector_JST:JST_XH_B4B-XH-A_1x04_P2.50mm_Vertical
Connections:
- net +5V: now also J19.3 (Pin_3)
- net GND: now also J19.4 (Pin_4)
- net PA4: now also J17.2 (Pin_2)
- net PA5: now also J17.3 (Pin_3)
- net PA6: now also J17.4 (Pin_4)
- net PD7: now also J16.1 (Pin_1)
- net PE0: now also J17.1 (Pin_1)
- net PE2: now also J16.2 (Pin_2)
- net PE3: now also J19.1 (Pin_1)
- net PE4: now also J16.4 (Pin_4)
- net PE5: now also J16.3 (Pin_3)
- net PF2: now also J19.2 (Pin_2)
Other:
- sheet IHM ports: added none; removed CS_LCD, CS_SD, DC_LCD, MISO_LCD, MISO_SD, MOSI_LCD, MOSI_SD, RESET_LCD, SCK_LCD, SCK_SD, T_CS_LCD, T_IRQ_LCD, T_MISO_LCD, T_MOSI_LCD, T_SCK_LCD
- note added: "TIM23 -> Encodeur Droit TIM24 -> Encodeur Gauche TIM1 -> PWM Moteurs USART2 -> AX12 USART3 -> Debug + Serial console USART6 -> ESP32 I2C1 -> Sensors + Servos PF2 -> EXTI2 Touch PF3 -> EXTI3 Sensors"
- note removed: "TIM23 -> Encodeur Droit TIM24 -> Encodeur Gauche TIM1 -> PWM Moteurs USART2 -> AX12 USART3 -> Debug + Serial console I2C1 -> Sensors + Servos SPI1 -> LCD + Touch + SD PF2 -> EXTI2 Touch PF3 -> EXTI3 Sensors"
- moved on the sheet: J2

Commit message: FInal
Parts:
- removed J10, J12, J16, J19: GPIO, Connector_JST:JST_XH_B4B-XH-A_1x04_P2.50mm_Vertical, symbol Connector:Conn_01x04_Pin
- removed J11: I2C2, Connector_JST:JST_XH_B4B-XH-A_1x04_P2.50mm_Vertical, symbol Connector:Conn_01x04_Pin
- removed J17: SMD_Conn, Connector_PinHeader_2.54mm:PinHeader_1x04_P2.54mm_Vertical_SMD_Pin1Right, symbol Connector:Conn_01x04_Pin
- removed J7: UART, Connector_JST:JST_XH_B4B-XH-A_1x04_P2.50mm_Vertical, symbol Connector:Conn_01x04_Pin
- added J7: GPIO, Connector_JST:JST_XH_B10B-XH-A_1x10_P2.50mm_Vertical, symbol Connector:Conn_01x10_Pin
Connections:
- net PC6 is gone; now on net AX12_RX: U2.CN7_1 (D16/I2S_A_MCK)
- net PC7 is gone; now on net AX12_RX: U2.CN7_11 (D21/I2S_B_MCK)
- net PF6 is gone; now on net Encodeur_Droit_A: U2.CN10_11 (A8/ADC_C_IN)
- net PF7 is gone; now on net Encodeur_Droit_B: U2.CN9_26 (D62/SAI_B_MCLK)
- net +5V: now also U2.CN11_6 (5V_EXT)
- net AX12_RX: no longer U2.CN11_41 (PD5), U2.CN12_37 (PA3)
- net Encodeur_Droit_A: no longer U2.CN11_9 (PF6)
- net Encodeur_Droit_B: no longer U2.CN11_11 (PF7)
- net GND: now also J7.1 (Pin_1)
- net PA4: now also J7.6 (Pin_6)
- net PA5: now also J7.5 (Pin_5)
- net PD6: now also J7.4 (Pin_4)
- net PD7: now also J7.7 (Pin_7)
- net PE0: now also J7.2 (Pin_2)
- net PF2: now also J7.10 (Pin_10)
- net PF3: now also J7.9 (Pin_9)
- net PF8: now also J7.3 (Pin_3)
- net PF9: now also J7.8 (Pin_8)
- no-connect marks 161 -> 163
Other:
- sheet Actionneurs + sensors ports: added SHUT_1, SHUT_2, SHUT_3, SHUT_4, SHUT_5, SHUT_6, SHUT_7, SHUT_8; removed IT_Ready_Sensors
- sheet IHM ports: added Buzzer, LCD_SCK, LCD_SDA; removed none
- note added: "Bien Def Pull Down sur les inputs"
- note added: "TIM23 -> Encodeur Droit (PF6 & PF7) TIM24 -> Encodeur Gauche (PF11 & PF12) TIM1 -> PWM Moteurs (PE9 & PE11) USART6 -> AX12 USART3 -> Debug + Serial console I2C1 -> Écran + Servos + ESP32? I2C2 -> Sensors"
- note removed: "Alimenté via USB"
- note removed: "Bien Def Pull Down"
- note removed: "TIM23 -> Encodeur Droit TIM24 -> Encodeur Gauche TIM1 -> PWM Moteurs USART2 -> AX12 USART3 -> Debug + Serial console USART6 -> ESP32 I2C1 -> Sensors + Servos PF2 -> EXTI2 Touch PF3 -> EXTI3 Sensors"

Commit message: abcdefgh
Other:
- note added: "TODO: -tirette -Revoir forme PCB pour btn reset et leds user -Meilleurs connecteurs Alim ?"
- company: CRINSA -> CRINSA - Boris HILKENS
Changed lines of the file:
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@@
 	(title_block
 		(title "Carte Principale")
-		(date "2024-08-12")
-		(company "CRINSA")
+		(date "2024-12-27")
+		(rev "V1")
+		(company "CRINSA - Boris HILKENS")
 		(comment 1 "Carte de contrôle pour le robot")
 	)
@@
 		)
 	)
+	(text "TODO: \n-tirette\n-Revoir forme PCB pour btn reset et leds user\n-Meilleurs connecteurs Alim ?\n"
+		(exclude_from_sim no)
+		(at 262.89 167.64 0)
+		(effects
+			(font
+				(size 4 4)
+			)
+			(justify left)
+		)
+	)
