File: Carte-Principale/Puissance.kicad_sch (KiCad schematic)
At the start: 14 parts, among them J3 12VA, J4 5V

Commit message: FInal
Other:
- note removed: "Todo: faire BMS sur pcb annexe"
Changed lines of the file:
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@@
-		)
-	)
-	(text "Todo: faire BMS sur pcb annexe\n"
-		(exclude_from_sim no)
-		(at 115.57 77.47 0)
-		(effects
-			(font
-				(size 1.27 1.27)
-			)
 		)
 	)

Commit message: abcdefgh
Parts:
- added D1: D, Diode_SMD:D_SMB, symbol Device:D
- added D2: 200V 3A, Diode_SMD:D_SMC, symbol Device:D
- J3: footprint Connector_AMASS:AMASS_XT60-M_1x02_P7.20mm_Vertical -> TerminalBlock:TerminalBlock_bornier-2_P5.08mm
- J4: footprint Connector_AMASS:AMASS_XT30U-M_1x02_P5.0mm_Vertical -> TerminalBlock:TerminalBlock_bornier-2_P5.08mm
Connections:
- net at F1.1: now also D2.1 (K); no longer J3.2 (Pin_2)
- net at F2.1: now also D1.1 (K); no longer J4.2 (Pin_2)
- new net: D2.2 (A), J3.2 (Pin_2)
- new net: D1.2 (A), J4.2 (Pin_2)
Other:
- company: CRINSA -> CRINSA - Boris HILKENS
- moved on the sheet: F1, F2
